File: pcb/labAThome.sch (KiCad schematic (older format))
At the start: 81 parts, among them J1 I2C, J10 SRV2, J11 24.5.GND.3, J12 NEOPIXEL, J13 Barrel_Jack_Switch, J14 Conn_Coaxial, J15 WS2812_OUT, J2 SRV1, J3 5V, J4 EXT, J5 VPS, J6 FAN3, J7 1wire, J8 1wire, J9 FAN1, K1 G5V-2, K2 G5V-2, K3 G5V-2, M1 HXJ8002_MODULE, M3 SN65HVD230_MODULE, Q1 IRLML6344, Q2 IRLZ44N, Q3 IRLML6344, Q4 BC847, SW1 RED, SW2 GREEN, SW4 BLUE, SW5 WHITE, SW7 ROTENC, U1 SR602, U10 MAX3485_MODULE, U11 AM312, U2 24V->5V, U3 PDC004_Module, U4 ESP32_DEVKITC_COMPATIBLE, U5 LD06AJSA, U6 GY-302, U7 Display, U8 INMP441_Module, U9 RFM95W-868S2, X1 FAN_6024, m1 Attribution

Commit message: Overall unspecific update
Parts:
- removed J10: SRV2, Connector_PinHeader_2.54mm:PinHeader_1x03_P2.54mm_Vertical, symbol Connector:Conn_01x03_Male
- removed J2: SRV1, Connector_PinHeader_2.54mm:PinHeader_1x03_P2.54mm_Vertical, symbol Connector:Conn_01x03_Male
- removed J7, J8: 1wire, Connector_JST:JST_XH_B3B-XH-A_1x03_P2.50mm_Vertical, symbol Connector_Generic:Conn_01x03
- removed JP2, JP3: MECHANICAL, Connector_PinHeader_2.54mm:PinHeader_1x02_P2.54mm_Vertical, symbol Device:Jumper_NO_Small
- added C3: 1m, Capacitor_Tantalum_SMD:CP_EIA-7360-38_Kemet-E_Pad2.25x4.25mm_HandSolder, symbol Device:CP
- added C4, C5: u1, Capacitor_SMD:C_1206_3216Metric_Pad1.42x1.75mm_HandSolder, symbol Device:C
- added D10, D11, D2, D3, D9: 3528, LED_SMD:LED_PLCC_2835_Handsoldering, symbol Device:LED_Small
- added GSM_Module1: SIM800L, smopla:SIM800L, symbol sim800l:SIM800L
- added J2: SRVx, Connector_PinHeader_2.54mm:PinHeader_2x03_P2.54mm_Vertical, symbol Connector_Generic:Conn_02x03_Odd_Even
- added J8, j/1: 1wire, Connector_JST:JST_XH_B4B-XH-A_1x04_P2.50mm_Vertical, symbol Connector:Conn_01x04_Male
- added Q5: IRLZ44N, Package_TO_SOT_THT:TO-220-3_Horizontal_TabDown, symbol Device:Q_NMOS_GDS
- added R17, R8: 1K, Resistor_SMD:R_1206_3216Metric_Pad1.42x1.75mm_HandSolder, symbol Device:R
- added R22: K1, Resistor_SMD:R_1206_3216Metric_Pad1.42x1.75mm_HandSolder, symbol Device:R
- added R23: 1k, Resistor_SMD:R_1206_3216Metric_Pad1.42x1.75mm_HandSolder, symbol Device:R
- added R24: R1, Resistor_SMD:R_1206_3216Metric_Pad1.42x1.75mm_HandSolder, symbol Device:R
- added RV2: 10k, Potentiometer_SMD:Potentiometer_Vishay_TS53YL_Vertical, symbol Device:R_POT
- added U12: 24V->4V, sensact:MODULE_STEPDOWN, symbol sensact:MODULE_STEPDOWN
- added U13: LM358, sensact:SOIC-8_3.9x4.9mm_Pitch1.27mm_handsolder, symbol Amplifier_Operational:LM358
- J6: value FAN3 -> FAN2
Connections:
- net labels added: +4V, FAN_SUPPLY
- wire segments 143 -> 163
- no-connect marks 19 -> 26
Other:
- note added: "Drawings & Mounting"
- note added: "Wireless Long Range Communication Options"
- moved on the sheet: D5, D6, D7, FID1, FID3, J12, J13, J14, J15, J3, J4, J5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

Commit message: labathome V5.1 as ordered at JLCPCB
Parts:
- added C6: u1, Capacitor_SMD:C_1206_3216Metric_Pad1.42x1.75mm_HandSolder, symbol Device:C
- added U14: MS4525DO, smopla:MS4525DO, symbol smopla:MS4525DO
- D1: value LED -> HEATER ON; footprint LED_SMD:LED_0805_2012Metric_Pad1.15x1.40mm_HandSolder -> LED_THT:LED_D5.0mm
- renumbered j/1 to J7
Connections:
- net +5V: now also C6.1, U14.2 (SUPPLY)
- net GND: now also C6.2, U14.1 (GND)
- net SCL: now also U14.4 (CLK)
- net SDA: now also U14.3 (SDA/MISO)
- no-connect marks 26 -> 29
Other:
- moved on the sheet: J4, J7, J8, M3, R5, U10

Commit message: lab@home5.3 as ordered at jlcpcb
Parts:
- removed D4: POWER_LED, smopla:3W_LED, symbol Device:LED
- removed M1: HXJ8002_MODULE, smopla:HXJ8002_MODULE_VERTICAL, symbol smopla:HXJ8002_MODULE
- removed Q1: IRLML6344, Package_TO_SOT_SMD:SOT-23_Handsoldering, symbol Transistor_FET:IRLML0030
- removed RV1: 10k, Potentiometer_THT:Potentiometer_Alps_RK09K_Single_Vertical, symbol Device:R_POT
- removed RV2: 10k, Potentiometer_SMD:Potentiometer_Vishay_TS53YL_Vertical, symbol Device:R_POT
- removed U2: 24V->5V, sensact:MODULE_STEPDOWN, symbol sensact:MODULE_STEPDOWN
- removed U5: LD06AJSA, smopla:LD06AJSA, symbol smopla:LD06AJSA
- added C10: 22u, Capacitor_SMD:C_1206_3216Metric_Pad1.33x1.80mm_HandSolder, symbol Device:C
- added C7: 10u, Capacitor_SMD:C_1206_3216Metric_Pad1.33x1.80mm_HandSolder, symbol Device:C
- added C8: 10n, Capacitor_SMD:C_1206_3216Metric_Pad1.33x1.80mm_HandSolder, symbol Device:C
- added C9: 100u, Capacitor_SMD:C_1206_3216Metric_Pad1.33x1.80mm_HandSolder, symbol Device:C
- added D12: 10V, Diode_SMD:D_SMA_Handsoldering, symbol Device:D_Zener
- added D4: 2A, sensact:do214aa_handsolder, symbol Device:D_Schottky
- added L1: 47u, sensact:Inductor_CD104_handsolder, symbol Device:L
- added Q1: BC847, Package_TO_SOT_SMD:SOT-23_Handsoldering, symbol Transistor_BJT:BC847
- added Q6: IRLML5203, Package_TO_SOT_SMD:SOT-23_Handsoldering, symbol Transistor_FET:IRLML5203
- added R25: 1K, Resistor_SMD:R_1206_3216Metric_Pad1.30x1.75mm_HandSolder, symbol Device:R
- added R26: 10k, Resistor_SMD:R_1206_3216Metric_Pad1.30x1.75mm_HandSolder, symbol Device:R
- added R27: 3K3, Resistor_SMD:R_1206_3216Metric_Pad1.30x1.75mm_HandSolder, symbol Device:R
- added U15: CCS811_MODULE, liebler_MODULES:CCS811_MODULE, symbol liebler_MODULES:CCS811_MODULE
- added U16: 24V->5V, sensact:MODULE_STEPDOWN, symbol sensact:MODULE_STEPDOWN
- added U17: DS18B20, Package_TO_SOT_THT:TO-92_Inline, symbol Sensor_Temperature:DS18B20
- added U2: TPS5430DDA, sensact:SOIC-8_3.9x4.9mm_Pitch1.27mm_pad_handsolder, symbol Regulator_Switching:TPS5430DDA
- C4: value u1 -> 10n
- GSM_Module1: symbol sim800l:SIM800L -> labAThome-rescue:SIM800L-sim800l
- J13: value Barrel_Jack_Switch -> Power Input 1
- JP8, JP9: value I2C_SPI -> 1I2C_3SPI
- Q5: value IRLZ44N -> IRF530
- R16: value 10K -> 220R
- R24: value R1 -> 1R
- R8: value 1K -> 22k
- U3: value PDC004_Module -> Power Input 2
- U8: value INMP441_Module -> MIC
Connections:
- net FAN_SWITCH is gone; now on net GND: J9.1 (Pin_1)
- net +24V: now also C5.1, U13.8 (V+), C7.1, U16.3 (IN), U2.7 (VIN)
- net +3V3: now also U15.1 (VCC), U17.3 (VDD)
- net +5V: no longer C5.1, U13.8 (V+)
- net 1wire: now also U17.2 (DQ)
- net FAN_SUPPLY: now also D12.1 (K), Q6.2 (S), R25.1; no longer J9.2 (Pin_2)
- net GND: now also C10.2, C7.2, C9.2, D4.2 (A), R27.1, U15.2 (GND), U15.5 (WAK), U16.2 (GND), U17.1 (GND), U2.6 (GND), U2.9 (GNDPAD)
- net SCL: now also U15.3 (SCL)
- net SDA: now also U15.4 (SDA)
- net at JP1.2: now also C10.1, C9.1, L1.1, R26.2, U16.1 (OUT)
- net at R16.2: now also Q1.2 (E); no longer R15.2
- net FAN_SWITCH2 renamed FAN2_SWITCH
- net SPEAKER renamed I2S_DATA
- new net: Q1.1 (B), R15.2
- new net: D12.2 (A), Q1.3 (C), Q6.1 (G), R25.2
- new net: C8.1, U2.1 (BOOT)
- new net: R26.1, R27.2, U2.4 (VSENSE)
- new net FAN1_SWITCH: J9.2 (Pin_2), Q6.3 (D)
- new net PSU_SW: C8.2, D4.1 (K), L1.2, U2.8 (PH)
- no-connect marks 29 -> 33
Other:
- note added: "LED Constant Current"
- note removed: "Drawings & Mounting"
- moved on the sheet: C1, J1, J11, J13, J2, J6, J9, JP1, JP4, JP8, JP9, Q3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
