File: pcb/analog_amp.sch (KiCad schematic (older format))
At the start: 4 parts, among them J10 SPK, U18 TDA7052A

Commit message: I2S-Amp --> Analog (damn cheap) Amp
Parts:
- removed C13: CP, Capacitor_THT:C_Radial_D8.0mm_H11.5mm_P3.50mm, symbol Device:CP
- removed U18: TDA7052A, Package_DIP:DIP-8_W7.62mm, symbol Amplifier_Audio:TDA7052A
- added C11, C13: u1, Capacitor_SMD:C_1206_3216Metric_Pad1.33x1.80mm_HandSolder, symbol Device:C
- added C12: 1u, Capacitor_SMD:C_1206_3216Metric_Pad1.33x1.80mm_HandSolder, symbol Device:C
- added C14: 10u, Capacitor_SMD:C_1206_3216Metric_Pad1.33x1.80mm_HandSolder, symbol Device:C
- added IC1: MD8002A, sensact:SOIC-8_3.9x4.9mm_Pitch1.27mm_handsolder, symbol liebler_IC:MD8002A
- added JP2: 1=5V,3=3V, Jumper:SolderJumper-3_P1.3mm_Open_RoundedPad1.0x1.5mm_NumberLabels, symbol Jumper:Jumper_3_Open
- added R28: 10k, Resistor_SMD:R_1206_3216Metric_Pad1.30x1.75mm_HandSolder, symbol Device:R
- added R29: 22k, Resistor_SMD:R_1206_3216Metric_Pad1.30x1.75mm_HandSolder, symbol Device:R
- RV1: renamed from RV?; value R_POT -> 5k; footprint (none) -> Potentiometer_THT:Potentiometer_Alps_RK09K_Single_Vertical
Connections:
- net labels added: +3V3
- wire segments 15 -> 16
Other:
- moved on the sheet: J10, RV1

Commit message: Minor PCB update
Parts:
- IC1: symbol liebler_IC:MD8002A -> liebler_SEMICONDUCTORS:MD8002A
Connections:
- net at J10.1 (Pin_1): now also IC1.5 (VO1), R29.1; no longer IC1.8 (VO2)
- new net: IC1.8 (VO2), J10.2 (Pin_2)
Changed lines of the file:
@@
 L Connector_Generic:Conn_01x02 J?
 U 1 1 60B7BC42
-P 5300 3500
+P 5300 3600
 AR Path="/5FDDB245/60B7BC42" Ref="J?"  Part="1"
 AR Path="/60B762EC/60B7BC42" Ref="J10"  Part="1"
-F 0 "J10" H 5380 3492 50  0000 L CNN
-F 1 "SPK" H 5380 3401 50  0000 L CNN
-F 2 "Connector_PinHeader_2.54mm:PinHeader_1x02_P2.54mm_Vertical" H 5300 3500 50  0001 C CNN
-F 3 "~" H 5300 3500 50  0001 C CNN
-	1    5300 3500
-	1    0    0    -1
+F 0 "J10" H 5380 3592 50  0000 L CNN
+F 1 "SPK" H 5380 3501 50  0000 L CNN
+F 2 "Connector_PinHeader_2.54mm:PinHeader_1x02_P2.54mm_Vertical" H 5300 3600 50  0001 C CNN
+F 3 "~" H 5300 3600 50  0001 C CNN
+	1    5300 3600
+	1    0    0    1
 $EndComp
 Text GLabel 2900 4250 1    50   Input ~ 0
@@
 $EndComp
 $Comp
-L liebler_IC:MD8002A IC1
+L liebler_SEMICONDUCTORS:MD8002A IC1
 U 1 1 60B8825A
 P 3700 3500
+AR Path="/60B8825A" Ref="IC1"  Part="1"
+AR Path="/60B762EC/60B8825A" Ref="IC1"  Part="1"
 F 0 "IC1" H 4200 3765 50  0000 C CNN
 F 1 "MD8002A" H 4200 3674 50  0000 C CNN

Commit message: Added option description for PCB
Parts:
- C11, C12, C13, C14, R28, R29, RV1: Option (none) -> Sound only
Changed lines of the file:
@@
 F 2 "Potentiometer_THT:Potentiometer_Alps_RK09K_Single_Vertical" H 2900 4400 50  0001 C CNN
 F 3 "~" H 2900 4400 50  0001 C CNN
+F 4 "Sound only" H 2900 4400 50  0001 C CNN "Option"
 	1    2900 4400
 	1    0    0    -1
@@
 F 2 "Capacitor_SMD:C_1206_3216Metric_Pad1.33x1.80mm_HandSolder" H 5838 3400 50  0001 C CNN
 F 3 "~" H 5800 3550 50  0001 C CNN
+F 4 "Sound only" H 5800 3550 50  0001 C CNN "Option"
 	1    5800 3550
 	1    0    0    -1
@@
 F 2 "Capacitor_SMD:C_1206_3216Metric_Pad1.33x1.80mm_HandSolder" H 3188 3600 50  0001 C CNN
 F 3 "~" H 3150 3750 50  0001 C CNN
+F 4 "Sound only" H 3150 3750 50  0001 C CNN "Option"
 	1    3150 3750
 	1    0    0    -1
@@
 F 2 "Capacitor_SMD:C_1206_3216Metric_Pad1.33x1.80mm_HandSolder" H 3538 4100 50  0001 C CNN
 F 3 "~" H 3500 4250 50  0001 C CNN
+F 4 "Sound only" H 3500 4250 50  0001 C CNN "Option"
 	1    3500 4250
 	1    0    0    -1
@@
 F 2 "Resistor_SMD:R_1206_3216Metric_Pad1.30x1.75mm_HandSolder" V 3430 3950 50  0001 C CNN
 F 3 "~" H 3500 3950 50  0001 C CNN
+F 4 "Sound only" H 3500 3950 50  0001 C CNN "Option"
 	1    3500 3950
 	1    0    0    -1
@@
 F 2 "Resistor_SMD:R_1206_3216Metric_Pad1.30x1.75mm_HandSolder" V 4130 4150 50  0001 C CNN
 F 3 "~" H 4200 4150 50  0001 C CNN
+F 4 "Sound only" V 4200 4150 50  0001 C CNN "Option"
 	1    4200 4150
 	0    1    1    0
@@
 F 2 "Capacitor_SMD:C_1206_3216Metric_Pad1.33x1.80mm_HandSolder" H 6188 3400 50  0001 C CNN
 F 3 "~" H 6150 3550 50  0001 C CNN
+F 4 "Sound only" H 6150 3550 50  0001 C CNN "Option"
 	1    6150 3550
 	1    0    0    -1
