File: pcbV10/pcbV10.sch (KiCad schematic (older format))
At the start: 130 parts, among them J1 PROG, J10 Fan1, J11 Fan2, J12 VPS, J2 Servo, J3 I2C, J4 1wire, J5 EXT, J6 Power, J7 485, J8 POWER, J9 RGB, K1 G6K-2, K2 G6K-2, K3 G6K-2, Q1 BC817, Q2 BC817, Q3 AO3400A, Q4 BC817, Q5 IRLML6344, Q6 BC817, Q7 IRLML5203, Q8 IRF530, Q9 IRLML6344, SW1 BLUE, SW2 YELLOW, SW3 GREEN, SW4 RED, SW5 WHITE, U1 AMS1117-3.3, U10 SR602, U11 LM358, U12 DS18B20, U13 DS18B20, U14 IPS_240_240, U15 DS18B20, U19 BME280, U2 ESP32-WROOM-32, U20 CCS811, U3 CH340K, U4 MS4525DO, U5 INMP441_Module, U6 MAX3485, U7 BME680, U8 IP2721, U9 BH1750_Module, X1 FAN_6024

Commit message: pcb V10 as ordered at JLCPCB
Parts:
- removed C22: 10n, Capacitor_SMD:C_0603_1608Metric, symbol Device:C
- removed D9: 10V, Diode_SMD:D_MiniMELF, symbol Device:D_Zener
- removed JP1: 485_TERM, Connector_PinHeader_2.54mm:PinHeader_1x02_P2.54mm_Vertical, symbol Device:Jumper_NO_Small
- removed JP2: FAN 5V 24V, Connector_PinHeader_2.54mm:PinHeader_1x03_P2.54mm_Vertical, symbol Device:Jumper_NC_Dual
- removed Q6: BC817, Package_TO_SOT_SMD:SOT-23, symbol Transistor_BJT:BC817
- removed Q7: IRLML5203, Package_TO_SOT_SMD:SOT-23, symbol Transistor_FET:IRLML5203
- removed Q8: IRF530, Package_TO_SOT_THT:TO-220-3_Horizontal_TabDown, symbol Device:Q_NMOS_GDS
- removed R27, R28, R29, R32: 1k, Resistor_SMD:R_0603_1608Metric, symbol Device:R
- removed R30: 220R, Resistor_SMD:R_1206_3216Metric, symbol Device:R
- removed R31: k1, Resistor_SMD:R_0603_1608Metric, symbol Device:R
- removed U11: LM358, Package_SO:SO-8_3.9x4.9mm_P1.27mm, symbol Amplifier_Operational:LM358
- removed U5: INMP441_Module, liebler_MODULES:INMP441_Module, symbol smopla:INMP441_Module
- added C31: u1, Capacitor_SMD:C_0603_1608Metric, symbol Device:C
- added D16: Schttky, Diode_SMD:D_SMA, symbol Device:D_Schottky
- added FID1, FID2: Fiducial, Fiducial:Fiducial_1mm_Mask2mm, symbol Mechanical:Fiducial
- added IMG1: Speaker, liebler_DRAWINGS:speaker, symbol Mechanical:Fiducial
- added IMG2: Augenschutz, liebler_DRAWINGS:augenschutz, symbol Mechanical:Fiducial
- added IMG3, IMG7: HOT, liebler_DRAWINGS:hot, symbol Mechanical:Fiducial
- added IMG4: WHS, liebler_DRAWINGS:LOGO_WHS, symbol Mechanical:Fiducial
- added IMG5: QR-CODE, liebler_DRAWINGS:QR_CODE_smopla_de, symbol Mechanical:Fiducial
- added IMG6: OPEN Hardware, Symbol:OSHW-Logo2_7.3x6mm_SilkScreen, symbol Mechanical:Fiducial
- added IMG8: HOT_BIG, liebler_DRAWINGS:hot_big, symbol Mechanical:Fiducial
- added J15: 1B 2A, Connector_Phoenix_MC:PhoenixContact_MCV_1,5_2-G-3.81_1x02_P3.81mm_Vertical, symbol Connector_Generic:Conn_01x02
- added J16: BME280, Connector_PinSocket_2.54mm:PinSocket_1x06_P2.54mm_Vertical, symbol Connector_Generic:Conn_01x06
- added J17: CCS811, Connector_PinSocket_2.54mm:PinSocket_1x08_P2.54mm_Vertical, symbol Connector_Generic:Conn_01x08
- added J18: Barrel_Jack_Switch, Connector_BarrelJack:BarrelJack_Horizontal, symbol Connector:Barrel_Jack_Switch
- added J19: Supply, Connector_PinHeader_2.54mm:PinHeader_2x04_P2.54mm_Vertical, symbol Connector_Generic:Conn_02x04_Odd_Even
- added L1: 47u, Inductor_SMD:L_Abracon_ASPI-0630LR, symbol Device:L
- added MK1: ICS-43434, liebler_SEMICONDUCTORS:MIC_ICS-43434, symbol liebler_SEMICONDUCTORS:ICS-43434
- added R41, R43: M1, Resistor_SMD:R_0603_1608Metric, symbol Device:R
- added R44: 1k, Resistor_SMD:R_0603_1608Metric, symbol Device:R
- added SW10: 5V FAN 24V, liebler_MECH:Switch_SS12D00, symbol Switch:SW_SPDT
- added SW12: RESET, Button_Switch_SMD:SW_Push_1P1T_NO_6x6mm_H9.5mm, symbol Switch:SW_Push
- added SW6: TERM ON, liebler_MECH:Switch_SS12D00, symbol Switch:SW_SPDT
- added SW7: LED HEATER, liebler_MECH:Switch_SS12D00, symbol Switch:SW_SPDT
- added SW8: REL ROT, liebler_MECH:Switch_SS12D00, symbol Switch:SW_SPDT
- added SW9: SNS MOV, liebler_MECH:Switch_SS12D00, symbol Switch:SW_SPDT
- added U21: BTS462T, Package_TO_SOT_SMD:TO-252-5_TabPin3, symbol liebler_SEMICONDUCTORS:BTS462T
- added U5: ZXLD1350, Package_TO_SOT_SMD:SOT-23-5, symbol liebler_SEMICONDUCTORS:ZXLD1350
- C17, C19: footprint Capacitor_SMD:C_0805_2012Metric -> Capacitor_SMD:C_1206_3216Metric
- C2: footprint Capacitor_SMD:C_0805_2012Metric -> Capacitor_SMD:C_0603_1608Metric
- C21: value u1 -> 1u; footprint Capacitor_SMD:C_0603_1608Metric -> Capacitor_SMD:C_1206_3216Metric
- D10, D11, D12, D13, D14: footprint liebler_OPTO:LED_PLCC_2835_Handsoldering -> liebler_OPTO:LED_PLCC_2835
- D6, D7, D8: footprint LED_SMD:LED_PLCC_2835 -> liebler_OPTO:LED_PLCC_2835
- J1, J8: footprint Connector_USB:USB_C_Receptacle_HRO_TYPE-C-31-M-12 -> liebler_CONN:USB_C_Receptacle_HRO_TYPE-C-31-M-12_IMPROVED
- J12: footprint Connector_PinSocket_2.54mm:PinSocket_2x25_P2.54mm_Vertical -> Connector_PinHeader_2.54mm:PinHeader_2x25_P2.54mm_Vertical
- J6: value Power -> 5V 3V GN 24
- J9: value RGB -> GN 5V RGB GN
- R13: value 120R -> K12
- R26: value 22k -> 10k
- R33: value 1R -> R68
- SW1: value BLUE -> BTN BLUE; footprint Button_Switch_SMD:SW_Push_1P1T_NO_CK_PTS125Sx43PSMTR -> liebler_MECH:SW_Push_1P1T_NO_CK_PTS125Sx43PSMTR
- SW3, SW4: footprint Button_Switch_SMD:SW_Push_1P1T_NO_CK_PTS125Sx43PSMTR -> liebler_MECH:SW_Push_1P1T_NO_CK_PTS125Sx43PSMTR
- SW5: value WHITE -> BTN WHITE; footprint Button_Switch_SMD:SW_Push_1P1T_NO_CK_PTS125Sx43PSMTR -> liebler_MECH:SW_Push_1P1T_NO_CK_PTS125Sx43PSMTR
- U6: footprint Package_SO:SO-8_3.9x4.9mm_P1.27mm -> Package_SO:SOIC-8_3.9x4.9mm_P1.27mm
Connections:
- net +24V: now also C21.2, R33.1, D16.1 (K), J18.1, SW10.3 (C), U5.5 (VIN); no longer C21.1, D14.2 (A)
- net +3V3: now also C31.2, J16.1 (Pin_1), J17.1 (Pin_1), J19.1 (Pin_1), J19.2 (Pin_2), MK1.5 (VDD), R44.1
- net +5V: now also J19.5 (Pin_5), J19.6 (Pin_6), J19.7 (Pin_7), J19.8 (Pin_8), SW10.1 (A)
- net 485_DI: no longer J2.1 (Pin_1)
- net FAN1_DRIVE: now also J2.1 (Pin_1), U21.2 (IN)
- net FAN1_SENSE: now also SW9.3 (C); no longer J2.2 (Pin_2), U2.28 (IO17)
- net GND: now also C21.1, C31.1, J16.2 (Pin_2), J17.2 (Pin_2), J17.5 (Pin_5), J18.2, J18.3, J19.3 (Pin_3), J19.4 (Pin_4), MK1.2 (LR), MK1.3 (GND), R43.1, SW12.2, U21.1 (GND), U5.2 (GND); no longer C21.2, R33.2
- net HEATER: now also SW7.1 (A); no longer U2.14 (IO12)
- net K3_A1: now also SW8.1 (A); no longer U2.6 (IO34)
- net LED_WHITE_P: now also SW7.3 (C); no longer U2.16 (IO13)
- net MOVE: now also SW9.1 (A); no longer U2.7 (IO35)
- net PROG_EN: now also SW12.1
- net ROT_B: now also R44.2, SW8.3 (C); no longer U2.29 (IO5)
- net RS485A: now also J15.2 (Pin_2)
- net RS485B: now also J15.1 (Pin_1), SW6.2 (B)
- net SCL: now also J16.3 (Pin_3), J17.3 (Pin_3)
- net SDA: now also J16.4 (Pin_4), J17.4 (Pin_4)
- net VBUS: now also R41.1; no longer U8.11 (SEL)
- net at R26.1: now also U5.3 (ADJ)
- net at D13.1 (K): now also D16.2 (A), L1.1
- net at J10.2 (Pin_2): now also U21.5 (OUT)
- net at J11.2 (Pin_2): now also SW10.2 (B), U21.3 (Vbb)
- net at R13.2: now also SW6.3 (C)
- net SPI_IO1 renamed SERVO2
- net SERVO2: now also J2.2 (Pin_2)
- new net: R41.2, U8.11 (SEL)
- new net: D14.2 (A), R33.2, U5.4 (Isense)
- new net: L1.2, U5.1 (LX)
- new net HEATER_LED: SW7.2 (B), U2.14 (IO12)
- new net I2S_SCK: MK1.4 (SCK), U2.16 (IO13)
- new net I2S_SD: MK1.6 (SD), R43.2, U2.29 (IO5)
- new net I2S_WS: MK1.1 (WS), U2.28 (IO17)
- new net I34: SW8.2 (B), U2.6 (IO34)
- new net I35: SW9.2 (B), U2.7 (IO35)
- no-connect marks 22 -> 28
Other:
- moved on the sheet: C5, D10, D11, D12, D13, D14, D4, D7, D8, J10, J3, J4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

Commit message: labathome v11 as ordered @ JLCPCB
Parts:
- removed C15, C28, C29, C31: u1, Capacitor_SMD:C_0603_1608Metric, symbol Device:C
- removed C30: 1u, Capacitor_SMD:C_0603_1608Metric, symbol Device:C
- removed J16: BME280, Connector_PinSocket_2.54mm:PinSocket_1x06_P2.54mm_Vertical, symbol Connector_Generic:Conn_01x06
- removed J17: CCS811, Connector_PinSocket_2.54mm:PinSocket_1x08_P2.54mm_Vertical, symbol Connector_Generic:Conn_01x08
- removed MK1: ICS-43434, liebler_SEMICONDUCTORS:MIC_ICS-43434, symbol liebler_SEMICONDUCTORS:ICS-43434
- removed R40: 4k7, Resistor_SMD:R_0603_1608Metric, symbol Device:R
- removed R43: M1, Resistor_SMD:R_0603_1608Metric, symbol Device:R
- removed U10: SR602, liebler_MODULES:PIR_Sensor_SR602, symbol smopla:SR602
- removed U12, U13, U15: DS18B20, Package_TO_SOT_THT:TO-92_HandSolder, symbol Sensor_Temperature:DS18B20
- removed U19: BME280, Package_LGA:Bosch_LGA-8_2.5x2.5mm_P0.65mm_ClockwisePinNumbering, symbol Sensor:BME280
- removed U20: CCS811, liebler_SEMICONDUCTORS:AMS_LGA-10-1EP_2.7x4mm_P0.6mm, symbol Sensor_Gas:CCS811
- removed U4: MS4525DO, liebler_MODULES:MS4525DO, symbol smopla:MS4525DO
- removed U7: BME680, Package_LGA:Bosch_LGA-8_3x3mm_P0.8mm_ClockwisePinNumbering, symbol Sensor:BME680
- removed U9: BH1750_Module, liebler_MODULES:GY-302, symbol smopla:GY-302
- added IMG9: Augenschutz, liebler_DRAWINGS:qwiic, symbol Mechanical:Fiducial
- added J20: FAN5V, Connector_JST:JST_XH_B2B-XH-A_1x02_P2.50mm_Vertical, symbol Connector_Generic:Conn_01x02
- added U4: CH340C, Package_SO:SOIC-16_3.9x9.9mm_P1.27mm, symbol Interface_USB:CH340C
- C11, C13: footprint Capacitor_SMD:C_0603_1608Metric -> Capacitor_SMD:C_0805_2012Metric_Pad1.18x1.45mm_HandSolder; Option (none) -> CH340C
- D16: value Schttky -> D
- IMG2: footprint liebler_DRAWINGS:augenschutz -> liebler_DRAWINGS:googles
- J18: value Barrel_Jack_Switch -> Power
- JP3, JP4: value 1I2C_3SPI -> SPI-I2C
- L1: value 47u -> 68u
- R37: value 2k2 -> 2k2?
- U1: value AMS1117-3.3 -> AMS1117
Connections:
- net +3V3: no longer C11.2, C13.2
- net +5V: now also C13.1, J20.1 (Pin_1), U4.16 (VCC)
- net DTR: now also U4.13 (~DTR)
- net GND: now also C13.2, U4.1 (GND); no longer C13.1
- net I2S_SCK: now also U2.29 (IO5); no longer U2.16 (IO13)
- net I2S_SD: now also U2.28 (IO17); no longer U2.29 (IO5)
- net I2S_WS: now also U2.16 (IO13); no longer U2.28 (IO17)
- net PROG_RX: now also U4.3 (RXD)
- net PROG_TX: now also U4.2 (TXD)
- net RTS: now also U4.14 (~RTS)
- net UD+: now reaches J1.A6 (D+), J1.B6 (D+), U3.1 (UD+)
- net UD+: now also U4.5 (UD+)
- net UD-: now reaches J1.A7 (D-), J1.B7 (D-), U3.2 (UD-)
- net UD-: now also U4.6 (UD-)
- net D13_COOL: now reaches D13.1 (K), D16.2 (A), L1.1
- net D11_COOL: now reaches D11.1 (K), D13.2 (A)
- net D10_COOL: now reaches D10.1 (K), D11.2 (A)
- net D12_COOL: now reaches D10.2 (A), D12.1 (K)
- net D14_COOL: now reaches D12.2 (A), D14.1 (K)
- net at J11.1 (Pin_1), Q9.3 (D): now also J20.2 (Pin_2)
- new net: C11.2, U4.4 (V3)
- no-connect marks 28 -> 24
Other:
- note added: "Images"
- note removed: "1wire Temperature Sensors"
- note removed: "7bit-ADDR=0x76"
- note removed: "CSB=3V -> I2C"
- note removed: "Sensors"
- moved on the sheet: C14, C16, C18, C7, D1, D15, D2, D3, FID1, FID2, IMG1, IMG2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
