File: pcbV10/pcbV10.kicad_pcb (KiCad board)
At the start: 2 copper layers, 100 x 100 mm, 215 parts, among them J1 PROG, J10 Fan1, J11 Fan2, J12 VPS, J13 SPK, J14 LoRa Antenna, J15 1B 2A, J16 BME280, J17 CCS811, J18 Power, J19 Supply, J2 Srvo, J20 FAN5V, J21 QWIIC, J22 AudioJack3_SwitchT, J23 USB_PD, J24 AOUT, J3 I2C, J4 1wire, J5 EXT, J6 5V 3V GN 24, J7 485, J8 POWER, J9 GN 5V RGB GN, K1 G6K-2, K2 G6K-2, K3 G6K-2, Q1 BC817, Q2 BC817, Q4 BC817, Q5 IRLML6344, Q6 BC817, Q7 TIP41, Q9 IRLML6344, SW1 BTN BLUE, SW10 5V FAN 24V, SW11 PROG 5V POWER, SW12 RESET, SW2 YELLOW, SW3 GREEN, SW4 RED, SW5 BTN WHITE, SW6 TERM ON, SW7 LED HTR, SW8 REL ROT, SW9 SNS MOV, U1 AMS1117, U10 LM358, U11 FUSB302BMPX, U12 BME680, U13 BME280, U14 IPS_240_240, U15 CCS811, U16 MODULE_STEPDOWN, U17 RFM95W-868S2, U18 MD8002A, U19 DS18B20, U2 ESP32-WROOM-32, U20 BH1750, U21 BTS462T, U22 AM612, U23 MPU-6050, U24 SRV05, U3 ICS-43432, U4 CH340C, U5 UDA1334, U6 MAX3485, U7 DS18B20, U8 HDC1080, U9 EUP3458, X1 FAN_6024, X2 XGZP6897D

Commit message: PCBs as ordered at JLCPCB with assembly
Parts:
- RV1: value 1k -> 10k
- moved IMG4 99.8 mm to (32.4, 127.5)
- moved IMG7 11.0 mm to (134.7, 64.8)
- moved R49 1.10 mm to (104.9, 97.5)
- moved C57 0.95 mm to (60.6, 102.6)
- moved JP7 0.70 mm to (90.2, 91.9)
- moved C19 0.54 mm to (62.4, 111.3)
- moved R6 0.36 mm to (66.3, 129.2)
- moved Q2 0.26 mm to (63.1, 128.6)
- moved R7 0.22 mm to (66.3, 127.5)
- moved Q1 0.10 mm to (69.5, 128.5)
Connections:
- C19 pad 2: /psu/5Vx -> +3V3
- U11 pad 3: /psu/5Vx -> +3V3
- U11 pad 4: /psu/5Vx -> +3V3
Routing:
- net +3V3: track 538.1 -> 548.3 mm
- net GND: track 162.8 -> 167.3 mm, vias 217 -> 228
- net /psu/5Vx: track 41.1 -> 36.8 mm, vias 2 -> 1
- net RS485A: track 53.4 -> 49.4 mm, vias 1 -> 2
- net Net-(JP2-Pad2): track 31.1 -> 28.1 mm
- net 485_DE: track 34.1 -> 36.8 mm
- net 485_RO: track 35.5 -> 38.1 mm
- net Net-(J12-Pad29): track 50.3 -> 52.7 mm
- net PROG_TX: track 19.5 -> 21.4 mm
- net Net-(JP1-Pad2): track 2.98 -> 4.83 mm
- net +5V: track 373.4 -> 371.8 mm
- net AUDIO: track 90.9 -> 92.3 mm
- net Net-(D15-Pad2): track 8.57 -> 7.31 mm
- net SCL: track 218.5 -> 219.7 mm
- net Net-(Q2-Pad1): track 1.30 -> 2.41 mm
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Other:
- board text added: "2022-03-11 Klaus Liebler"
- board text removed: "2022-02-25 Klaus Liebler"
