File: pcbV10/pcbV10.kicad_pcb (KiCad board)
At the start: 2 copper layers, 100 x 100 mm, 215 parts, among them J1 PROG, J10 Fan1, J11 Fan2, J12 VPS, J13 SPK, J14 LoRa Antenna, J15 1B 2A, J16 BME280, J17 CCS811, J18 Power, J19 Supply, J2 Srvo, J20 FAN5V, J21 QWIIC, J22 AudioJack3_SwitchT, J23 USB_PD, J24 AOUT, J3 I2C, J4 1wire, J5 EXT, J6 5V 3V GN 24, J7 485, J8 POWER, J9 GN 5V RGB GN, K1 G6K-2, K2 G6K-2, K3 G6K-2, Q1 BC817, Q2 BC817, Q4 BC817, Q5 IRLML6344, Q6 BC817, Q7 TIP41, Q9 IRLML6344, SW1 BTN BLUE, SW10 5V FAN 24V, SW11 PROG 5V POWER, SW12 RESET, SW2 YELLOW, SW3 GREEN, SW4 RED, SW5 BTN WHITE, SW6 TERM ON, SW7 LED HTR, SW8 REL ROT, SW9 SNS MOV, U1 AMS1117, U10 LM358, U11 FUSB302BMPX, U12 BME680, U13 BME280, U14 IPS_240_240, U15 CCS811, U16 MODULE_STEPDOWN, U17 RFM95W-868S2, U18 MD8002A, U19 DS18B20, U2 ESP32-WROOM-32, U20 BH1750, U21 BTS462T, U22 AM612, U23 MPU-6050, U24 SRV05, U3 ICS-43432, U4 CH340C, U5 UDA1334, U6 MAX3485, U7 DS18B20, U8 HDC1080, U9 EUP3458, X1 FAN_6024, X2 XGZP6897D

Commit message: Minor fixes in PCB
Parts:
- removed J23: USB_PD, Connector_PinHeader_2.54mm:PinHeader_1x04_P2.54mm_Vertical
- added R9: GL5516, OptoDevice:R_LDR_5.1x4.3mm_P3.4mm_Vertical, F.Cu at (136.0, 78.5)
- J9: value GN 5V RGB GN -> GN RGB 5V GN
- SW6: value TERM ON -> TERM ON
- moved C5 11.4 mm to (80.6, 131.2), turned to 90 degrees
- moved R3 1.01 mm to (59.4, 128.8)
- moved C9 0.90 mm to (80.6, 128.2)
- moved K1 0.12 mm to (135.9, 86.1)
Connections:
- J12 pad 45: LED_BLUE -> SW_WHITE
- J12 pad 46: LED_BLUE -> SW_WHITE
- J12 pad 47: SW_WHITE -> LED_BLUE
- J12 pad 48: SW_WHITE -> LED_BLUE
Routing:
- net ROT_A: track 10.6 -> 76.4 mm
- net +24V: track 219.7 -> 215.3 mm
- net GND: track 167.3 -> 163.7 mm
- net LED_BLUE: track 14.2 -> 11.7 mm
- net SW_WHITE: track 22.4 -> 23.1 mm
Other:
- board text added: "2022-03-29 Klaus Liebler"
- board text added: "3V3 GND 5V0 5V0"
- board text added: "Testen mit ES8374"
- board text removed: "2022-03-11 Klaus Liebler"

Commit message: Sicherung
Other:
- board text added: "24V GND 3V3 5V0"
- board text added: "SRV1 5V GND"
- board text removed: "24 GN 3V 5V"
- board text removed: "S1 5 G"
Changed lines of the file:
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@@
     (property "Sheetname" "wireless")
     (attr smd exclude_from_pos_files)
-    (fp_text reference "DWM1" (at -5.08 -13.97) (layer "B.SilkS")
+    (fp_text reference "DWM1" (at 0 -13.7) (layer "B.SilkS")
       (effects (font (size 1 1) (thickness 0.15)) (justify mirror))
     )
@@
   (gr_line (start 70 53) (end 53 53) (layer "Edge.Cuts") (width 0.05))
   (gr_line (start 150 70) (end 150 130) (layer "Edge.Cuts") (width 0.05))
-  (gr_text "S1 5 G" (at 63.8 89.9) (layer "B.SilkS")
+  (gr_text "SRV1 5V GND" (at 57.9 88.1) (layer "B.SilkS")
     (effects (font (size 1.5 1) (thickness 0.2)) (justify mirror))
   )
@@
     (effects (font (size 1.5 1) (thickness 0.2)) (justify mirror))
   )
-  (gr_text "24\nGN\n3V\n5V" (at 54.864 112.268) (layer "B.SilkS")
-    (effects (font (size 1.5 1) (thickness 0.2)) (justify mirror))
+  (gr_text "24V\nGND\n3V3\n5V0" (at 55.8 111.7) (layer "B.SilkS")
+    (effects (font (size 1.5 1) (thickness 0.2)) (justify left mirror))
   )
   (gr_text "SDA\nSCL\nGND\n3V3\n5V0" (at 54.4 139) (layer "B.SilkS")
@@
     (effects (font (size 1.5 1) (thickness 0.2)) (justify mirror))
   )
-  (gr_text "GND\n+F1\nSEN" (at 56.007 74.93) (layer "B.SilkS")
-    (effects (font (size 1.5 1.5) (thickness 0.3)) (justify left mirror))
+  (gr_text "GND\n+F1\nSEN" (at 55.8 74.6) (layer "B.SilkS")
+    (effects (font (size 1.5 1) (thickness 0.2)) (justify left mirror))
   )
   (gr_text "F2\n5V\n" (at 61.214 82.423) (layer "B.SilkS")
-    (effects (font (size 1.5 1.5) (thickness 0.3)) (justify left mirror))
+    (effects (font (size 1.5 1) (thickness 0.2)) (justify left mirror))
   )
   (gr_text "SW_BLUE\nLED_BLUE\nSW_WHITE\nLED_WHITE" (at 138.938 134.366) (layer "B.SilkS")
@@
     (effects (font (size 1.5 1) (thickness 0.2)) (justify mirror))
   )
-  (gr_text "Micro" (at 82 105.3) (layer "B.SilkS")
+  (gr_text "Micro" (at 81.8 105.1) (layer "B.SilkS")
     (effects (font (size 1.5 1.5) (thickness 0.3)) (justify right mirror))
   )
@@
     (effects (font (size 1.5 1) (thickness 0.2)) (justify left mirror))
   )
-  (gr_text "S2 5 G" (at 63.8 92.583) (layer "B.SilkS")
-    (effects (font (size 1.5 1) (thickness 0.2)) (justify mirror))
-  )
-  (gr_text " GND\n5V\nDATA\nGND" (at 66 64.9) (layer "B.SilkS")
-    (effects (font (size 1.5 1.5) (thickness 0.3)) (justify left mirror))
+  (gr_text "S2 5 G" (at 63.9 92.583) (layer "B.SilkS")
+    (effects (font (size 1.5 1) (thickness 0.2)) (justify mirror))
+  )
+  (gr_text "GND\n5V\nDATA\nGND" (at 64.5 64.9) (layer "B.SilkS")
+    (effects (font (size 1.5 1) (thickness 0.2)) (justify left mirror))
   )
   (gr_text "TERM: for RS485-Termination\nLED HEATER: power LED or heating-R@ io12\n\nREL ROT: K3-A1 or rotary encoder @ io34\nSNS MOV: fan1- or movem.-sensor @ io35\n24V->5V: activate 24V-to-5V converter\n5V FAN 24V: select 24V or 5V for both fans" (at 41.5 94.4) (layer "B.SilkS")

Commit message: Various
Other:
- board text added: "Alle Jumper in der Mini-Ausführung statt lötbare Module lieber diesen miniPCIE-Connector Die 5V/3V/GND direkt mit dem Relais_Connector koppeln Modbus nicht mehr über RJ11"
Changed lines of the file:
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@@
     (effects (font (size 1 1) (thickness 0.15)))
+  )
+  (gr_text "Alle Jumper in der Mini-Ausführung\nstatt lötbare Module lieber diesen miniPCIE-Connector\nDie 5V/3V/GND direkt mit dem Relais_Connector koppeln\nModbus nicht mehr über RJ11" (at 184.2 99.3) (layer "F.SilkS")
+    (effects (font (size 1.5 1.5) (thickness 0.3)))
   )
   (gr_text "A1 11 12 14 21 22 24" (at 147.32 84.836 270) (layer "F.SilkS")
