File: pcbV10/psu.kicad_sch (KiCad schematic)
At the start: 22 parts, among them J23 USB_PD, J8 POWER, SW11 PROG 5V POWER, U11 FUSB302BMPX, U24 SRV05, U9 EUP3458

Commit message: PCBs as ordered at JLCPCB with assembly
Connections:
- net 5Vx: no longer C19.2, U11.3 (VDD), U11.4 (VDD)
- new net +3V3: C19.2, U11.3 (VDD), U11.4 (VDD)
Changed lines of the file:
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@@
   (junction (at 82.55 95.25) (diameter 0) (color 0 0 0 0)
   )
-  (junction (at 64.77 106.68) (diameter 0) (color 0 0 0 0)
-  )
   (junction (at 83.82 95.25) (diameter 0) (color 0 0 0 0)
   )
@@
   (junction (at 80.01 90.17) (diameter 0) (color 0 0 0 0)
   )
+  (junction (at 97.79 64.77) (diameter 0) (color 0 0 0 0)
+  )
   (junction (at 77.47 90.17) (diameter 0) (color 0 0 0 0)
   )
-  (junction (at 97.79 57.15) (diameter 0) (color 0 0 0 0)
-  )
   (junction (at 59.69 95.25) (diameter 0) (color 0 0 0 0)
   )
@@
   )
   (junction (at 125.73 58.42) (diameter 0) (color 0 0 0 0)
-  )
-  (junction (at 62.23 106.68) (diameter 0) (color 0 0 0 0)
-  )
-  (junction (at 97.79 64.77) (diameter 0) (color 0 0 0 0)
   )
   (junction (at 134.62 58.42) (diameter 0) (color 0 0 0 0)
@@
     (stroke (width 0) (type default) (color 0 0 0 0))
   )
+  (wire (pts (xy 64.77 106.68) (xy 67.31 106.68))
+    (stroke (width 0) (type default) (color 0 0 0 0))
+  )
   (wire (pts (xy 160.02 57.15) (xy 160.02 58.42))
     (stroke (width 0) (type default) (color 0 0 0 0))
@@
     (stroke (width 0) (type default) (color 0 0 0 0))
   )
-  (wire (pts (xy 97.79 64.77) (xy 106.68 64.77))
-    (stroke (width 0) (type default) (color 0 0 0 0))
-  )
   (wire (pts (xy 119.38 66.04) (xy 119.38 88.9))
     (stroke (width 0) (type default) (color 0 0 0 0))
@@
     (stroke (width 0) (type default) (color 0 0 0 0))
   )
-  (wire (pts (xy 64.77 106.68) (xy 67.31 106.68))
-    (stroke (width 0) (type default) (color 0 0 0 0))
-  )
   (wire (pts (xy 125.73 88.9) (xy 147.32 88.9))
     (stroke (width 0) (type default) (color 0 0 0 0))
@@
   )
   (wire (pts (xy 74.93 57.15) (xy 77.47 57.15))
-    (stroke (width 0) (type default) (color 0 0 0 0))
-  )
-  (wire (pts (xy 97.79 57.15) (xy 106.68 57.15))
-    (stroke (width 0) (type default) (color 0 0 0 0))
-  )
-  (wire (pts (xy 62.23 106.68) (xy 64.77 106.68))
     (stroke (width 0) (type default) (color 0 0 0 0))
   )
@@
     (effects (font (size 1.27 1.27)) (justify left bottom))
   )
+  (label "5Vx" (at 67.31 106.68 0)
+    (effects (font (size 1.27 1.27)) (justify left bottom))
+  )
   (label "SW" (at 161.29 63.5 0)
-    (effects (font (size 1.27 1.27)) (justify left bottom))
-  )
-  (label "5Vx" (at 40.64 100.33 0)
     (effects (font (size 1.27 1.27)) (justify left bottom))
   )
@@
     )
     (property "Datasheet" "~" (id 3) (at 220.98 58.42 0)
+      (effects (font (size 1.27 1.27)) hide)
+    )
+    (pin "1")
+  )
+  (symbol (lib_id "power:+3V3") (at 40.64 100.33 0) (unit 1)
+    (in_bom yes) (on_board yes) (fields_autoplaced)
+    (property "Reference" "#PWR0114" (id 0) (at 40.64 104.14 0)
+      (effects (font (size 1.27 1.27)) hide)
+    )
+    (property "Value" "+3V3" (id 1) (at 40.64 95.25 0))
+    (property "Footprint" "" (id 2) (at 40.64 100.33 0)
+      (effects (font (size 1.27 1.27)) hide)
+    )
+    (property "Datasheet" "" (id 3) (at 40.64 100.33 0)
       (effects (font (size 1.27 1.27)) hide)
     )
@@
     (pin "1")
   )
-  (symbol (lib_id "power:GND") (at 106.68 64.77 0) (unit 1)
-    (in_bom yes) (on_board yes)
-    (property "Reference" "#PWR0115" (id 0) (at 106.68 71.12 0)
-      (effects (font (size 1.27 1.27)) hide)
-    )
-    (property "Value" "GND" (id 1) (at 106.68 69.85 90))
-    (property "Footprint" "" (id 2) (at 106.68 64.77 0)
-      (effects (font (size 1.27 1.27)) hide)
-    )
-    (property "Datasheet" "" (id 3) (at 106.68 64.77 0)
-      (effects (font (size 1.27 1.27)) hide)
-    )
+  (symbol (lib_id "power:GND") (at 97.79 64.77 0) (unit 1)
+    (in_bom yes) (on_board yes)
+    (property "Reference" "#PWR0115" (id 0) (at 97.79 71.12 0)
+      (effects (font (size 1.27 1.27)) hide)
+    )
+    (property "Value" "GND" (id 1) (at 97.79 69.85 90))
+    (property "Footprint" "" (id 2) (at 97.79 64.77 0)
+      (effects (font (size 1.27 1.27)) hide)
+    )
+    (property "Datasheet" "" (id 3) (at 97.79 64.77 0)
+      (effects (font (size 1.27 1.27)) hide)
+    )

Commit message: Minor fixes in PCB
Parts:
- removed J23: USB_PD, Connector_PinHeader_2.54mm:PinHeader_1x04_P2.54mm_Vertical, symbol Connector_Generic:Conn_01x04
Changed lines of the file:
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@@
   (junction (at 167.64 88.9) (diameter 0) (color 0 0 0 0)
   )
-  (junction (at 140.97 114.3) (diameter 0) (color 0 0 0 0)
-  )
   (junction (at 167.64 60.96) (diameter 0) (color 0 0 0 0)
   )
@@
   )
   (junction (at 220.98 58.42) (diameter 0) (color 0 0 0 0)
-  )
-  (junction (at 140.97 121.92) (diameter 0) (color 0 0 0 0)
   )
   (junction (at 82.55 95.25) (diameter 0) (color 0 0 0 0)
@@
     (stroke (width 0) (type default) (color 0 0 0 0))
   )
-  (wire (pts (xy 140.97 114.3) (xy 140.97 116.84))
-    (stroke (width 0) (type default) (color 0 0 0 0))
-  )
   (wire (pts (xy 82.55 116.84) (xy 77.47 116.84))
     (stroke (width 0) (type default) (color 0 0 0 0))
@@
   )
   (wire (pts (xy 74.93 57.15) (xy 77.47 57.15))
-    (stroke (width 0) (type default) (color 0 0 0 0))
-  )
-  (wire (pts (xy 140.97 119.38) (xy 140.97 121.92))
     (stroke (width 0) (type default) (color 0 0 0 0))
   )
@@
     )
     (pin "1")
-  )
-  (symbol (lib_id "Connector_Generic:Conn_01x04") (at 135.89 116.84 0) (mirror y) (unit 1)
-    (in_bom yes) (on_board yes) (fields_autoplaced)
-    (property "Reference" "J23" (id 0) (at 135.89 107.95 0))
-    (property "Value" "USB_PD" (id 1) (at 135.89 110.49 0))
-    (property "Footprint" "Connector_PinHeader_2.54mm:PinHeader_1x04_P2.54mm_Vertical" (id 2) (at 135.89 116.84 0)
-      (effects (font (size 1.27 1.27)) hide)
-    )
-    (property "Datasheet" "~" (id 3) (at 135.89 116.84 0)
-      (effects (font (size 1.27 1.27)) hide)
-    )
-    (pin "1")
-    (pin "2")
-    (pin "3")
-    (pin "4")
   )
   (symbol (lib_id "power:PWR_FLAG") (at 74.93 57.15 0) (unit 1)
@@
       (effects (font (size 1.27 1.27)) hide)
     )
-    (pin "1")
-  )
-  (symbol (lib_id "power:+24V") (at 140.97 114.3 270) (unit 1)
-    (in_bom yes) (on_board yes)
-    (property "Reference" "#PWR070" (id 0) (at 137.16 114.3 0)
-      (effects (font (size 1.27 1.27)) hide)
-    )
-    (property "Value" "+24V" (id 1) (at 144.2212 114.681 90)
-      (effects (font (size 1.27 1.27)) (justify left))
-    )
-    (property "Footprint" "" (id 2) (at 140.97 114.3 0)
-      (effects (font (size 1.27 1.27)) hide)
-    )
-    (property "Datasheet" "" (id 3) (at 140.97 114.3 0)
-      (effects (font (size 1.27 1.27)) hide)
-    )
-    (pin "1")
-  )
-  (symbol (lib_id "power:GND") (at 140.97 121.92 0) (unit 1)
-    (in_bom yes) (on_board yes)
-    (property "Reference" "#PWR071" (id 0) (at 140.97 128.27 0)
-      (effects (font (size 1.27 1.27)) hide)
-    )
-    (property "Value" "GND" (id 1) (at 141.097 126.3142 0))
-    (property "Footprint" "" (id 2) (at 140.97 121.92 0)
-      (effects (font (size 1.27 1.27)) hide)
-    )
-    (property "Datasheet" "" (id 3) (at 140.97 121.92 0)
-      (effects (font (size 1.27 1.27)) hide)
-    )

Commit message: Various
Parts:
- removed D16: SS34, Diode_SMD:D_SMA, symbol Device:D_Schottky
- added C60: 10u, Capacitor_SMD:C_1206_3216Metric, symbol Device:C
- C35: value 10n -> u1
- L2: value 6u8 -> 4u7
- U9: value EUP3458 -> RY8310
Connections:
- net +24V: now also C60.2
- net GND: now also C60.1
Changed lines of the file:
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@@
 (kicad_sch (version 20211123) (generator eeschema)
   (paper "A4")
-  (junction (at 167.64 88.9) (diameter 0) (color 0 0 0 0)
-  )
   (junction (at 167.64 60.96) (diameter 0) (color 0 0 0 0)
   )
@@
   (junction (at 80.01 90.17) (diameter 0) (color 0 0 0 0)
   )
+  (junction (at 119.38 88.9) (diameter 0) (color 0 0 0 0)
+  )
   (junction (at 97.79 64.77) (diameter 0) (color 0 0 0 0)
   )
@@
   )
   (junction (at 90.17 119.38) (diameter 0) (color 0 0 0 0)
-  )
-  (junction (at 167.64 63.5) (diameter 0) (color 0 0 0 0)
   )
   (junction (at 74.93 57.15) (diameter 0) (color 0 0 0 0)
@@
     (stroke (width 0) (type default) (color 0 0 0 0))
   )
-  (wire (pts (xy 167.64 71.12) (xy 167.64 88.9))
-    (stroke (width 0) (type default) (color 0 0 0 0))
-  )
   (wire (pts (xy 62.23 100.33) (xy 62.23 106.68))
     (stroke (width 0) (type default) (color 0 0 0 0))
@@
     (stroke (width 0) (type default) (color 0 0 0 0))
   )
+  (wire (pts (xy 114.3 88.9) (xy 119.38 88.9))
+    (stroke (width 0) (type default) (color 0 0 0 0))
+  )
   (wire (pts (xy 80.01 90.17) (xy 80.01 119.38))
     (stroke (width 0) (type default) (color 0 0 0 0))
@@
     (stroke (width 0) (type default) (color 0 0 0 0))
   )
+  (wire (pts (xy 114.3 58.42) (xy 119.38 58.42))
+    (stroke (width 0) (type default) (color 0 0 0 0))
+  )
   (wire (pts (xy 201.93 60.96) (xy 210.82 60.96))
     (stroke (width 0) (type default) (color 0 0 0 0))
@@
     (stroke (width 0) (type default) (color 0 0 0 0))
   )
+  (wire (pts (xy 114.3 66.04) (xy 114.3 88.9))
+    (stroke (width 0) (type default) (color 0 0 0 0))
+  )
   (wire (pts (xy 77.47 90.17) (xy 77.47 114.3))
     (stroke (width 0) (type default) (color 0 0 0 0))
@@
     (stroke (width 0) (type default) (color 0 0 0 0))
   )
-  (wire (pts (xy 151.13 88.9) (xy 167.64 88.9))
-    (stroke (width 0) (type default) (color 0 0 0 0))
-  )
   (wire (pts (xy 160.02 49.53) (xy 167.64 49.53))
     (stroke (width 0) (type default) (color 0 0 0 0))
@@
     (stroke (width 0) (type default) (color 0 0 0 0))
   )
-  (wire (pts (xy 167.64 88.9) (xy 177.8 88.9))
+  (wire (pts (xy 151.13 88.9) (xy 177.8 88.9))
     (stroke (width 0) (type default) (color 0 0 0 0))
   )
@@
     (in_bom yes) (on_board yes)
     (property "Reference" "C35" (id 0) (at 161.29 50.8 0))
-    (property "Value" "10n" (id 1) (at 162.56 55.88 0))
+    (property "Value" "u1" (id 1) (at 162.56 55.88 0))
     (property "Footprint" "Capacitor_SMD:C_0603_1608Metric" (id 2) (at 159.0548 49.53 0)
       (effects (font (size 1.27 1.27)) hide)
@@
     (in_bom yes) (on_board yes)
     (property "Reference" "L2" (id 0) (at 172.72 56.3626 90))
-    (property "Value" "6u8" (id 1) (at 172.72 58.674 90))
+    (property "Value" "4u7" (id 1) (at 172.72 58.674 90))
     (property "Footprint" "Inductor_SMD:L_Abracon_ASPI-0630LR" (id 2) (at 172.72 60.96 0)
       (effects (font (size 1.27 1.27)) hide)
@@
     )
     (pin "1")
-  )
-  (symbol (lib_id "Device:D_Schottky") (at 167.64 67.31 270) (unit 1)
-    (in_bom yes) (on_board yes) (fields_autoplaced)
-    (property "Reference" "D16" (id 0) (at 170.18 65.7224 90)
-      (effects (font (size 1.27 1.27)) (justify left))
-    )
-    (property "Value" "SS34" (id 1) (at 170.18 68.2624 90)
-      (effects (font (size 1.27 1.27)) (justify left))
-    )
-    (property "Footprint" "Diode_SMD:D_SMA" (id 2) (at 167.64 67.31 0)
-      (effects (font (size 1.27 1.27)) hide)
-    )
-    (property "Datasheet" "~" (id 3) (at 167.64 67.31 0)
-      (effects (font (size 1.27 1.27)) hide)
-    )
-    (pin "1")
-    (pin "2")
   )
   (symbol (lib_id "power:GND") (at 96.52 105.41 0) (unit 1)
@@
     (in_bom yes) (on_board yes) (fields_autoplaced)
     (property "Reference" "U9" (id 0) (at 147.32 50.8 0))
-    (property "Value" "EUP3458" (id 1) (at 147.32 53.34 0))
+    (property "Value" "RY8310" (id 1) (at 147.32 53.34 0))
     (property "Footprint" "Package_TO_SOT_SMD:SOT-23-6" (id 2) (at 147.32 76.2 0)
       (effects (font (size 1.27 1.27) italic) hide)
@@
     (pin "6")
   )
+  (symbol (lib_id "Device:C") (at 114.3 62.23 180) (unit 1)
+    (in_bom yes) (on_board yes)
+    (property "Reference" "C60" (id 0) (at 116.84 59.69 0))
+    (property "Value" "10u" (id 1) (at 116.84 64.77 0))
+    (property "Footprint" "Capacitor_SMD:C_1206_3216Metric" (id 2) (at 113.3348 58.42 0)
+      (effects (font (size 1.27 1.27)) hide)
+    )
+    (property "Datasheet" "~" (id 3) (at 114.3 62.23 0)
+      (effects (font (size 1.27 1.27)) hide)
+    )
+    (pin "1")
+    (pin "2")
+  )
   (symbol (lib_id "power:GND") (at 40.64 107.95 0) (unit 1)
