File: pcbV10/analog_amp.kicad_sch (KiCad schematic)
At the start: 35 parts, among them J13 SPK, J22 AudioJack3_SwitchT, J24 AOUT, U10 LM358, U18 MD8002A, U5 UDA1334

Commit message: Various
Parts:
- added C21: 1u, Capacitor_SMD:C_0805_2012Metric_Pad1.18x1.45mm_HandSolder, symbol Device:C
- added C34: 100u, Capacitor_SMD:C_1206_3216Metric_Pad1.33x1.80mm_HandSolder, symbol Device:C
- added FB1: 100R, Inductor_SMD:L_0805_2012Metric, symbol Device:FerriteBead
- added J19: SPK, Connector_Wire:SolderWire-0.1sqmm_1x02_P3.6mm_D0.4mm_OD1mm, symbol Connector_Generic:Conn_01x02
- added JP5: 5V AMP 3V, Jumper:SolderJumper-3_P1.3mm_Open_RoundedPad1.0x1.5mm_NumberLabels, symbol Jumper:SolderJumper_3_Open
- added NT1, NT2: 1, NetTie:NetTie-2_SMD_Pad0.5mm, symbol Device:NetTie_2
- added U25: NS4168, liebler_SEMICONDUCTORS:SOIC-8_3.9x4.9mm_Pitch1.27mm_pad_handsolder, symbol liebler_SEMICONDUCTORS:NS4168
Connections:
- net +3V3: now also JP5.3 (B)
- net +5V: now also JP5.1 (A), NT1.2; no longer C25.1, C26.1, U18.6 (VDD)
- net AUDIO: now also U25.4 (SDATA)
- net GND: now also C21.2, C34.2, NT2.1, U25.1 (CTRL), U25.7 (GND); no longer C23.2, C25.2, C26.2, U18.1 (SD), U18.7 (GND)
- net I2S_SCK: now also U25.3 (BCLK)
- net I2S_WS: now also U25.2 (LRCLK)
- net SPK+: now reaches J13.1 (Pin_1), R39.1, U18.5 (VO1)
- net SPK-: now reaches J13.2 (Pin_2), U18.8 (VO2)
- new net: C21.1, C34.1, FB1.2, U25.6 (VDD)
- new net: FB1.1, JP5.2 (C)
- new net +5VA: C25.1, C26.1, NT1.1, U18.6 (VDD)
- new net GNDA: C23.2, C25.2, C26.2, NT2.2, U18.1 (SD), U18.7 (GND)
- new net VoN: J19.2 (Pin_2), U25.5 (VoN)
- new net VoP: J19.1 (Pin_1), U25.8 (VoP)

Commit message: Bugfix: digital amplifier not in standby
Connections:
- net GND: no longer U25.1 (CTRL)
- net at C21.1, C34.1, FB1.2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: now also U25.1 (CTRL)
Changed lines of the file:
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@@
   (junction (at 198.12 80.01) (diameter 0) (color 0 0 0 0)
+  )
+  (junction (at 135.255 170.815) (diameter 0) (color 0 0 0 0)
   )
   (junction (at 93.98 189.23) (diameter 0) (color 0 0 0 0)
@@
     (stroke (width 0) (type default) (color 0 0 0 0))
   )
+  (wire (pts (xy 105.41 159.385) (xy 115.57 159.385))
+    (stroke (width 0) (type default) (color 0 0 0 0))
+  )
+  (wire (pts (xy 135.255 170.815) (xy 105.41 170.815))
+    (stroke (width 0) (type default) (color 0 0 0 0))
+  )
   (wire (pts (xy 246.38 101.6) (xy 236.22 101.6))
     (stroke (width 0) (type default) (color 0 0 0 0))
@@
   )
   (wire (pts (xy 214.63 97.79) (xy 215.9 97.79))
+    (stroke (width 0) (type default) (color 0 0 0 0))
+  )
+  (wire (pts (xy 105.41 170.815) (xy 105.41 159.385))
     (stroke (width 0) (type default) (color 0 0 0 0))
   )
@@
     (pin "2")
   )
-  (symbol (lib_id "power:GND") (at 115.57 159.385 270) (unit 1)
-    (in_bom yes) (on_board yes)
-    (property "Reference" "#PWR0201" (id 0) (at 109.22 159.385 0)
-      (effects (font (size 1.27 1.27)) hide)
-    )
-    (property "Value" "GND" (id 1) (at 108.585 159.385 90)
-      (effects (font (size 1.27 1.27)) (justify left))
-    )
-    (property "Footprint" "" (id 2) (at 115.57 159.385 0)
-      (effects (font (size 1.27 1.27)) hide)
-    )
-    (property "Datasheet" "" (id 3) (at 115.57 159.385 0)
-      (effects (font (size 1.27 1.27)) hide)
-    )
-    (pin "1")
-  )
   (symbol (lib_id "power:GND") (at 50.8 143.51 0) (unit 1)
