File: pcbV10/pcbV10.kicad_sch (KiCad schematic)
At the start: 118 parts, among them J1 PROG, J10 Fan1, J11 Fan2, J12 VPS, J15 1B 2A, J18 Power, J19 Supply, J2 Srvo, J20 FAN5V, J3 I2C, J4 1wire, J5 EXT, J6 5V 3V GN 24, J7 485, J9 GN 5V RGB GN, K1 G6K-2, K2 G6K-2, K3 G6K-2, Q1 BC817, Q2 BC817, Q4 BC817, Q5 IRLML6344, Q6 BC817, Q7 TIP41, Q9 IRLML6344, SW1 BTN BLUE, SW10 5V FAN 24V, SW12 RESET, SW2 YELLOW, SW3 GREEN, SW4 RED, SW5 BTN WHITE, SW6 TERM ON, SW7 LED HTR, SW8 REL ROT, SW9 SNS MOV, U1 AMS1117, U14 IPS_240_240, U2 ESP32-WROOM-32, U21 BTS462T, U4 CH340C, U6 MAX3485, X1 FAN_6024

Commit message: Minor fixes in PCB
Parts:
- added R9: GL5516, OptoDevice:R_LDR_5.1x4.3mm_P3.4mm_Vertical, symbol Device:R_Photo
- SW6: value TERM ON -> TERM ON
Connections:
- net GND: now also R9.2
- net LED_BLUE: now also J12.47 (Pin_47), J12.48 (Pin_48); no longer J12.45 (Pin_45), J12.46 (Pin_46)
- net ROT_A: now also R9.1
- net SW_WHITE: now also J12.45 (Pin_45), J12.46 (Pin_46); no longer J12.47 (Pin_47), J12.48 (Pin_48)
Changed lines of the file:
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@@
     )
   )
-  (global_label "LED_BLUE" (shape output) (at 265.43 73.66 180) (fields_autoplaced)
+  (global_label "LED_BLUE" (shape output) (at 265.43 76.2 180) (fields_autoplaced)
     (effects (font (size 1.27 1.27)) (justify right))
-    (property "Intersheet References" "${INTERSHEET_REFS}" (id 0) (at 0 0 0)
+    (property "Intersheet References" "${INTERSHEET_REFS}" (id 0) (at 0 2.54 0)
       (effects (font (size 1.27 1.27)) hide)
     )
@@
     )
   )
-  (global_label "SW_WHITE" (shape input) (at 265.43 76.2 180) (fields_autoplaced)
+  (global_label "SW_WHITE" (shape input) (at 265.43 73.66 180) (fields_autoplaced)
     (effects (font (size 1.27 1.27)) (justify right))
-    (property "Intersheet References" "${INTERSHEET_REFS}" (id 0) (at 0 0 0)
+    (property "Intersheet References" "${INTERSHEET_REFS}" (id 0) (at 0 -2.54 0)
       (effects (font (size 1.27 1.27)) hide)
     )
@@
     )
   )
+  (global_label "ROT_A" (shape output) (at 125.73 43.815 180) (fields_autoplaced)
+    (effects (font (size 1.27 1.27)) (justify right))
+    (property "Intersheet References" "${INTERSHEET_REFS}" (id 0) (at -40.64 -95.885 0)
+      (effects (font (size 1.27 1.27)) hide)
+    )
+  )
   (global_label "I34" (shape input) (at 62.23 82.55 0) (fields_autoplaced)
     (effects (font (size 1.27 1.27)) (justify left))
@@
     (in_bom yes) (on_board yes)
     (property "Reference" "SW6" (id 0) (at 144.78 66.421 0))
-    (property "Value" "TERM ON" (id 1) (at 144.78 68.7324 0))
+    (property "Value" "TERM  ON" (id 1) (at 144.78 68.7324 0))
     (property "Footprint" "liebler_MECH:Switch_SS12D00" (id 2) (at 144.78 73.66 0)
       (effects (font (size 1.27 1.27)) hide)
@@
     (pin "1")
   )
+  (symbol (lib_id "Device:R_Photo") (at 125.73 47.625 0) (unit 1)
+    (in_bom yes) (on_board yes) (fields_autoplaced)
+    (property "Reference" "R9" (id 0) (at 128.27 46.3549 0)
+      (effects (font (size 1.27 1.27)) (justify left))
+    )
+    (property "Value" "GL5516" (id 1) (at 128.27 48.8949 0)
+      (effects (font (size 1.27 1.27)) (justify left))
+    )
+    (property "Footprint" "OptoDevice:R_LDR_5.1x4.3mm_P3.4mm_Vertical" (id 2) (at 127 53.975 90)
+      (effects (font (size 1.27 1.27)) (justify left) hide)
+    )
+    (property "Datasheet" "~" (id 3) (at 125.73 48.895 0)
+      (effects (font (size 1.27 1.27)) hide)
+    )
+    (pin "1")
+    (pin "2")
+  )
   (symbol (lib_id "power:PWR_FLAG") (at 39.37 107.95 270) (unit 1)
     (in_bom yes) (on_board yes) (fields_autoplaced)
@@
     (pin "2")
   )
+  (symbol (lib_id "power:GND") (at 125.73 51.435 90) (unit 1)
+    (in_bom yes) (on_board yes)
+    (property "Reference" "#PWR0112" (id 0) (at 132.08 51.435 0)
+      (effects (font (size 1.27 1.27)) hide)
+    )
+    (property "Value" "GND" (id 1) (at 130.81 51.435 90))
+    (property "Footprint" "" (id 2) (at 125.73 51.435 0)
+      (effects (font (size 1.27 1.27)) hide)
+    )
+    (property "Datasheet" "" (id 3) (at 125.73 51.435 0)
+      (effects (font (size 1.27 1.27)) hide)
+    )
+    (pin "1")
+  )
   (symbol (lib_id "Transistor_BJT:TIP41") (at 234.95 132.08 0) (unit 1)
     (in_bom yes) (on_board yes)
@@
       (reference "#PWR069") (unit 1) (value "GND") (footprint "")
     )
-    (path "/00000000-0000-0000-0000-0000619d0503/ad7fc7e6-3610-455e-998c-d380a0904445"
-      (reference "#PWR070") (unit 1) (value "+24V") (footprint "")
-    )
-    (path "/00000000-0000-0000-0000-0000619d0503/aeacec52-02b6-4d92-afbb-ffce24322b4e"
-      (reference "#PWR071") (unit 1) (value "GND") (footprint "")
-    )
     (path "/00000000-0000-0000-0000-0000619d0503/d0308254-37b5-4ea9-8c28-7173fa94c20f"
       (reference "#PWR072") (unit 1) (value "GND") (footprint "")
@@
       (reference "#PWR0111") (unit 1) (value "GND") (footprint "")
     )
+    (path "/cd3398eb-87bd-45fa-98d7-ae21f2e3fb96"
+      (reference "#PWR0112") (unit 1) (value "GND") (footprint "")
+    )
     (path "/00000000-0000-0000-0000-0000619d0503/31995acd-80df-4908-80d1-82c6b238f1ef"
       (reference "#PWR0113") (unit 1) (value "GND") (footprint "")
@@
       (reference "J22") (unit 1) (value "AudioJack3_SwitchT") (footprint "liebler_CONN:PJ-327A")
     )
-    (path "/00000000-0000-0000-0000-0000619d0503/3b5afaf3-e4c2-4cf0-932f-92cccca5c155"
-      (reference "J23") (unit 1) (value "USB_PD") (footprint "Connector_PinHeader_2.54mm:PinHeader_1x04_P2.54mm_Vertical")
-    )
     (path "/00000000-0000-0000-0000-000061349a3c/b0f885e6-bad8-4725-9d62-48d952608fb4"
       (reference "J24") (unit 1) (value "AOUT") (footprint "Connector_JST:JST_XH_S4B-XH-A_1x04_P2.50mm_Horizontal")
@@
       (reference "R8") (unit 1) (value "4k7") (footprint "Resistor_SMD:R_0603_1608Metric")
     )
+    (path "/5e4bcb54-6c58-48ef-9d8e-93cd3ac9bec0"
+      (reference "R9") (unit 1) (value "GL5516") (footprint "OptoDevice:R_LDR_5.1x4.3mm_P3.4mm_Vertical")
+    )
     (path "/00000000-0000-0000-0000-00006193d61b"
       (reference "R11") (unit 1) (value "1k") (footprint "Resistor_SMD:R_0603_1608Metric")
@@
     )
     (path "/00000000-0000-0000-0000-00006196162e"
-      (reference "SW6") (unit 1) (value "TERM ON") (footprint "liebler_MECH:Switch_SS12D00")
+      (reference "SW6") (unit 1) (value "TERM  ON") (footprint "liebler_MECH:Switch_SS12D00")
     )
     (path "/00000000-0000-0000-0000-0000619f4587"

Commit message: Various
Parts:
- removed J12: VPS, Connector_PinHeader_2.54mm:PinHeader_2x25_P2.54mm_Vertical, symbol Connector_Generic:Conn_02x25_Odd_Even
- removed J19: Supply, Connector_PinHeader_2.54mm:PinHeader_2x04_P2.54mm_Vertical, symbol Connector_Generic:Conn_02x04_Odd_Even
- added J12: VPS, Connector_PinHeader_2.54mm:PinHeader_2x29_P2.54mm_Vertical, symbol Connector_Generic:Conn_02x29_Odd_Even
- SW6: value TERM ON -> OFF TERM ON
Connections:
- net +3V3: now also J12.1 (Pin_1), J12.2 (Pin_2)
- net +5V: now also J12.5 (Pin_5), J12.6 (Pin_6), J12.7 (Pin_7), J12.8 (Pin_8)
- net GND: now also J12.3 (Pin_3), J12.4 (Pin_4)
- net K1_11: now also J12.11 (Pin_11), J12.12 (Pin_12)
- net K1_12: now also J12.13 (Pin_13), J12.14 (Pin_14)
- net K1_14: now also J12.15 (Pin_15), J12.16 (Pin_16)
- net K1_21: now also J12.17 (Pin_17), J12.18 (Pin_18)
- net K1_22: now also J12.19 (Pin_19), J12.20 (Pin_20)
- net K1_24: now also J12.21 (Pin_21), J12.22 (Pin_22)
- net K1_A1: now also J12.10 (Pin_10), J12.9 (Pin_9)
- net K2_11: now also J12.25 (Pin_25), J12.26 (Pin_26)
- net K2_12: now also J12.27 (Pin_27), J12.28 (Pin_28)
- net K2_14: now also J12.29 (Pin_29), J12.30 (Pin_30)
- net K2_21: now also J12.31 (Pin_31), J12.32 (Pin_32)
- net K2_22: now also J12.33 (Pin_33), J12.34 (Pin_34)
- net K2_24: now also J12.35 (Pin_35), J12.36 (Pin_36)
- net K2_A1: now also J12.23 (Pin_23), J12.24 (Pin_24)
- net K3_11: now also J12.39 (Pin_39), J12.40 (Pin_40)
- net K3_12: now also J12.41 (Pin_41), J12.42 (Pin_42)
- net K3_14: now also J12.43 (Pin_43), J12.44 (Pin_44)
- net K3_21: now also J12.45 (Pin_45), J12.46 (Pin_46)
- net K3_22: now also J12.47 (Pin_47), J12.48 (Pin_48)
- net K3_24: now also J12.49 (Pin_49), J12.50 (Pin_50)
- net LED_BLUE: now also J12.55 (Pin_55), J12.56 (Pin_56)
- net LED_WHITE: now also J12.57 (Pin_57), J12.58 (Pin_58)
- net SW_BLUE: now also J12.51 (Pin_51), J12.52 (Pin_52)
- net SW_WHITE: now also J12.53 (Pin_53), J12.54 (Pin_54)
- net at R37.2: now also J12.37 (Pin_37), J12.38 (Pin_38)
