File: pcb_frontplate/pcbV10_front.kicad_pcb (KiCad board)
At the start: 2 copper layers, 100 x 100 mm, 5 parts

Commit message: Minor fixes in PCB
Parts:
- moved G*** 2.00 mm to (100.4, 89.9)
Other:
- outline, holes or cut-outs redrawn
- board text added: "5V 5V"
- board text added: "Brightness"
- board text added: "Für Forschung und Lehre in Friede und Freiheit, überall und jederzeit!"
- board text added: "RGB-LED Ext"
- board text added: "Rotary Encoder Time Relay A1"
- board text added: "TERM ON TERM OFF"
- board text removed: "LED EXT"
- board text removed: "Rotary Encoder Time Relay"
- board text removed: "SW BLUE LED BLUE SW_WHITE LED WHITE"
- board text removed: "TERM OFF TERM ON"

Commit message: Various
Parts:
- moved G*** 0.40 mm to (100.4, 90.3)
Other:
- outline, holes or cut-outs redrawn
Changed lines of the file:
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@@
   )
   (footprint "liebler_DRAWINGS:speaker" (layer "F.Cu")
-    (at 100.4 89.9)
+    (at 100.4 90.3)
     (attr through_hole)
     (fp_text reference "G***" (at 0 0) (layer "F.SilkS") hide
@@
   (gr_circle (center 71.5 66) (end 71.5 64) (layer "Edge.Cuts") (width 0.05) (fill none))
   (gr_circle (center 134.5 138.5) (end 141.5 138.5) (layer "Edge.Cuts") (width 0.05) (fill none))
-  (gr_line (start 100.5 75.5) (end 105.6 75.5) (layer "Edge.Cuts") (width 0.05))
+  (gr_line (start 100.5 75.3) (end 105.8 75.3) (layer "Edge.Cuts") (width 0.05))
   (gr_rect (start 61.8 87.3) (end 67 85.1) (layer "Edge.Cuts") (width 0.05) (fill none))
   (gr_line (start 78.3 88.2) (end 78.3 104.2) (layer "Edge.Cuts") (width 0.05))
   (gr_circle (center 76.65 58.4) (end 78.25 58.4) (layer "Edge.Cuts") (width 0.05) (fill none))
-  (gr_line (start 105.6 75.5) (end 105.6 87.3) (layer "Edge.Cuts") (width 0.05))
-  (gr_line (start 120.699999 106.8) (end 120.7 114.8) (layer "Edge.Cuts") (width 0.05))
-  (gr_line (start 95.4 87.3) (end 95.4 75.5) (layer "Edge.Cuts") (width 0.05))
+  (gr_line (start 105.8 75.3) (end 105.8 88) (layer "Edge.Cuts") (width 0.05))
+  (gr_line (start 120.699999 106.8) (end 120.7 113.8) (layer "Edge.Cuts") (width 0.05))
+  (gr_line (start 95.2 88) (end 95.2 75.3) (layer "Edge.Cuts") (width 0.05))
   (gr_circle (center 126.9 67) (end 132.3 67) (layer "Edge.Cuts") (width 0.05) (fill none))
   (gr_rect (start 105 119.6) (end 107.2 124.8) (layer "Edge.Cuts") (width 0.05) (fill none))
@@
   (gr_arc (start 136.2 80.6) (mid 135.119302 78.5) (end 136.2 76.4) (layer "Edge.Cuts") (width 0.05))
   (gr_line (start 50 50) (end 150 50) (layer "Edge.Cuts") (width 0.05))
-  (gr_line (start 120.7 114.8) (end 108.5 114.8) (layer "Edge.Cuts") (width 0.05))
+  (gr_line (start 120.7 113.8) (end 108.5 113.8) (layer "Edge.Cuts") (width 0.05))
   (gr_line (start 60.1 70.2) (end 53 70.2) (layer "Edge.Cuts") (width 0.05))
-  (gr_line (start 108.5 114.8) (end 108.5 127.2) (layer "Edge.Cuts") (width 0.05))
+  (gr_line (start 108.5 113.8) (end 108.5 127.2) (layer "Edge.Cuts") (width 0.05))
   (gr_rect (start 119.1 72.8) (end 140.4 75.8) (layer "Edge.Cuts") (width 0.05) (fill none))
   (gr_circle (center 78.5 66) (end 78.5 64) (layer "Edge.Cuts") (width 0.05) (fill none))
   (gr_line (start 78.3 104.2) (end 61.5 104.2) (layer "Edge.Cuts") (width 0.05))
   (gr_rect (start 105.6 91) (end 119.2 94) (layer "Edge.Cuts") (width 0.05) (fill none))
-  (gr_line (start 105.6 87.3) (end 95.4 87.3) (layer "Edge.Cuts") (width 0.05))
+  (gr_line (start 105.8 88) (end 95.2 88) (layer "Edge.Cuts") (width 0.05))
   (gr_line (start 150 150) (end 50 150) (layer "Edge.Cuts") (width 0.05))
   (gr_circle (center 121.15 58.4) (end 122.75 58.4) (layer "Edge.Cuts") (width 0.05) (fill none))
   (gr_line (start 53 94.1) (end 53 70.2) (layer "Edge.Cuts") (width 0.05))
   (gr_line (start 127.4 124.8) (end 127.4 100.7) (layer "Edge.Cuts") (width 0.05))
-  (gr_line (start 95.4 75.5) (end 100.5 75.5) (layer "Edge.Cuts") (width 0.05))
+  (gr_line (start 95.2 75.3) (end 100.5 75.3) (layer "Edge.Cuts") (width 0.05))
   (gr_arc (start 121.499999 138.2) (mid 107.739945 140.34164) (end 120.684899 135.208038) (layer "Edge.Cuts") (width 0.05))
   (gr_line (start 61.5 104.2) (end 61.5 94.1) (layer "Edge.Cuts") (width 0.05))
@@
     (effects (font (size 1.5 1) (thickness 0.15)) (justify right))
   )
+  (gr_text "EXT" (at 124.3 99.3) (layer "F.SilkS")
+    (effects (font (size 2 1.3) (thickness 0.2)))
+  )
+  (gr_text "RGB-LED\nExt" (at 53.6 64.5 90) (layer "F.SilkS")
+    (effects (font (size 2 1.3) (thickness 0.2)))
+  )
   (gr_text "A1\n11\n12\n14\n21\n22\n24" (at 149.5 84.9) (layer "F.SilkS")
     (effects (font (size 1.6 1.2) (thickness 0.2)) (justify right))
   )
-  (gr_text "EXT" (at 124.3 99.3) (layer "F.SilkS")
-    (effects (font (size 2 1.3) (thickness 0.2)))
-  )
-  (gr_text "RGB-LED\nExt" (at 53.6 64.5 90) (layer "F.SilkS")
-    (effects (font (size 2 1.3) (thickness 0.2)))
-  )
   (gr_text "Lab@Home v11" (at 92.1 146.2) (layer "F.SilkS")

Commit message: Various
Other:
- outline, holes or cut-outs redrawn
- board text added: "Lab@Home v12"
- board text added: "blue 5V white 5V"
- board text removed: "5V 5V"
- board text removed: "Lab@Home v11"
Changed lines of the file:
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@@
   (gr_line (start 146.5 138.7) (end 146.1 138.7) (layer "F.SilkS") (width 0.12))
   (gr_line (start 145.9 81.7) (end 145.9 82.4) (layer "F.SilkS") (width 0.12))
-  (gr_rect (start 150 139.1) (end 140 129.5) (layer "F.SilkS") (width 0.12) (fill none))
+  (gr_rect (start 150 139.1) (end 139.35 129.5) (layer "F.SilkS") (width 0.12) (fill none))
   (gr_line (start 147.4 130.4) (end 147.4 129.7) (layer "F.SilkS") (width 0.12))
   (gr_line (start 144 125) (end 144 128.3) (layer "F.SilkS") (width 0.12))
@@
   (gr_line (start 144 85) (end 147.1 85) (layer "F.SilkS") (width 0.12))
   (gr_line (start 144.6 89.4) (end 145.9 89.4) (layer "F.SilkS") (width 0.12))
-  (gr_rect (start 150 111.7) (end 140 129.3) (layer "F.SilkS") (width 0.12) (fill none))
+  (gr_rect (start 150 111.7) (end 139.35 129.3) (layer "F.SilkS") (width 0.12) (fill none))
   (gr_line (start 161 125.8) (end 161.9 125.2) (layer "F.SilkS") (width 0.12))
   (gr_line (start 144 105.3) (end 147.1 105.3) (layer "F.SilkS") (width 0.12))
@@
   (gr_line (start 144 87.5) (end 147.1 87.5) (layer "F.SilkS") (width 0.12))
   (gr_line (start 161.7 123.9) (end 161.7 124.1) (layer "F.SilkS") (width 0.12))
-  (gr_line (start 146.45 136.4) (end 144.95 141.6) (layer "F.SilkS") (width 0.12))
+  (gr_line (start 146.3 136.45) (end 144.95 141.6) (layer "F.SilkS") (width 0.12))
   (gr_line (start 161 125.8) (end 161 124.6) (layer "F.SilkS") (width 0.12))
-  (gr_rect (start 150 74.5) (end 140 64.9) (layer "F.SilkS") (width 0.12) (fill none))
+  (gr_rect (start 150 74.5) (end 139.35 64.9) (layer "F.SilkS") (width 0.12) (fill none))
   (gr_line (start 144 87.5) (end 145.5 90.1) (layer "F.SilkS") (width 0.12))
   (gr_line (start 147.1 137.7) (end 148.1 138.75) (layer "F.SilkS") (width 0.12))
@@
   (gr_line (start 146.3 135.7) (end 146.3 136.2) (layer "F.SilkS") (width 0.12))
   (gr_line (start 144 115.4) (end 145.5 118) (layer "F.SilkS") (width 0.12))
-  (gr_line (start 138.4 130.2) (end 137.1 127.6) (layer "F.SilkS") (width 0.12))
   (gr_line (start 142.8 77.3) (end 142.8 77.9) (layer "F.SilkS") (width 0.12))
   (gr_line (start 147.35 139.3) (end 145.85 144.5) (layer "F.SilkS") (width 0.12))
@@
   (gr_line (start 146.8 138.2) (end 146.3 138.2) (layer "F.SilkS") (width 0.12))
   (gr_circle (center 146.2 133.2) (end 146.2 133) (layer "F.SilkS") (width 0.12) (fill none))
-  (gr_rect (start 150 76.1) (end 140 93.7) (layer "F.SilkS") (width 0.12) (fill none))
+  (gr_rect (start 150 76.1) (end 139.35 93.7) (layer "F.SilkS") (width 0.12) (fill none))
   (gr_line (start 144 105.3) (end 145.5 107.9) (layer "F.SilkS") (width 0.12))
-  (gr_line (start 143.7 133.4) (end 141.5 137.2) (layer "F.SilkS") (width 0.12))
   (gr_line (start 147.1 136.2) (end 148.1 135.2) (layer "F.SilkS") (width 0.12))
   (gr_line (start 144 95.1) (end 142.8 95.1) (layer "F.SilkS") (width 0.12))
   (gr_line (start 161.7 124.4) (end 162.2 123.9) (layer "F.SilkS") (width 0.12))
-  (gr_rect (start 150 93.9) (end 140 111.5) (layer "F.SilkS") (width 0.12) (fill none))
-  (gr_line (start 143.7 130.8) (end 138.4 130.2) (layer "F.SilkS") (width 0.12))
+  (gr_rect (start 150 93.9) (end 139.35 111.5) (layer "F.SilkS") (width 0.12) (fill none))
   (gr_line (start 142.5 95.7) (end 143.1 95.7) (layer "F.SilkS") (width 0.12))
   (gr_line (start 145.8 77.3) (end 147.1 77.3) (layer "F.SilkS") (width 0.12))
@@
   (gr_rect (start 61.6 115.9) (end 66.8 118.1) (layer "Edge.Cuts") (width 0.05) (fill none))
   (gr_line (start 136.2 80.6) (end 139.1 80.6) (layer "Edge.Cuts") (width 0.05))
-  (gr_rect (start 78.9 96.4) (end 81.1 101.6) (layer "Edge.Cuts") (width 0.05) (fill none))
+  (gr_rect (start 79.1 96.4) (end 81.3 101.6) (layer "Edge.Cuts") (width 0.05) (fill none))
   (gr_arc (start 139.1 76.400001) (mid 140.223885 78.5) (end 139.1 80.599999) (layer "Edge.Cuts") (width 0.05))
   (gr_circle (center 134.5 121) (end 141.5 121) (layer "Edge.Cuts") (width 0.05) (fill none))
@@
     (effects (font (size 1.6 1.2) (thickness 0.2)) (justify right))
   )
-  (gr_text "TERM ON\nTERM OFF" (at 81 99) (layer "F.SilkS")
+  (gr_text "TERM ON\nTERM OFF" (at 81.3 99) (layer "F.SilkS")
     (effects (font (size 1 1) (thickness 0.15)) (justify left))
   )
@@
     (effects (font (size 2 1.3) (thickness 0.2)) (justify left))
   )
-  (gr_text "5V\n5V" (at 146 132.1) (layer "F.SilkS")
+  (gr_text "blue 5V\nwhite 5V" (at 145.9 132.1) (layer "F.SilkS")
     (effects (font (size 1.5 1) (thickness 0.15)) (justify right))
   )
@@
     (effects (font (size 1.6 1.2) (thickness 0.2)) (justify right))
   )
-  (gr_text "Lab@Home v11" (at 92.1 146.2) (layer "F.SilkS")
+  (gr_text "Lab@Home v12" (at 92.1 146.2) (layer "F.SilkS")
     (effects (font (size 3 2) (thickness 0.4)))
   )
