File: labathome_pcb/pcbV10.kicad_pcb (KiCad board)
At the start: 2 copper layers, 100 x 100 mm, 221 parts, among them J1 PROG, J10 Fan1, J11 Fan2, J12 VPS, J13 SPK, J15 1B 2A, J16 BME280, J17 CCS811, J18 Power, J19 SPK, J2 Srvo, J20 FAN5V, J21 QWIIC, J22 AudioJack3_SwitchT, J24 AOUT, J3 I2C, J4 1wire, J5 EXT, J6 5V 3V GN 24, J7 485, J8 POWER, J9 GN 5V RGB GN, K1 G6K-2, K2 G6K-2, K3 G6K-2, Q1 BC817, Q2 BC817, Q4 BC817, Q5 IRLML6344, Q6 BC817, Q7 TIP41, Q9 IRLML6344, SW1 BTN BLUE, SW10 5V FAN 24V, SW11 PROG 5V POWER, SW12 RESET, SW2 YELLOW, SW3 GREEN, SW4 RED, SW5 BTN WHITE, SW6 OFF TERM ON, SW7 LED HTR, SW8 REL ROT, SW9 SNS MOV, U1 AMS1117, U10 LM358, U11 FUSB302BMPX, U12 BME680, U13 BME280, U14 IPS_240_240, U15 CCS811, U16 AS4950, U18 MD8002A, U19 DS18B20, U2 ESP32-WROOM-32, U20 BH1750, U22 AM612, U23 MPU-6050, U24 SRV05, U25 NS4168, U26 MSM261D4030H1CPM, U3 AHT21, U4 CH340C, U5 UDA1334, U6 MAX3485, U7 DS18B20, U8 NRF24L01, U9 RY8310, X1 FAN_6024, X2 XGZP6897D, X3 Ebyte E32, X4 SIM7080G

Commit message: LTSpice Simulation & minor optical fixes
Parts:
- J24: value AOUT -> 24 GN GN OUT
Changed lines of the file:
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@@
       (effects (font (size 1 1) (thickness 0.15)))
     )
-    (fp_text value "IRLML6344" (at -7.5 1.6) (layer "F.SilkS")
+    (fp_text value "IRLML6344" (at -7.5 1.6) (layer "F.SilkS") hide
       (effects (font (size 1 1) (thickness 0.15)))
     )
@@
       (effects (font (size 1 1) (thickness 0.15)))
     )
-    (fp_text value "IRLML6344" (at 3.15 -1.8 90) (layer "F.SilkS")
+    (fp_text value "IRLML6344" (at 3.15 -1.8 90) (layer "F.SilkS") hide
       (effects (font (size 1 1) (thickness 0.15)))
     )
@@
       (effects (font (size 1 1) (thickness 0.15)))
     )
-    (fp_text value "10k" (at 0 -2.7) (layer "F.SilkS")
+    (fp_text value "10k" (at 0 -2.7) (layer "F.SilkS") hide
       (effects (font (size 1 1) (thickness 0.15)))
     )
@@
     (pad "8" smd roundrect (at 4.5 -3.81 270) (size 1.6 1) (layers "F.Cu" "F.Paste" "F.Mask") (roundrect_rratio 0.25)
       (net 2 "GND") (pinfunction "GND") (pintype "power_in"))
+    (model "${CUSTOM_LIBS}/liebler_SEMICONDUCTORS.pretty/sop8.STEP"
+      (offset (xyz 0 0 3))
+      (scale (xyz 2 2 1.7))
+      (rotate (xyz -90 0 90))
+    )
   )
   (footprint "Capacitor_SMD:C_0402_1005Metric" (layer "F.Cu")
@@
     (property "Sheetname" "analog_amp")
     (attr through_hole exclude_from_pos_files)
-    (fp_text reference "J24" (at 3.75 -3.5) (layer "F.SilkS")
+    (fp_text reference "J24" (at 3.75 -3.5) (layer "F.SilkS") hide
       (effects (font (size 1 1) (thickness 0.15)))
     )
-    (fp_text value "AOUT" (at 3.75 10.4) (layer "F.Fab")
+    (fp_text value "24 GN GN OUT" (at 3.75 -1.9) (layer "F.SilkS")
       (effects (font (size 1 1) (thickness 0.15)))
     )
