File: labathome_pcb/actors.kicad_sch (KiCad schematic)
At the start: 33 parts, among them J26 Servos, J7 FAN5V, J8 3V GN RGB 5V, Q1 BC817, Q2 IRLML6344, Q3 MJD31C, Q5 IRLML6344, X1 FAN_6024

Commit message: Optimized PCB
Parts:
- added JP8: Heater, Jumper:SolderJumper-2_P1.3mm_Bridged2Bar_RoundedPad1.0x1.5mm, symbol Jumper:Jumper_2_Bridged
- added JP9: Fan, Jumper:SolderJumper-2_P1.3mm_Bridged2Bar_RoundedPad1.0x1.5mm, symbol Jumper:Jumper_2_Bridged
Connections:
- net FAN_DRIVE: now also JP9.1 (A); no longer R35.2
- net HEATER: now also JP8.1 (A); no longer D14.2 (A), R30.2
- new net: D14.2 (A), JP8.2 (B), R30.2
- new net: JP9.2 (B), R35.2
Other:
- moved on the sheet: D14, J26, Q2, R30, R31, R33, R6

Commit message: Bus servos
Parts:
- removed J26: Servos, liebler_CONN:PinHeader_2x09_P2.54mm_Horizontal_SMD, symbol Connector_Generic:Conn_02x09_Odd_Even
- added C10, C8, C9: 10p, Capacitor_SMD:C_0402_1005Metric, symbol Device:C
- added C100, C99: u1, Capacitor_SMD:C_0201_0603Metric, symbol Device:C
- added C38: 10n/35V, Capacitor_SMD:C_0402_1005Metric, symbol Device:C
- added C39: 100u, Capacitor_SMD:CP_Elec_6.3x5.4, symbol Device:C_Polarized
- added C51: u1/16V, Capacitor_SMD:C_0603_1608Metric, symbol Device:C
- added C52, C63: u1/35V, Capacitor_SMD:C_0603_1608Metric, symbol Device:C
- added C61: 4u7/6V3, Capacitor_SMD:C_0402_1005Metric, symbol Device:C
- added J1: HALL, liebler_CONN:PhoenixContact_MC_1,5_4-G-3.5_1x04_P3.50mm_Horizontal_smallerCourtyard, symbol Connector_Generic:Conn_01x04
- added J18: Bus-Servo, Connector_Molex:Molex_SPOX_5267-03A_1x03_P2.50mm_Vertical, symbol Connector_Generic:Conn_01x03
- added J25: Servos, liebler_CONN:PinHeader_2x09_P2.54mm_Horizontal_SMD, symbol Connector_Generic:Conn_02x09_Odd_Even
- added J28: Brushless, liebler_CONN:PhoenixContact_MC_1,5_4-G-3.5_1x04_P3.50mm_Horizontal_smallerCourtyard, symbol Connector_Generic:Conn_01x04
- added R10, R14, R16: 2k2, Resistor_SMD:R_0402_1005Metric, symbol Device:R
- added R17, R51, R63, R64, R76, R81: 10k, Resistor_SMD:R_0201_0603Metric, symbol Device:R
- added R38: r1, Resistor_SMD:R_2010_5025Metric, symbol Device:R
- added U24: 74HCT1G125, Package_TO_SOT_SMD:SOT-353_SC-70-5, symbol 74xGxx:74LVC1G125
- added U25: 74HCT1G126, Package_TO_SOT_SMD:SOT-353_SC-70-5, symbol 74xGxx:74LVC1G126
- added U3: DRV8313, Package_SO:HTSSOP-28-1EP_4.4x9.7mm_P0.65mm_EP2.85x5.4mm_ThermalVias, symbol liebler_SEMICONDUCTORS:DRV8313
Connections:
- net +3V3: now also C99.2, R17.1, R51.1, R64.1, R81.1, U25.5 (VCC)
- net +5V: now also C100.2, J25.10 (Pin_10), J25.15 (Pin_15), J25.16 (Pin_16), J25.3 (Pin_3), J25.4 (Pin_4), J25.9 (Pin_9), R76.1, U24.5 (VCC)
- net FAN_DRIVE: now also J25.5 (Pin_5)
- net GND: now also C10.2, C100.1, C39.2, C52.1, C61.2, C63.2, C8.2, C9.2, C99.1, J1.4 (Pin_4), J18.3 (Pin_3), J25.1 (Pin_1), J25.13 (Pin_13), J25.14 (Pin_14), J25.2 (Pin_2), J25.7 (Pin_7), J25.8 (Pin_8), J28.4 (Pin_4), R38.2, U24.3 (GND), U25.3 (GND), U3.12 (COMPP), U3.13 (COMPN), U3.14 (GND), U3.20 (GND), U3.21 (NC_GND), U3.28 (GND), U3.29 (EP_GND)
- net LED_WHITE_P: now also J25.6 (Pin_6)
- net Servo0: now also J25.17 (Pin_17)
- net Servo1: now also J25.18 (Pin_18)
- net Servo2: now also J25.11 (Pin_11)
- net Servo3: now also J25.12 (Pin_12)
- net +24V renamed 5-24V
- net 5-24V: now also C39.1, C51.2, C52.2, C63.1, J18.2 (Pin_2), U3.11 (VM), U3.4 (VM)
- new net: C61.1, U3.15 (V3P3)
- new net: J1.2 (Pin_2), R14.1
- new net: J1.1 (Pin_1), R16.1
- new net: J1.3 (Pin_3), R10.1
- new net: C51.1, U3.3 (VCP)
- new net: C38.1, U3.1 (CPL)
- new net: C38.2, U3.2 (CPH)
- new net: J28.3 (Pin_3), U3.5 (OUT1)
- new net: J28.2 (Pin_2), U3.8 (OUT2)
- new net: J28.1 (Pin_1), U3.9 (OUT3)
- new net BL_DRV1: U3.27 (IN1)
- new net BL_DRV2: U3.25 (IN2)
- new net BL_DRV3: U3.23 (IN3)
- new net BL_ENABLE: R63.2, U3.22 (EN3), U3.24 (EN2), U3.26 (EN1)
- new net BL_ENABLEx: R63.1
- new net BL_FAULT: U3.18 (nFAULT)
- new net BL_HALL1: C8.1, R16.2, R17.2
- new net BL_HALL2: C9.1, R14.2, R51.2
- new net BL_HALL3: C10.1, R10.2, R64.2
- new net BL_ISENSE: R38.1, U3.10 (PGND3), U3.6 (PGND1), U3.7 (PGND2)
- new net BL_RESET: U3.16 (nRESET)
- new net BL_SLEEP: U3.17 (nSLEEP)
- new net SERVO_BUS: J18.1 (Pin_1), R76.2, U24.4, U25.2
- new net SERVO_BUS_RX: R81.2, U25.4
- new net SERVO_BUS_TX: U24.2
- new net SERVO_BUS_TX_EN: U24.1, U25.1
- no-connect marks 0 -> 1
Other:
- note added: "Brushless Driver"
- moved on the sheet: C45, C46, C47, C48, D15, D16, D17, D20, D21, J8, R70
