File: labathome_pcb/actors.kicad_sch (KiCad schematic)
At the start: 62 parts, among them J1 HALL, J18 Bus-Servo, J25 Servos, J28 Brushless, J7 FAN5V, J8 3V GN RGB 5V, Q1 BC817, Q2 IRLML6344, Q3 MJD31C, Q5 IRLML6344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

Commit message: Merge
Parts:
- removed C100, C99: u1, Capacitor_SMD:C_0201_0603Metric, symbol Device:C
- removed R81: 10k, Resistor_SMD:R_0201_0603Metric, symbol Device:R
- removed U24: 74HCT1G125, Package_TO_SOT_SMD:SOT-353_SC-70-5, symbol 74xGxx:74LVC1G125
- removed U25: 74HCT1G126, Package_TO_SOT_SMD:SOT-353_SC-70-5, symbol 74xGxx:74LVC1G126
- added R77: 1k, Resistor_SMD:R_0805_2012Metric_Pad1.20x1.40mm_HandSolder, symbol Device:R
- R76: footprint Resistor_SMD:R_0201_0603Metric -> Resistor_SMD:R_0805_2012Metric_Pad1.20x1.40mm_HandSolder
Connections:
- net SERVO_BUS is gone; now on net SERVO_BUS_RX: J18.1 (Pin_1), R76.2
- net +3V3: now also R76.1
- net +5V: no longer R76.1
- net SERVO_BUS_RX: now also R77.2
- net SERVO_BUS_TX: now also R77.1

Commit message: Minor changes
Parts:
- C10, C8, C9: MPN (none) -> CL05C100JB5NNNC; Manufacturer (none) -> Samsung Electro-Mechanics
- C38: MPN (none) -> CL05B103KB5NNNC; Manufacturer (none) -> Samsung Electro-Mechanics
- C39: MPN (none) -> RST100UF35V009; Manufacturer (none) -> KNSCHA
- C45, C46, C47, C48: MPN (none) -> GRM033R61A104KE15D; Manufacturer (none) -> Murata Electronics
- C51, C52, C63: MPN (none) -> CC0603KRX7R9BB104; Manufacturer (none) -> YAGEO
- C61: MPN (none) -> CL05A475MP5NRNC; Manufacturer (none) -> Samsung Electro-Mechanics
- D10, D11, D12, D8, D9: MPN (none) -> HL-A-2835D46W-S1-08-HR3(2800-3100K); Manufacturer (none) -> HONGLITRONIC(Hongli Zhihui (HONGLITRONIC))
- D14: MPN (none) -> LTST-C230KRKT; Manufacturer (none) -> Lite-On
- D15, D16, D17, D21: MPN (none) -> SK6812MINI-EA; Manufacturer (none) -> OPSCO Optoelectronics
- D20: MPN (none) -> 1N5819WS; Manufacturer (none) -> Guangdong Hottech
- J1, J28: MPN (none) -> KF2EDGR-3.5-4P; Manufacturer (none) -> Cixi Kefa Elec
- J18: MPN (none) -> 5267-03A / 22035035; Manufacturer (none) -> Molex
- J25: MPN (none) -> PZ254-2-09-WS; Manufacturer (none) -> HCTL
- J7: MPN (none) -> B2B-XH-A(LF)(SN); Manufacturer (none) -> JST
- J8: MPN (none) -> 2.54-1*4P; Manufacturer (none) -> BOOMELE(Boom Precision Elec)
- Q1: MPN (none) -> MMBT3904(RANGE:100-300); Manufacturer (none) -> Jiangsu Changjing Electronics Technology Co., Ltd.
- Q2, Q5: MPN (none) -> AO3400; Manufacturer (none) -> GOODWORK
- Q3: MPN (none) -> MJD31C; Manufacturer (none) -> Jiangsu Changjing Electronics Technology Co., Ltd.
- R10, R14, R16: MPN (none) -> 0402WGF2201TCE; Manufacturer (none) -> UNI-ROYAL(Uniroyal Elec)
- R12, R30, R35, R6: MPN (none) -> 0402WGF1001TCE; Manufacturer (none) -> UNI-ROYAL(Uniroyal Elec)
- R13, R15: MPN (none) -> 1206W4F100JT5E; Manufacturer (none) -> UNI-ROYAL(Uniroyal Elec)
- R17, R31, R45, R51, R63, R64: MPN (none) -> 0201WMF1002TEE; Manufacturer (none) -> UNI-ROYAL(Uniroyal Elec)
- R38: MPN (none) -> 201007F100LT4E; Manufacturer (none) -> UNI-ROYAL(Uniroyal Elec)
- R70: MPN (none) -> 0402WGF2200TCE; Manufacturer (none) -> UNI-ROYAL(Uniroyal Elec)
- U3: MPN (none) -> DRV8313PWPR; Manufacturer (none) -> Texas Instruments

Commit message: Various
Parts:
- R38: footprint Resistor_SMD:R_2010_5025Metric -> Resistor_SMD:R_1206_3216Metric; MPN 201007F100LT4E -> FRM121WFR100TM; Manufacturer UNI-ROYAL(Uniroyal Elec) -> FOJAN
Changed lines of the file:
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@@
 			)
 		)
-		(property "Footprint" "Resistor_SMD:R_2010_5025Metric"
+		(property "Footprint" "Resistor_SMD:R_1206_3216Metric"
 			(at 249.682 58.42 90)
 			(effects
@@
 			)
 		)
-		(property "MPN" "201007F100LT4E"
+		(property "MPN" "FRM121WFR100TM"
 			(at 251.46 58.42 0)
 			(effects
@@
 			)
 		)
-		(property "Manufacturer" "UNI-ROYAL(Uniroyal Elec)"
+		(property "Manufacturer" " FOJAN"
 			(at 251.46 58.42 0)
 			(effects
