File: labathome_pcb/psu.kicad_sch (KiCad schematic)
At the start: 21 parts, among them J8 POWER, SW11 PROG 5V POWER, U11 FUSB302BMPX, U24 SRV05, U9 RY8310

Commit message: Reorganization of code
Parts:
- removed C17, C58: 1u, Capacitor_SMD:C_1206_3216Metric, symbol Device:C
- removed C19, C32, C33, C35: u1, Capacitor_SMD:C_0603_1608Metric, symbol Device:C
- removed C22, C60: 10u, Capacitor_SMD:C_1206_3216Metric, symbol Device:C
- removed C36: 22u, Capacitor_SMD:C_0603_1608Metric, symbol Device:C
- removed C56, C57: n33, Capacitor_SMD:C_0603_1608Metric, symbol Device:C
- removed J8: POWER, liebler_CONN:USB_C_Receptacle_HRO_TYPE-C-31-M-12_IMPROVED, symbol Connector:USB_C_Receptacle_USB2.0
- removed JP2: USBC_INT, liebler_CONN:Jumper_Trace_025x150x015, symbol Jumper:Jumper_2_Open
- removed L2: 4u7, Inductor_SMD:L_Abracon_ASPI-0630LR, symbol Device:L
- removed R45: 13k, Resistor_SMD:R_0603_1608Metric, symbol Device:R
- removed R46: 68k, Resistor_SMD:R_0603_1608Metric, symbol Device:R
- removed SW11: PROG 5V POWER, liebler_MECH:Switch_SS12D00, symbol Switch:SW_SPDT
- removed TP1: TP_INT, TestPoint:TestPoint_THTPad_1.0x1.0mm_Drill0.5mm, symbol Connector:TestPoint
- removed U11: FUSB302BMPX, Package_DFN_QFN:WQFN-14-1EP_2.5x2.5mm_P0.5mm_EP1.45x1.45mm, symbol Interface_USB:FUSB302BMPX
- removed U24: SRV05, Package_TO_SOT_SMD:SOT-23-6, symbol Power_Protection:SRV05-4
- removed U9: RY8310, Package_TO_SOT_SMD:SOT-23-6, symbol Regulator_Switching:LMR14206
- added BT1: 18650, Battery:BatteryHolder_MPD_BH-18650-PC2, symbol Device:Battery_Cell
- added C1, C4: 10u, Capacitor_SMD:C_0805_2012Metric, symbol Device:C
- added C28, C29, C30, C31, C7, C83, C84: 22u, Capacitor_SMD:C_0603_1608Metric, symbol Device:C
- added C41, C43: 4u7, Capacitor_SMD:C_0402_1005Metric, symbol Device:C
- added C42, C44: 1u, Capacitor_SMD:C_0402_1005Metric, symbol Device:C
- added C79: u1/35V, Capacitor_SMD:C_0603_1608Metric, symbol Device:C
- added C80: 10u/35V, Capacitor_SMD:C_0805_2012Metric, symbol Device:C
- added C81: u1/16V, Capacitor_SMD:C_0603_1608Metric, symbol Device:C
- added C82: 56p, Capacitor_SMD:C_0402_1005Metric, symbol Device:C
- added J8: POWER, liebler_CONN:USB_C_Receptacle_HRO_TYPE-C-31-M-12_IMPROVED, symbol Connector:USB_C_Receptacle_USB2.0_16P
- added J9: Barrel_Jack_Switch, Connector_BarrelJack:BarrelJack_Horizontal, symbol Connector:Barrel_Jack_Switch
- added JP2: 5V DIR, Jumper:SolderJumper-2_P1.3mm_Bridged2Bar_Pad1.0x1.5mm, symbol Jumper:Jumper_2_Bridged
- added L1: 1u, liebler_PASSIVES:L_0630, symbol Device:L
- added L4: 10u, liebler_PASSIVES:L_0630, symbol Device:L
- added R28, R3, R47, R7: 1R, Resistor_SMD:R_0603_1608Metric, symbol Device:R
- added R4, R60, R72: 10k, Resistor_SMD:R_0201_0603Metric, symbol Device:R
- added R48, R73: 3k3, Resistor_SMD:R_0402_1005Metric, symbol Device:R
- added R59: M1, Resistor_SMD:R_0201_0603Metric, symbol Device:R
- added SW5: POWER, liebler_MECH:SW_Push_1P1T_NO_6x6mm_H6.5mm_Reverse, symbol Switch:SW_Push
- added U11: AMS1117, Package_TO_SOT_SMD:SOT-223-3_TabPin2, symbol Regulator_Linear:AMS1117-3.3
- added U18: TPS2116DRL, Package_TO_SOT_SMD:SOT-583-8, symbol Power_Management:TPS2116DRL
- added U2: IP5306_I2C, Package_SO:HSOP-8-1EP_3.9x4.9mm_P1.27mm_EP2.3x2.3mm_ThermalVias, symbol liebler_SEMICONDUCTORS:IP5306_I2C
- added U27: TPS54202DDC, Package_TO_SOT_SMD:SOT-23-6_Handsoldering, symbol Regulator_Switching:TPS54202DDC
Connections:
- net +24V: now also C79.2, C80.2, J8.A4 (VBUS), J8.A9 (VBUS), J8.B4 (VBUS), J8.B9 (VBUS), J9.2, U27.3 (VIN)
- net +3V3: now also C43.2, C44.1, U11.2 (VO)
- net +5V: now also C28.2, C30.2, C31.2, C41.2, C42.1, JP2.2 (B), U11.3 (VI), U2.8 (VOUT)
- net GND: now also BT1.2 (-), C1.2, C28.1, C29.2, C30.1, C31.1, C4.2, C41.1, C42.2, C43.1, C44.2, C7.2, C79.1, C80.1, C83.2, C84.2, J8.A1 (GND), J8.A12 (GND), J8.B1 (GND), J8.B12 (GND), J8.S1 (SHIELD), J9.1, R48.1, R73.1, SW5.1, U11.1 (GND), U18.1 (GND), U2.9, U27.1 (GND)
- net SCL: now also U2.2 (SCL)
- net SDA: now also U2.3 (SDA)
- net SW: now also C81.2, L4.2, U27.2 (SW)
- new net: C4.1, JP2.1 (A), R47.1, U18.2 (VOUT), U18.7 (VOUT), U2.1 (VIN)
- new net: R4.1, U2.5 (KEY)
- new net: C7.1, R28.2, R7.2, U2.6 (BAT)
- new net: L1.1, U2.7 (SW)
- new net: R48.2, R60.1
- new net: R3.1, R47.2
- new net: C1.1, R3.2
- new net: R4.2, SW5.2
- new net: R72.1, R73.2, U18.4 (PR1)
- new net +3V8: BT1.1 (+), C29.1, L1.2, R28.1, R7.1
- new net 5V_PD: C82.2, C83.1, C84.1, L4.1, R59.1, R72.2, U18.3 (VIN1), U18.5 (MODE)
- new net 5V_USB: U18.6 (VIN2)
- new net BOOT: C81.1, U27.6 (BOOT)
- new net FB: C82.1, R59.2, R60.2, U27.4 (FB)
- new net USBPD_CC1: J8.A5 (CC1)
- new net USBPD_CC2: J8.B5 (CC2)
- new net USBPD_D+: J8.A6 (D+), J8.B6 (D+)
- new net USBPD_D-: J8.A7 (D-), J8.B7 (D-)
- no-connect marks 7 -> 6
Other:
- note added: "5V->3V3"
- note added: "Barrel Jack 24V"
- note added: "Battery"
- note added: "PSU"
- note added: "USB PD"
- company: (none) -> Klaus Liebler
- title: (none) -> lab@home

Commit message: Optimized PCB
Parts:
- removed JP2: 5V DIR, Jumper:SolderJumper-2_P1.3mm_Bridged2Bar_Pad1.0x1.5mm, symbol Jumper:Jumper_2_Bridged
- added SW4: 5V DIR, liebler_MECH:Switch_SS12D00, symbol Switch:SW_Push_SPDT
Connections:
- net +5V: now also SW4.2 (B); no longer C28.2, C30.2, C31.2, U2.8 (VOUT)
- net at C4.1, R47.1, U18.2 (VOUT)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: now also SW4.3 (C)
- new net: C28.2, C30.2, C31.2, SW4.1 (A), U2.8 (VOUT)
Changed lines of the file:
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@@
 	)
 	(junction
+		(at 199.39 33.02)
+		(diameter 0)
+		(color 0 0 0 0)
+	)
+	(junction
 		(at 209.55 33.02)
 		(diameter 0)
@@
 	)
 	(junction
-		(at 187.96 33.02)
-		(diameter 0)
-		(color 0 0 0 0)
-	)
-	(junction
 		(at 38.1 81.28)
 		(diameter 0)
@@
 	)
 	(junction
-		(at 199.39 33.02)
-		(diameter 0)
-		(color 0 0 0 0)
-	)
-	(junction
 		(at 158.75 57.15)
 		(diameter 0)
@@
 	(wire
 		(pts
-			(xy 219.71 33.02) (xy 220.98 33.02)
+			(xy 219.71 33.02) (xy 231.14 33.02)
 		)
 		(stroke
@@
 	(wire
 		(pts
+			(xy 186.69 33.02) (xy 199.39 33.02)
+		)
+		(stroke
+			(width 0)
+			(type default)
+		)
+	)
+	(wire
+		(pts
 			(xy 107.95 27.94) (xy 110.49 27.94)
 		)
@@
 	(wire
 		(pts
-			(xy 25.4 116.84) (xy 25.4 120.65)
+			(xy 231.14 19.05) (xy 158.75 19.05)
 		)
 		(stroke
@@
 	(wire
 		(pts
-			(xy 208.28 35.56) (xy 201.93 35.56)
+			(xy 25.4 116.84) (xy 25.4 120.65)
 		)
 		(stroke
@@
 	(wire
 		(pts
-			(xy 158.75 22.86) (xy 158.75 33.02)
+			(xy 208.28 35.56) (xy 201.93 35.56)
 		)
 		(stroke
@@
 	(wire
 		(pts
-			(xy 187.96 22.86) (xy 187.96 33.02)
+			(xy 231.14 33.02) (xy 231.14 24.13)
 		)
 		(stroke
@@
 	(wire
 		(pts
-			(xy 173.99 22.86) (xy 158.75 22.86)
-		)
-		(stroke
-			(width 0)
-			(type default)
-		)
-	)
-	(wire
-		(pts
-			(xy 187.96 33.02) (xy 199.39 33.02)
-		)
-		(stroke
-			(width 0)
-			(type default)
-		)
-	)
-	(wire
-		(pts
-			(xy 186.69 33.02) (xy 187.96 33.02)
-		)
-		(stroke
-			(width 0)
-			(type default)
-		)
-	)
-	(wire
-		(pts
 			(xy 90.17 113.03) (xy 90.17 128.27)
 		)
@@
 	(wire
 		(pts
-			(xy 184.15 22.86) (xy 187.96 22.86)
+			(xy 100.33 113.03) (xy 100.33 128.27)
 		)
 		(stroke
@@
 	(wire
 		(pts
-			(xy 100.33 113.03) (xy 100.33 128.27)
+			(xy 158.75 19.05) (xy 158.75 33.02)
 		)
 		(stroke
@@
 	(rectangle
 		(start 99.06 15.24)
-		(end 232.41 62.23)
+		(end 252.73 62.23)
 		(stroke
 			(width 0)
@@
 		)
 		(property "Value" "GND"
-			(at 207.01 24.1301 0)
+			(at 211.582 21.336 0)
 			(effects
 				(font
@@
 		)
 		(property "Value" "GND"
-			(at 196.85 24.1301 0)
+			(at 201.422 21.59 0)
 			(effects
 				(font
@@
 	)
 	(symbol
-		(lib_id "Jumper:Jumper_2_Bridged")
-		(at 179.07 22.86 0)
-		(unit 1)
-		(exclude_from_sim yes)
-		(in_bom yes)
-		(on_board yes)
-		(dnp no)
-		(fields_autoplaced yes)
-		(property "Reference" "JP2"
-			(at 179.07 17.78 0)
-			(effects
-				(font
-					(size 1.27 1.27)
-				)
-			)
-		)
-		(property "Value" "5V DIR"
-			(at 179.07 20.32 0)
-			(effects
-				(font
-					(size 1.27 1.27)
-				)
-			)
-		)
-		(property "Footprint" "Jumper:SolderJumper-2_P1.3mm_Bridged2Bar_Pad1.0x1.5mm"
-			(at 179.07 22.86 0)
-			(effects
-				(font
-					(size 1.27 1.27)
-				)
-				(hide yes)
-			)
-		)
-		(property "Datasheet" "~"
-			(at 179.07 22.86 0)
-			(effects
-				(font
-					(size 1.27 1.27)
-				)
-				(hide yes)
-			)
-		)
-		(property "Description" "Jumper, 2-pole, closed/bridged"
-			(at 179.07 22.86 0)
-			(effects
-				(font
-					(size 1.27 1.27)
-				)
-				(hide yes)
-			)
-		)
-		(pin "2"
-		)
-		(pin "1"
-		)
-		(instances
-			(project ""
-				(path "/e4d6926a-1a8b-424d-97c4-66b6ad87e4ac/77dfbe0c-d674-478a-bf0e-cfa040fb2e8f"
-					(reference "JP2")
-					(unit 1)
-				)
-			)
-		)
-	)
-	(symbol
 		(lib_id "Device:R")
 		(at 201.93 39.37 0)
@@
 	)
 	(symbol
+		(lib_id "Switch:SW_Push_SPDT")
+		(at 236.22 21.59 180)
+		(unit 1)
+		(exclude_from_sim no)
+		(in_bom yes)
+		(on_board yes)
+		(dnp no)
+		(fields_autoplaced yes)
+		(property "Reference" "SW4"
+			(at 236.22 12.7 0)
+			(effects
+				(font
+					(size 1.27 1.27)
+				)
+			)
+		)
+		(property "Value" "5V DIR"
+			(at 236.22 15.24 0)
+			(effects
+				(font
+					(size 1.27 1.27)
+				)
+			)
+		)
+		(property "Footprint" "liebler_MECH:Switch_SS12D00"
+			(at 236.22 21.59 0)
+			(effects
+				(font
+					(size 1.27 1.27)
+				)
+				(hide yes)
+			)
+		)
+		(property "Datasheet" "~"
+			(at 236.22 21.59 0)
+			(effects
+				(font
+					(size 1.27 1.27)
+				)
+				(hide yes)
+			)
+		)
+		(property "Description" "Momentary Switch, single pole double throw"
+			(at 236.22 21.59 0)
+			(effects
+				(font
+					(size 1.27 1.27)
+				)
+				(hide yes)
+			)
+		)
+		(pin "3"
+		)
+		(pin "2"
+		)
+		(pin "1"
+		)
+		(instances
+			(project ""
+				(path "/e4d6926a-1a8b-424d-97c4-66b6ad87e4ac/77dfbe0c-d674-478a-bf0e-cfa040fb2e8f"
+					(reference "SW4")
+					(unit 1)
+				)
+			)
+		)
+	)
+	(symbol
 		(lib_id "Device:C")
 		(at 20.32 113.03 180)
@@
 	(symbol
 		(lib_id "power:+5V")
-		(at 220.98 33.02 270)
+		(at 241.3 21.59 270)
 		(unit 1)
 		(exclude_from_sim no)
@@
 		(fields_autoplaced yes)
 		(property "Reference" "#PWR037"
-			(at 217.17 33.02 0)
+			(at 237.49 21.59 0)
 			(effects
 				(font
@@
 		)
 		(property "Value" "+5V"
-			(at 224.79 33.0199 90)
+			(at 245.11 21.5899 90)
 			(effects
 				(font
@@
 		)
 		(property "Footprint" ""
-			(at 220.98 33.02 0)
+			(at 241.3 21.59 0)
 			(effects
 				(font
@@
 		)
 		(property "Datasheet" ""
-			(at 220.98 33.02 0)
+			(at 241.3 21.59 0)
 			(effects
 				(font
@@
 		)
 		(property "Description" "Power symbol creates a global label with name \"+5V\""
-			(at 220.98 33.02 0)
+			(at 241.3 21.59 0)
 			(effects
 				(font
@@
 		)
 		(property "Value" "GND"
-			(at 217.17 24.1301 0)
+			(at 221.742 21.336 0)
 			(effects
 				(font

Commit message: Continued with severe refactoring. Now builds, but completely untested
Connections:
- net +24V renamed 5-24V
- net +3V8 renamed +BATT

Commit message: Various
Parts:
- removed SW4: 5V DIR, liebler_MECH:Switch_SS12D00, symbol Switch:SW_Push_SPDT
- added JP2: 5V_DIR, Jumper:SolderJumper-3_P1.3mm_Bridged2Bar12_RoundedPad1.0x1.5mm, symbol Jumper:Jumper_3_Bridged12
Connections:
- net +5V: now also JP2.2 (C)
- net at C4.1, R47.1, U18.2 (VOUT)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: now also JP2.3 (B)
- net at C28.2, C30.2, C31.2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: now also JP2.1 (A)
Changed lines of the file:
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@@
 	(wire
 		(pts
-			(xy 219.71 33.02) (xy 231.14 33.02)
+			(xy 219.71 33.02) (xy 236.22 33.02)
 		)
 		(stroke
@@
 	(wire
 		(pts
-			(xy 231.14 19.05) (xy 158.75 19.05)
+			(xy 158.75 19.05) (xy 236.22 19.05)
 		)
 		(stroke
@@
 	(wire
 		(pts
-			(xy 231.14 33.02) (xy 231.14 24.13)
+			(xy 110.49 27.94) (xy 120.65 27.94)
 		)
 		(stroke
@@
 	(wire
 		(pts
-			(xy 110.49 27.94) (xy 120.65 27.94)
+			(xy 17.78 73.66) (xy 26.67 73.66)
 		)
 		(stroke
@@
 	(wire
 		(pts
-			(xy 17.78 73.66) (xy 26.67 73.66)
+			(xy 46.99 73.66) (xy 55.88 73.66)
 		)
 		(stroke
@@
 	(wire
 		(pts
-			(xy 46.99 73.66) (xy 55.88 73.66)
+			(xy 107.95 105.41) (xy 100.33 105.41)
 		)
 		(stroke
@@
 	(wire
 		(pts
-			(xy 107.95 105.41) (xy 100.33 105.41)
+			(xy 90.17 113.03) (xy 90.17 128.27)
 		)
 		(stroke
@@
 	(wire
 		(pts
-			(xy 90.17 113.03) (xy 90.17 128.27)
+			(xy 236.22 33.02) (xy 236.22 31.75)
 		)
 		(stroke
@@
 	)
 	(symbol
+		(lib_id "Jumper:Jumper_3_Bridged12")
+		(at 236.22 25.4 90)
+		(unit 1)
+		(exclude_from_sim yes)
+		(in_bom no)
+		(on_board yes)
+		(dnp no)
+		(fields_autoplaced yes)
+		(property "Reference" "JP2"
+			(at 233.68 24.1299 90)
+			(effects
+				(font
+					(size 1.27 1.27)
+				)
+				(justify left)
+			)
+		)
+		(property "Value" "5V_DIR"
+			(at 233.68 26.6699 90)
+			(effects
+				(font
+					(size 1.27 1.27)
+				)
+				(justify left)
+			)
+		)
+		(property "Footprint" "Jumper:SolderJumper-3_P1.3mm_Bridged2Bar12_RoundedPad1.0x1.5mm"
+			(at 236.22 25.4 0)
+			(effects
+				(font
+					(size 1.27 1.27)
+				)
+				(hide yes)
+			)
+		)
+		(property "Datasheet" "~"
+			(at 236.22 25.4 0)
+			(effects
+				(font
+					(size 1.27 1.27)
+				)
+				(hide yes)
+			)
+		)
+		(property "Description" "Jumper, 3-pole, pins 1+2 closed/bridged"
+			(at 236.22 25.4 0)
+			(effects
+				(font
+					(size 1.27 1.27)
+				)
+				(hide yes)
+			)
+		)
+		(pin "2"
+		)
+		(pin "3"
+		)
+		(pin "1"
+		)
+		(instances
+			(project ""
+				(path "/e4d6926a-1a8b-424d-97c4-66b6ad87e4ac/77dfbe0c-d674-478a-bf0e-cfa040fb2e8f"
+					(reference "JP2")
+					(unit 1)
+				)
+			)
+		)
+	)
+	(symbol
 		(lib_id "liebler_SEMICONDUCTORS:IP5306_I2C")
 		(at 179.07 36.83 0)
@@
 	)
 	(symbol
-		(lib_id "Switch:SW_Push_SPDT")
-		(at 236.22 21.59 180)
-		(unit 1)
-		(exclude_from_sim no)
-		(in_bom yes)
-		(on_board yes)
-		(dnp no)
-		(fields_autoplaced yes)
-		(property "Reference" "SW4"
-			(at 236.22 12.7 0)
-			(effects
-				(font
-					(size 1.27 1.27)
-				)
-			)
-		)
-		(property "Value" "5V DIR"
-			(at 236.22 15.24 0)
-			(effects
-				(font
-					(size 1.27 1.27)
-				)
-			)
-		)
-		(property "Footprint" "liebler_MECH:Switch_SS12D00"
-			(at 236.22 21.59 0)
-			(effects
-				(font
-					(size 1.27 1.27)
-				)
-				(hide yes)
-			)
-		)
-		(property "Datasheet" "~"
-			(at 236.22 21.59 0)
-			(effects
-				(font
-					(size 1.27 1.27)
-				)
-				(hide yes)
-			)
-		)
-		(property "Description" "Momentary Switch, single pole double throw"
-			(at 236.22 21.59 0)
-			(effects
-				(font
-					(size 1.27 1.27)
-				)
-				(hide yes)
-			)
-		)
-		(pin "3"
-		)
-		(pin "2"
-		)
-		(pin "1"
-		)
-		(instances
-			(project ""
-				(path "/e4d6926a-1a8b-424d-97c4-66b6ad87e4ac/77dfbe0c-d674-478a-bf0e-cfa040fb2e8f"
-					(reference "SW4")
-					(unit 1)
-				)
-			)
-		)
-	)
-	(symbol
 		(lib_id "Device:C")
 		(at 20.32 113.03 180)
@@
 	(symbol
 		(lib_id "power:+5V")
-		(at 241.3 21.59 270)
+		(at 240.03 25.4 270)
 		(unit 1)
 		(exclude_from_sim no)
@@
 		(fields_autoplaced yes)
 		(property "Reference" "#PWR037"
-			(at 237.49 21.59 0)
+			(at 236.22 25.4 0)
 			(effects
 				(font
@@
 		)
 		(property "Value" "+5V"
-			(at 245.11 21.5899 90)
+			(at 243.84 25.3999 90)
 			(effects
 				(font
@@
 		)
 		(property "Footprint" ""
-			(at 241.3 21.59 0)
+			(at 240.03 25.4 0)
 			(effects
 				(font
@@
 		)
 		(property "Datasheet" ""
-			(at 241.3 21.59 0)
+			(at 240.03 25.4 0)
 			(effects
 				(font
@@
 		)
 		(property "Description" "Power symbol creates a global label with name \"+5V\""
-			(at 241.3 21.59 0)
+			(at 240.03 25.4 0)
 			(effects
 				(font

Commit message: Minor improments on pcb
Parts:
- J8: footprint liebler_CONN:USB_C_Receptacle_HRO_TYPE-C-31-M-12_IMPROVED -> liebler_CONN:USB_C_Receptacle_HRO_TYPE-C-31-M-12_smaller
Changed lines of the file:
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@@
 			)
 		)
-		(property "Footprint" "liebler_CONN:USB_C_Receptacle_HRO_TYPE-C-31-M-12_IMPROVED"
+		(property "Footprint" "liebler_CONN:USB_C_Receptacle_HRO_TYPE-C-31-M-12_smaller"
 			(at 29.21 36.83 0)
 			(effects
