File: labathome_pcb/psu.kicad_sch (KiCad schematic)
At the start: 38 parts, among them J8 POWER, J9 Barrel_Jack_Switch, SW5 POWER, U11 AMS1117, U18 TPS2116DRL, U2 IP5306_I2C, U27 TPS54202DDC

Commit message: Minor changes
Parts:
- C1, C4, C80: MPN (none) -> CGA0805X5R106K350MT; Manufacturer (none) -> HRE
- C28, C29, C30, C31, C7, C83, C84: MPN (none) -> CL10A226MP8NUNE; Manufacturer (none) -> Samsung Electro-Mechanics
- C41, C43: MPN (none) -> CL05A475MP5NRNC; Manufacturer (none) -> Samsung Electro-Mechanics
- C42, C44: MPN (none) -> CL05A105KA5NQNC; Manufacturer (none) -> Samsung Electro-Mechanics
- C79, C81: MPN (none) -> CC0603KRX7R9BB104; Manufacturer (none) -> YAGEO
- C82: MPN (none) -> CC0402JRNPO9BN560; Manufacturer (none) -> YAGEO
- J8: value POWER -> USB STM32; MPN (none) -> TYPE-C-31-M-12; Manufacturer (none) -> Korean Hroparts Elec
- J9: MPN (none) -> DC-005 2.0; Manufacturer (none) -> BOOMELE(Boom Precision Elec)
- L1: value 1u -> 1uH; MPN (none) -> FXL0630-1R0-M; Manufacturer (none) -> cjiang (Changjiang Microelectronics Tech)
- L4: value 10u -> 10uH; MPN (none) -> FXL0630-100-M; Manufacturer (none) -> cjiang (Changjiang Microelectronics Tech)
- R28, R3, R47, R7: MPN (none) -> 0603WAF100KT5E; Manufacturer (none) -> UNI-ROYAL(Uniroyal Elec)
- R4, R60, R72: MPN (none) -> 0201WMF1002TEE; Manufacturer (none) -> UNI-ROYAL(Uniroyal Elec)
- R48, R73: MPN (none) -> 0402WGF3301TCE; Manufacturer (none) -> UNI-ROYAL(Uniroyal Elec)
- R59: MPN (none) -> 0201WMF1003TEE; Manufacturer (none) -> UNI-ROYAL(Uniroyal Elec)
- SW5: MPN (none) -> TS-1095E-A6B3-D2; Manufacturer (none) -> Yuandi
- U11: MPN (none) -> AMS1117-3.3; Manufacturer (none) -> Advanced Monolithic Systems
- U18: MPN (none) -> TPS2116DRLR; Manufacturer (none) -> Texas Instruments
- U2: MPN (none) -> INJOINIC IP5306-I2C; Manufacturer (none) -> INJOINIC
- U27: MPN (none) -> TPS54202DDCR; Manufacturer (none) -> Texas Instruments

Commit message: Labathome PCB -> KICAD 9
Parts:
- renumbered J8 to J13
Changed lines of the file:
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@@
 (kicad_sch
-	(version 20231120)
+	(version 20250114)
 	(generator "eeschema")
-	(generator_version "8.0")
+	(generator_version "9.0")
 	(paper "A4")
 	(title_block
@@
 		(company "Klaus Liebler")
 	)
+	(rectangle
+		(start 99.06 15.24)
+		(end 252.73 62.23)
+		(stroke
+			(width 0)
+			(type default)
+		)
+		(fill
+			(type none)
+		)
+	)
+	(rectangle
+		(start 13.97 15.24)
+		(end 97.79 62.23)
+		(stroke
+			(width 0)
+			(type default)
+		)
+		(fill
+			(type none)
+		)
+	)
+	(rectangle
+		(start 64.77 66.04)
+		(end 96.52 83.82)
+		(stroke
+			(width 0)
+			(type default)
+		)
+		(fill
+			(type none)
+		)
+	)
+	(rectangle
+		(start 13.97 88.9)
+		(end 153.67 130.81)
+		(stroke
+			(width 0)
+			(type default)
+		)
+		(fill
+			(type none)
+		)
+	)
+	(text "USB PD"
+		(exclude_from_sim no)
+		(at 13.97 15.24 0)
+		(effects
+			(font
+				(size 1.27 1.27)
+			)
+			(justify left bottom)
+		)
+	)
+	(text "Barrel Jack 24V"
+		(exclude_from_sim no)
+		(at 64.77 66.04 0)
+		(effects
+			(font
+				(size 1.27 1.27)
+			)
+			(justify left bottom)
+		)
+	)
+	(text "5V->3V3"
+		(exclude_from_sim no)
+		(at 13.97 66.04 0)
+		(effects
+			(font
+				(size 1.27 1.27)
+			)
+			(justify left bottom)
+		)
+	)
+	(text "Battery"
+		(exclude_from_sim no)
+		(at 99.314 14.986 0)
+		(effects
+			(font
+				(size 1.27 1.27)
+			)
+			(justify left bottom)
+		)
+	)
+	(text "PSU"
+		(exclude_from_sim no)
+		(at 13.97 88.9 0)
+		(effects
+			(font
+				(size 1.27 1.27)
+			)
+			(justify left bottom)
+		)
+	)
 	(junction
 		(at 194.31 43.18)
@@
 		)
 	)
-	(rectangle
-		(start 99.06 15.24)
-		(end 252.73 62.23)
-		(stroke
-			(width 0)
-			(type default)
-		)
-		(fill
-			(type none)
-		)
-	)
-	(rectangle
-		(start 13.97 15.24)
-		(end 97.79 62.23)
-		(stroke
-			(width 0)
-			(type default)
-		)
-		(fill
-			(type none)
-		)
-	)
-	(rectangle
-		(start 64.77 66.04)
-		(end 96.52 83.82)
-		(stroke
-			(width 0)
-			(type default)
-		)
-		(fill
-			(type none)
-		)
-	)
-	(rectangle
-		(start 13.97 88.9)
-		(end 153.67 130.81)
-		(stroke
-			(width 0)
-			(type default)
-		)
-		(fill
-			(type none)
-		)
-	)
-	(text "USB PD"
-		(exclude_from_sim no)
-		(at 13.97 15.24 0)
-		(effects
-			(font
-				(size 1.27 1.27)
-			)
-			(justify left bottom)
-		)
-	)
-	(text "Barrel Jack 24V"
-		(exclude_from_sim no)
-		(at 64.77 66.04 0)
-		(effects
-			(font
-				(size 1.27 1.27)
-			)
-			(justify left bottom)
-		)
-	)
-	(text "5V->3V3"
-		(exclude_from_sim no)
-		(at 13.97 66.04 0)
-		(effects
-			(font
-				(size 1.27 1.27)
-			)
-			(justify left bottom)
-		)
-	)
-	(text "Battery"
-		(exclude_from_sim no)
-		(at 99.314 14.986 0)
-		(effects
-			(font
-				(size 1.27 1.27)
-			)
-			(justify left bottom)
-		)
-	)
-	(text "PSU"
-		(exclude_from_sim no)
-		(at 13.97 88.9 0)
-		(effects
-			(font
-				(size 1.27 1.27)
-			)
-			(justify left bottom)
-		)
-	)
 	(label "SW"
 		(at 59.69 110.49 0)
@@
 		(on_board yes)
 		(dnp no)
-		(property "Reference" "#FLG0108"
+		(property "Reference" "#FLG02"
 			(at 40.64 19.685 0)
 			(effects
@@
 		(on_board yes)
 		(dnp no)
-		(property "Reference" "J8"
+		(property "Reference" "J13"
 			(at 16.51 17.78 0)
 			(effects
@@
 		(on_board yes)
 		(dnp no)
-		(property "Reference" "#PWR0113"
+		(property "Reference" "#PWR0164"
 			(at 31.75 59.69 0)
 			(effects
