File: labathome_pcb/stepper2209.kicad_sch (KiCad schematic)
At the start: 40 parts, among them J24 K1, J30 K1, J31 K1, U14 TMC2209, U19 TMC2209, U20 TMC2209

Commit message: Optimized PCB
Connections:
- net EXT_CLK renamed STEPPER_DIR1
- net EXT_CS renamed STEPPER_STEP1
- net EXT_IO1 renamed STEPPER_DIR2
- net EXT_IO2 renamed STEPPER_STEP2
- net EXT_MISO renamed STEPPER_UART
- net EXT_MOSI renamed UART3_TX
- net STEPPER_DIR3 renamed LED_WHITE_P
- net STEPPER_STEP3 renamed FAN_DRIVE
Changed lines of the file:
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@@
 		)
 	)
-	(global_label "EXT_MISO"
-		(shape output)
-		(at 68.58 109.22 180)
-		(fields_autoplaced yes)
-		(effects
-			(font
-				(size 1.27 1.27)
-			)
-			(justify right)
-		)
-		(property "Intersheetrefs" "${INTERSHEET_REFS}"
-			(at 56.7049 109.22 0)
+	(global_label "Servo0"
+		(shape input)
+		(at 53.34 127 180)
+		(fields_autoplaced yes)
+		(effects
+			(font
+				(size 1.27 1.27)
+			)
+			(justify right)
+		)
+		(property "Intersheetrefs" "${INTERSHEET_REFS}"
+			(at 43.9444 127 0)
 			(effects
 				(font
@@
 		)
 	)
-	(global_label "EXT_IO1"
-		(shape bidirectional)
+	(global_label "Servo2"
+		(shape input)
 		(at 53.34 132.08 180)
 		(fields_autoplaced yes)
@@
 		)
 		(property "Intersheetrefs" "${INTERSHEET_REFS}"
-			(at 41.805 132.08 0)
+			(at 43.9444 132.08 0)
+			(effects
+				(font
+					(size 1.27 1.27)
+				)
+				(justify right)
+				(hide yes)
+			)
+		)
+	)
+	(global_label "Servo3"
+		(shape input)
+		(at 53.34 134.62 180)
+		(fields_autoplaced yes)
+		(effects
+			(font
+				(size 1.27 1.27)
+			)
+			(justify right)
+		)
+		(property "Intersheetrefs" "${INTERSHEET_REFS}"
+			(at 43.9444 134.62 0)
 			(effects
 				(font
@@
 		)
 	)
+	(global_label "STEPPER_STEP3"
+		(shape output)
+		(at 53.34 138.43 0)
+		(fields_autoplaced yes)
+		(effects
+			(font
+				(size 1.27 1.27)
+			)
+			(justify left)
+		)
+		(property "Intersheetrefs" "${INTERSHEET_REFS}"
+			(at 71.3835 138.43 0)
+			(effects
+				(font
+					(size 1.27 1.27)
+				)
+				(justify left)
+				(hide yes)
+			)
+		)
+	)
 	(global_label "STEPPER_DIR1"
-		(shape input)
+		(shape output)
 		(at 53.34 127 0)
 		(fields_autoplaced yes)
@@
 		)
 	)
-	(global_label "EXT_CS"
-		(shape input)
-		(at 53.34 129.54 180)
-		(fields_autoplaced yes)
-		(effects
-			(font
-				(size 1.27 1.27)
-			)
-			(justify right)
-		)
-		(property "Intersheetrefs" "${INTERSHEET_REFS}"
-			(at 43.5816 129.54 0)
-			(effects
-				(font
-					(size 1.27 1.27)
-				)
-				(justify right)
-				(hide yes)
-			)
-		)
-	)
-	(global_label "EXT_MOSI"
+	(global_label "STEPPER_DIR2"
+		(shape output)
+		(at 53.34 134.62 0)
+		(fields_autoplaced yes)
+		(effects
+			(font
+				(size 1.27 1.27)
+			)
+			(justify left)
+		)
+		(property "Intersheetrefs" "${INTERSHEET_REFS}"
+			(at 69.9322 134.62 0)
+			(effects
+				(font
+					(size 1.27 1.27)
+				)
+				(justify left)
+				(hide yes)
+			)
+		)
+	)
+	(global_label "STEPPER_DIR3"
+		(shape output)
+		(at 53.34 140.97 0)
+		(fields_autoplaced yes)
+		(effects
+			(font
+				(size 1.27 1.27)
+			)
+			(justify left)
+		)
+		(property "Intersheetrefs" "${INTERSHEET_REFS}"
+			(at 69.9322 140.97 0)
+			(effects
+				(font
+					(size 1.27 1.27)
+				)
+				(justify left)
+				(hide yes)
+			)
+		)
+	)
+	(global_label "STEPPER_STEP1"
+		(shape input)
+		(at 35.56 62.23 180)
+		(fields_autoplaced yes)
+		(effects
+			(font
+				(size 1.27 1.27)
+			)
+			(justify right)
+		)
+		(property "Intersheetrefs" "${INTERSHEET_REFS}"
+			(at 17.5165 62.23 0)
+			(effects
+				(font
+					(size 1.27 1.27)
+				)
+				(justify right)
+				(hide yes)
+			)
+		)
+	)
+	(global_label "STEPPER_STEP1"
+		(shape output)
+		(at 53.34 129.54 0)
+		(fields_autoplaced yes)
+		(effects
+			(font
+				(size 1.27 1.27)
+			)
+			(justify left)
+		)
+		(property "Intersheetrefs" "${INTERSHEET_REFS}"
+			(at 71.3835 129.54 0)
+			(effects
+				(font
+					(size 1.27 1.27)
+				)
+				(justify left)
+				(hide yes)
+			)
+		)
+	)
+	(global_label "STEPPER_EN"
+		(shape input)
+		(at 210.82 71.12 180)
+		(fields_autoplaced yes)
+		(effects
+			(font
+				(size 1.27 1.27)
+			)
+			(justify right)
+		)
+		(property "Intersheetrefs" "${INTERSHEET_REFS}"
+			(at 196.1026 71.12 0)
+			(effects
+				(font
+					(size 1.27 1.27)
+				)
+				(justify right)
+				(hide yes)
+			)
+		)
+	)
+	(global_label "LED_WHITE_P"
+		(shape input)
+		(at 53.34 140.97 180)
+		(fields_autoplaced yes)
+		(effects
+			(font
+				(size 1.27 1.27)
+			)
+			(justify right)
+		)
+		(property "Intersheetrefs" "${INTERSHEET_REFS}"
+			(at 38.1992 140.97 0)
+			(effects
+				(font
+					(size 1.27 1.27)
+				)
+				(justify right)
+				(hide yes)
+			)
+		)
+	)
+	(global_label "FAN_DRIVE"
+		(shape input)
+		(at 53.34 138.43 180)
+		(fields_autoplaced yes)
+		(effects
+			(font
+				(size 1.27 1.27)
+			)
+			(justify right)
+		)
+		(property "Intersheetrefs" "${INTERSHEET_REFS}"
+			(at 40.4971 138.43 0)
+			(effects
+				(font
+					(size 1.27 1.27)
+				)
+				(justify right)
+				(hide yes)
+			)
+		)
+	)
+	(global_label "UART3_TX"
 		(shape input)
 		(at 68.58 116.84 180)
@@
 		)
 		(property "Intersheetrefs" "${INTERSHEET_REFS}"
-			(at 56.7049 116.84 0)
-			(effects
-				(font
-					(size 1.27 1.27)
-				)
-				(justify right)
-				(hide yes)
-			)
-		)
-	)
-	(global_label "EXT_IO2"
-		(shape bidirectional)
-		(at 53.34 134.62 180)
-		(fields_autoplaced yes)
-		(effects
-			(font
-				(size 1.27 1.27)
-			)
-			(justify right)
-		)
-		(property "Intersheetrefs" "${INTERSHEET_REFS}"
-			(at 41.805 134.62 0)
-			(effects
-				(font
-					(size 1.27 1.27)
-				)
-				(justify right)
-				(hide yes)
-			)
-		)
-	)
-	(global_label "STEPPER_DIR2"
-		(shape input)
-		(at 53.34 132.08 0)
-		(fields_autoplaced yes)
-		(effects
-			(font
-				(size 1.27 1.27)
-			)
-			(justify left)
-		)
-		(property "Intersheetrefs" "${INTERSHEET_REFS}"
-			(at 69.9322 132.08 0)
-			(effects
-				(font
-					(size 1.27 1.27)
-				)
-				(justify left)
-				(hide yes)
-			)
-		)
-	)
-	(global_label "STEPPER_STEP1"
-		(shape input)
-		(at 35.56 62.23 180)
-		(fields_autoplaced yes)
-		(effects
-			(font
-				(size 1.27 1.27)
-			)
-			(justify right)
-		)
-		(property "Intersheetrefs" "${INTERSHEET_REFS}"
-			(at 17.5165 62.23 0)
-			(effects
-				(font
-					(size 1.27 1.27)
-				)
-				(justify right)
-				(hide yes)
-			)
-		)
-	)
-	(global_label "STEPPER_STEP1"
-		(shape input)
-		(at 53.34 129.54 0)
-		(fields_autoplaced yes)
-		(effects
-			(font
-				(size 1.27 1.27)
-			)
-			(justify left)
-		)
-		(property "Intersheetrefs" "${INTERSHEET_REFS}"
-			(at 71.3835 129.54 0)
-			(effects
-				(font
-					(size 1.27 1.27)
-				)
-				(justify left)
-				(hide yes)
-			)
-		)
-	)
-	(global_label "STEPPER_EN"
-		(shape input)
-		(at 210.82 71.12 180)
-		(fields_autoplaced yes)
-		(effects
-			(font
-				(size 1.27 1.27)
-			)
-			(justify right)
-		)
-		(property "Intersheetrefs" "${INTERSHEET_REFS}"
-			(at 196.1026 71.12 0)
+			(at 56.5839 116.84 0)
 			(effects
 				(font
@@
 		)
 	)
-	(global_label "EXT_CLK"
-		(shape input)
-		(at 53.34 127 180)
-		(fields_autoplaced yes)
-		(effects
-			(font
-				(size 1.27 1.27)
-			)
-			(justify right)
-		)
-		(property "Intersheetrefs" "${INTERSHEET_REFS}"
-			(at 42.493 127 0)
+	(global_label "UART3_RX"
+		(shape output)
+		(at 68.58 109.22 180)
+		(fields_autoplaced yes)
+		(effects
+			(font
+				(size 1.27 1.27)
+			)
+			(justify right)
+		)
+		(property "Intersheetrefs" "${INTERSHEET_REFS}"
+			(at 56.2815 109.22 0)
+			(effects
+				(font
+					(size 1.27 1.27)
+				)
+				(justify right)
+				(hide yes)
+			)
+		)
+	)
+	(global_label "Servo1"
+		(shape input)
+		(at 53.34 129.54 180)
+		(fields_autoplaced yes)
+		(effects
+			(font
+				(size 1.27 1.27)
+			)
+			(justify right)
+		)
+		(property "Intersheetrefs" "${INTERSHEET_REFS}"
+			(at 43.9444 129.54 0)
 			(effects
 				(font
@@
 	)
 	(global_label "STEPPER_STEP2"
-		(shape input)
-		(at 53.34 134.62 0)
-		(fields_autoplaced yes)
-		(effects
-			(font
-				(size 1.27 1.27)
-			)
-			(justify left)
-		)
-		(property "Intersheetrefs" "${INTERSHEET_REFS}"
-			(at 71.3835 134.62 0)
-			(effects
-				(font
+		(shape output)
+		(at 53.34 132.08 0)
+		(fields_autoplaced yes)
+		(effects
+			(font
+				(size 1.27 1.27)
+			)
+			(justify left)
+		)
+		(property "Intersheetrefs" "${INTERSHEET_REFS}"
+			(at 71.3835 132.08 0)
+			(effects
+				(font

Commit message: Bus servos
Parts:
- removed R22: 1k, Resistor_SMD:R_0402_1005Metric, symbol Device:R
Connections:
- net +24V renamed 5-24V
- net FAN_DRIVE renamed STEPPER_STEP3
- net LED_WHITE_P renamed STEPPER_DIR3

Commit message: Minor changes
Parts:
- added C102, C103, C104: 22u/35V, Capacitor_SMD:C_0805_2012Metric, symbol Device:C
- C120, C58, C75, C87, C90, C91: MPN (none) -> GRM033R61A104KE15D; Manufacturer (none) -> Murata Electronics
- C68, C76, C86, C89, C92, C98: MPN (none) -> CC0603KRX7R9BB104; Manufacturer (none) -> YAGEO
- C69, C72, C77, C78, C85, C88, C93, C96, C97: value 10u/35V -> 22u/35V; MPN (none) -> CGA0805X5R106K350MT; Manufacturer (none) -> HRE
- C70, C73, C94: MPN (none) -> CL05A225MQ5NSNC; Manufacturer (none) -> Samsung Electro-Mechanics
- C71, C74, C95: MPN (none) -> GRM155R71H223KA12D; Manufacturer (none) -> Murata Electronics
- J24: value K1 -> STEP1; MPN (none) -> XH-4AW; Manufacturer (none) -> BOOMELE(Boom Precision Elec)
- J30: value K1 -> STEP2; MPN (none) -> XH-4AW; Manufacturer (none) -> BOOMELE(Boom Precision Elec)
- J31: value K1 -> STEP3; MPN (none) -> XH-4AW; Manufacturer (none) -> BOOMELE(Boom Precision Elec)
- R79, R80, R83, R84, R87, R88: footprint Resistor_SMD:R_2010_5025Metric -> Resistor_SMD:R_1206_3216Metric; MPN (none) -> 201007F100LT4E; Manufacturer (none) -> UNI-ROYAL(Uniroyal Elec)
- U14, U19, U20: MPN (none) -> TMC2209-LA-T; Manufacturer (none) -> TRINAMIC Motion Control GmbH
Connections:
- net 5-24V: now also C102.2, C103.2, C104.2
- net GND: now also C102.1, C103.1, C104.1

Commit message: Various
Parts:
- C102, C103, C104, C69, C72, C77, C78, C85, C88, C93, C96, C97: MPN CGA0805X5R106K350MT -> CGA0805X5R226M350MT
- R79, R80, R83, R84, R87, R88: MPN 201007F100LT4E -> FRM121WFR100TM; Manufacturer UNI-ROYAL(Uniroyal Elec) -> FOJAN
Connections:
- net GND: now also U14.25 (NC), U19.25 (NC), U20.25 (NC)
Changed lines of the file:
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@@
 			)
 		)
-		(property "MPN" "CGA0805X5R106K350MT"
+		(property "MPN" "CGA0805X5R226M350MT"
 			(at 71.12 29.21 0)
 			(effects
@@
 	)
 	(symbol
+		(lib_name "liebler_SEMICONDUCTORS:TMC2209")
 		(lib_id "liebler_SEMICONDUCTORS:TMC2209")
 		(at 226.06 60.96 0)
@@
 		(pin "26"
 		)
+		(pin "25"
+		)
 		(instances
 			(project "labathome_pcb15"
@@
 	)
 	(symbol
+		(lib_name "liebler_SEMICONDUCTORS:TMC2209")
 		(lib_id "liebler_SEMICONDUCTORS:TMC2209")
 		(at 50.8 59.69 0)
@@
 		(pin "26"
 		)
+		(pin "25"
+		)
 		(instances
 			(project ""
@@
 			)
 		)
-		(property "MPN" "201007F100LT4E"
+		(property "MPN" "FRM121WFR100TM"
 			(at 251.46 85.09 0)
 			(effects
@@
 			)
 		)
-		(property "Manufacturer" "UNI-ROYAL(Uniroyal Elec)"
+		(property "Manufacturer" " FOJAN"
 			(at 251.46 85.09 0)
 			(effects
@@
 			)
 		)
-		(property "MPN" "CGA0805X5R106K350MT"
+		(property "MPN" "CGA0805X5R226M350MT"
 			(at 158.75 30.48 0)
 			(effects
@@
 			)
 		)
-		(property "MPN" "201007F100LT4E"
+		(property "MPN" "FRM121WFR100TM"
 			(at 76.2 83.82 0)
 			(effects
@@
 			)
 		)
-		(property "Manufacturer" "UNI-ROYAL(Uniroyal Elec)"
+		(property "Manufacturer" " FOJAN"
 			(at 76.2 83.82 0)
 			(effects
@@
 			)
 		)
-		(property "MPN" "CGA0805X5R106K350MT"
+		(property "MPN" "CGA0805X5R226M350MT"
 			(at 257.81 30.48 0)
 			(effects
@@
 			)
 		)
-		(property "MPN" "CGA0805X5R106K350MT"
+		(property "MPN" "CGA0805X5R226M350MT"
 			(at 148.59 30.48 0)
 			(effects
@@
 			)
 		)
-		(property "MPN" "CGA0805X5R106K350MT"
+		(property "MPN" "CGA0805X5R226M350MT"
 			(at 129.54 120.65 0)
 			(effects
@@
 			)
 		)
-		(property "MPN" "CGA0805X5R106K350MT"
+		(property "MPN" "CGA0805X5R226M350MT"
 			(at 119.38 120.65 0)
 			(effects
@@
 			)
 		)
-		(property "MPN" "CGA0805X5R106K350MT"
+		(property "MPN" "CGA0805X5R226M350MT"
 			(at 168.91 30.48 0)
 			(effects
@@
 			)
 		)
-		(property "MPN" "201007F100LT4E"
+		(property "MPN" "FRM121WFR100TM"
 			(at 68.58 83.82 0)
 			(effects
@@
 			)
 		)
-		(property "Manufacturer" "UNI-ROYAL(Uniroyal Elec)"
+		(property "Manufacturer" " FOJAN"
 			(at 68.58 83.82 0)
 			(effects
@@
 	)
 	(symbol
+		(lib_name "liebler_SEMICONDUCTORS:TMC2209")
 		(lib_id "liebler_SEMICONDUCTORS:TMC2209")
 		(at 138.43 60.96 0)
@@
 		(pin "26"
 		)
+		(pin "25"
+		)
 		(instances
 			(project "labathome_pcb15"
@@
 			)
 		)
-		(property "MPN" "CGA0805X5R106K350MT"
+		(property "MPN" "CGA0805X5R226M350MT"
 			(at 247.65 30.48 0)
 			(effects
@@
 			)
 		)
-		(property "MPN" "201007F100LT4E"
+		(property "MPN" "FRM121WFR100TM"
 			(at 156.21 85.09 0)
 			(effects
@@
 			)
 		)
-		(property "Manufacturer" "UNI-ROYAL(Uniroyal Elec)"
+		(property "Manufacturer" " FOJAN"
 			(at 156.21 85.09 0)
 			(effects
@@
 			)
 		)
-		(property "MPN" "CGA0805X5R106K350MT"
+		(property "MPN" "CGA0805X5R226M350MT"
 			(at 139.7 120.65 0)
 			(effects
@@
 			)
 		)
-		(property "MPN" "201007F100LT4E"
+		(property "MPN" "FRM121WFR100TM"
 			(at 163.83 85.09 0)
 			(effects
@@
 			)
 		)
-		(property "Manufacturer" "UNI-ROYAL(Uniroyal Elec)"
+		(property "Manufacturer" " FOJAN"
 			(at 163.83 85.09 0)
 			(effects
@@
 			)
 		)
-		(property "MPN" "CGA0805X5R106K350MT"
+		(property "MPN" "CGA0805X5R226M350MT"
 			(at 60.96 29.21 0)
 			(effects
@@
 			)
 		)
-		(property "MPN" "201007F100LT4E"
+		(property "MPN" "FRM121WFR100TM"
 			(at 243.84 85.09 0)
 			(effects
@@
 			)
 		)
-		(property "Manufacturer" "UNI-ROYAL(Uniroyal Elec)"
+		(property "Manufacturer" " FOJAN"
 			(at 243.84 85.09 0)
 			(effects
@@
 			)
 		)
-		(property "MPN" "CGA0805X5R106K350MT"
+		(property "MPN" "CGA0805X5R226M350MT"
 			(at 237.49 30.48 0)
 			(effects
@@
 			)
 		)
-		(property "MPN" "CGA0805X5R106K350MT"
+		(property "MPN" "CGA0805X5R226M350MT"
 			(at 81.28 29.21 0)
 			(effects
