File: labathome_pcb15/psu.kicad_sch (KiCad schematic)
At the start: 21 parts, among them J8 POWER, SW11 PROG 5V POWER, U11 FUSB302BMPX, U24 SRV05, U9 RY8310

Commit message: PCB_v15 wip
Parts:
- removed C17, C58: 1u, Capacitor_SMD:C_1206_3216Metric, symbol Device:C
- removed C19, C32, C33, C35: u1, Capacitor_SMD:C_0603_1608Metric, symbol Device:C
- removed C22, C60: 10u, Capacitor_SMD:C_1206_3216Metric, symbol Device:C
- removed C36: 22u, Capacitor_SMD:C_0603_1608Metric, symbol Device:C
- removed C56, C57: n33, Capacitor_SMD:C_0603_1608Metric, symbol Device:C
- removed JP2: USBC_INT, liebler_CONN:Jumper_Trace_025x150x015, symbol Jumper:Jumper_2_Open
- removed L2: 4u7, Inductor_SMD:L_Abracon_ASPI-0630LR, symbol Device:L
- removed R45: 13k, Resistor_SMD:R_0603_1608Metric, symbol Device:R
- removed R46: 68k, Resistor_SMD:R_0603_1608Metric, symbol Device:R
- removed TP1: TP_INT, TestPoint:TestPoint_THTPad_1.0x1.0mm_Drill0.5mm, symbol Connector:TestPoint
- removed U11: FUSB302BMPX, Package_DFN_QFN:WQFN-14-1EP_2.5x2.5mm_P0.5mm_EP1.45x1.45mm, symbol Interface_USB:FUSB302BMPX
- removed U9: RY8310, Package_TO_SOT_SMD:SOT-23-6, symbol Regulator_Switching:LMR14206
- added BT1: 18650, Battery:BatteryHolder_MPD_BH-18650-PC2, symbol Device:Battery_Cell
- added C1, C4: 10u, Capacitor_SMD:C_0603_1608Metric, symbol Device:C
- added C28, C29, C30, C31, C7, C83, C84: 22u, Capacitor_SMD:C_0603_1608Metric, symbol Device:C
- added C79, C81: u1, Capacitor_SMD:C_0603_1608Metric, symbol Device:C
- added C80: 10u, Capacitor_SMD:C_1206_3216Metric, symbol Device:C
- added C82: 56p, Capacitor_SMD:C_0603_1608Metric, symbol Device:C
- added D1: 25%, LED_SMD:LED_0603_1608Metric, symbol Device:LED
- added D4: 50%, LED_SMD:LED_0603_1608Metric, symbol Device:LED
- added D5: 75%, LED_SMD:LED_0603_1608Metric, symbol Device:LED
- added D6: 100%, LED_SMD:LED_0603_1608Metric, symbol Device:LED
- added J9: Barrel_Jack_Switch, Connector_BarrelJack:BarrelJack_Horizontal, symbol Connector:Barrel_Jack_Switch
- added L1: 1u, Inductor_SMD:L_Abracon_ASPI-0630LR, symbol Device:L
- added L4: 10u, liebler_PASSIVES:L_0630, symbol Device:L
- added R28, R7: 1R, Resistor_SMD:R_0603_1608Metric, symbol Device:R
- added R3: 2R2, Resistor_SMD:R_0603_1608Metric, symbol Device:R
- added R4: 10k, Resistor_SMD:R_0603_1608Metric, symbol Device:R
- added R59: M1, Resistor_SMD:R_0402_1005Metric, symbol Device:R
- added R60: 13k3, Resistor_SMD:R_0402_1005Metric, symbol Device:R
- added SW5: POWER, liebler_MECH:SW_SPST_TL3342_smaller_handsolder, symbol Switch:SW_Push
- added U2: IP5306, Package_SO:HSOP-8-1EP_3.9x4.9mm_P1.27mm_EP2.3x2.3mm_ThermalVias, symbol liebler_SEMICONDUCTORS:IP5306
- added U27: TPS54202DDC, Package_TO_SOT_SMD:SOT-23-6_Handsoldering, symbol Regulator_Switching:TPS54202DDC
Connections:
- net +24V: now also C79.2, C80.2, J9.2, U27.3 (VIN)
- net +5V: now also C28.2, C30.2, C31.2, U2.8 (VOUT)
- net 5Vx: now also C82.2, C83.1, C84.1, L4.1, R59.1
- net GND: now also BT1.2 (-), C1.2, C28.1, C29.2, C30.1, C31.1, C4.2, C7.2, C79.1, C80.1, C83.2, C84.2, J9.1, R60.1, SW5.1, U2.9, U27.1 (GND)
- net SW: now also C81.2, L4.2, U27.2 (SW)
- net USBPD_CC2: now reaches U24.3 (IO2)
- net USBPD_CC2: now also J8.B5 (CC2)
- net USBPD_D+: now reaches J8.A6 (D+)
- net USBPD_D+: now also J8.B6 (D+), U24.1 (IO1)
- net USBPD_D-: now reaches J8.A7 (D-)
- net USBPD_D-: now also J8.B7 (D-), U24.6 (IO4)
- removed net CC1: J8.A5 (CC1), U24.1 (IO1), U24.6 (IO4)
- net CC2 renamed USBPD_CC1
- net USBPD_CC1: now also J8.A5 (CC1); no longer J8.B5 (CC2)
- new net: D5.2 (A), D6.1 (K), U2.3 (LED2)
- new net: D1.1 (K), D4.2 (A), D5.1 (K), D6.2 (A), U2.4 (LED3)
- new net: L1.1, U2.7 (SW)
- new net: D1.2 (A), D4.1 (K), U2.2 (LED1)
- new net: C7.1, R28.2, R7.2, U2.6 (BAT)
- new net: R4.1, U2.5 (KEY)
- new net: R4.2, SW5.2
- new net: C1.1, R3.2
- new net +3V8: BT1.1 (+), C29.1, L1.2, R28.1, R7.1
- new net +5VP: C4.1, R3.1, U2.1 (VIN)
- new net BOOT: C81.1, U27.6 (BOOT)
- new net FB: C82.1, R59.2, R60.2, U27.4 (FB)
- no-connect marks 7 -> 4
Other:
- note added: "PSU"
- moved on the sheet: SW11

Commit message: pcb15 WIP
Parts:
- C81, C82: footprint Capacitor_SMD:C_0603_1608Metric -> Capacitor_SMD:C_0402_1005Metric
Changed lines of the file:
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@@
 		)
 		(instances
-			(project ""
+			(project "labathome_pcb15"
 				(path "/e4d6926a-1a8b-424d-97c4-66b6ad87e4ac/77dfbe0c-d674-478a-bf0e-cfa040fb2e8f"
 					(reference "J9")
@@
 			)
 		)
-		(property "Footprint" "Capacitor_SMD:C_0603_1608Metric"
+		(property "Footprint" "Capacitor_SMD:C_0402_1005Metric"
 			(at 106.9848 154.94 0)
 			(effects
@@
 			)
 		)
-		(property "Footprint" "Capacitor_SMD:C_0603_1608Metric"
+		(property "Footprint" "Capacitor_SMD:C_0402_1005Metric"
 			(at 129.8448 160.02 0)
 			(effects
