File: labathome_pcb15/_autosave-labathome_pcb15.kicad_sch (KiCad schematic)
At the start: 42 parts, among them J11 USB_ESP32, J15 CAN RS 485, J17 Micro_SD_Card_Det1, J21 GPIO, J22 Volts, J6 OneWire, J7 PROG, SW2 YELLOW, SW3 GREEN, SW3 Reset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

Commit message: labathome wip
Parts:
- J6: value OneWire -> I2C
Connections:
- net AO0 is gone; now on net GND: J6.4 (Pin_4)
- net OneWire is gone; now on net SDA: J6.2 (Pin_2)
- net GND: no longer J6.1 (Pin_1)
- net SCL: now also J6.1 (Pin_1)
Changed lines of the file:
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@@
 		)
 	)
-	(label "AO0"
-		(at 24.13 138.43 180)
-		(fields_autoplaced yes)
-		(effects
-			(font
-				(size 1.27 1.27)
-			)
-			(justify right bottom)
-		)
-	)
 	(label "USB+"
 		(at 156.21 26.67 0)
@@
 		)
 	)
-	(global_label "OneWire"
+	(global_label "SCL"
 		(shape bidirectional)
-		(at 24.13 133.35 180)
+		(at 24.13 130.81 180)
 		(fields_autoplaced yes)
 		(effects
@@
 		)
 		(property "Intersheetrefs" "${INTERSHEET_REFS}"
-			(at -73.66 -7.62 0)
+			(at 16.5259 130.81 0)
 			(effects
 				(font
 					(size 1.27 1.27)
 				)
+				(justify right)
 				(hide yes)
 			)
@@
 		)
 	)
+	(global_label "SDA"
+		(shape bidirectional)
+		(at 24.13 133.35 180)
+		(fields_autoplaced yes)
+		(effects
+			(font
+				(size 1.27 1.27)
+			)
+			(justify right)
+		)
+		(property "Intersheetrefs" "${INTERSHEET_REFS}"
+			(at 16.4654 133.35 0)
+			(effects
+				(font
+					(size 1.27 1.27)
+				)
+				(justify right)
+				(hide yes)
+			)
+		)
+	)
 	(global_label "I2C_IRQ"
 		(shape input)
@@
 	(symbol
 		(lib_id "power:GND")
-		(at 24.13 130.81 270)
+		(at 24.13 138.43 270)
 		(unit 1)
 		(exclude_from_sim no)
@@
 		(dnp no)
 		(property "Reference" "#PWR038"
-			(at 17.78 130.81 0)
+			(at 17.78 138.43 0)
 			(effects
 				(font
@@
 		)
 		(property "Value" "GND"
-			(at 20.8788 130.937 90)
+			(at 20.8788 138.557 90)
 			(effects
 				(font
@@
 		)
 		(property "Footprint" ""
-			(at 24.13 130.81 0)
+			(at 24.13 138.43 0)
 			(effects
 				(font
@@
 		)
 		(property "Datasheet" ""
-			(at 24.13 130.81 0)
+			(at 24.13 138.43 0)
 			(effects
 				(font
@@
 		)
 		(property "Description" ""
-			(at 24.13 130.81 0)
+			(at 24.13 138.43 0)
 			(effects
 				(font
@@
 			)
 		)
-		(property "Value" "OneWire"
+		(property "Value" "I2C"
 			(at 31.242 135.8646 0)
 			(effects
