File: labathome_pcb15/_autosave-psu.kicad_sch (KiCad schematic)
At the start: 38 parts, among them J8 POWER, J9 Barrel_Jack_Switch, SW11 PROG 5V POWER, SW5 POWER, U11 AMS1117, U2 IP5306, U24 SRV05, U27 TPS54202DDC

Commit message: labathome wip
Parts:
- added SW4: BATT POWER, liebler_MECH:Switch_SS12D00, symbol Switch:SW_SPDT
Connections:
- net +5V: now also SW4.1 (A); no longer C28.2, C30.2, C31.2, U2.8 (VOUT)
- new net: C28.2, C30.2, C31.2, SW4.2 (B), U2.8 (VOUT)
Changed lines of the file:
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@@
 	)
 	(junction
-		(at 219.71 33.02)
-		(diameter 0)
-		(color 0 0 0 0)
-	)
-	(junction
 		(at 166.37 38.1)
 		(diameter 0)
@@
 	)
 	(junction
+		(at 219.71 33.02)
+		(diameter 0)
+		(color 0 0 0 0)
+	)
+	(junction
 		(at 218.44 35.56)
 		(diameter 0)
@@
 	(wire
 		(pts
+			(xy 246.38 31.75) (xy 226.06 31.75)
+		)
+		(stroke
+			(width 0)
+			(type default)
+		)
+	)
+	(wire
+		(pts
 			(xy 208.28 50.8) (xy 218.44 50.8)
 		)
@@
 	(wire
 		(pts
+			(xy 226.06 31.75) (xy 226.06 33.02)
+		)
+		(stroke
+			(width 0)
+			(type default)
+		)
+	)
+	(wire
+		(pts
 			(xy 80.01 20.32) (xy 80.01 25.4)
 		)
@@
 	(wire
 		(pts
+			(xy 226.06 33.02) (xy 219.71 33.02)
+		)
+		(stroke
+			(width 0)
+			(type default)
+		)
+	)
+	(wire
+		(pts
 			(xy 186.69 33.02) (xy 199.39 33.02)
 		)
@@
 	)
 	(symbol
+		(lib_id "Switch:SW_SPDT")
+		(at 251.46 31.75 0)
+		(unit 1)
+		(exclude_from_sim no)
+		(in_bom yes)
+		(on_board yes)
+		(dnp no)
+		(property "Reference" "SW4"
+			(at 251.46 24.511 0)
+			(effects
+				(font
+					(size 1.27 1.27)
+				)
+			)
+		)
+		(property "Value" "BATT POWER"
+			(at 251.46 36.576 0)
+			(effects
+				(font
+					(size 1.27 1.27)
+				)
+			)
+		)
+		(property "Footprint" "liebler_MECH:Switch_SS12D00"
+			(at 251.46 31.75 0)
+			(effects
+				(font
+					(size 1.27 1.27)
+				)
+				(hide yes)
+			)
+		)
+		(property "Datasheet" "~"
+			(at 251.46 31.75 0)
+			(effects
+				(font
+					(size 1.27 1.27)
+				)
+				(hide yes)
+			)
+		)
+		(property "Description" ""
+			(at 251.46 31.75 0)
+			(effects
+				(font
+					(size 1.27 1.27)
+				)
+				(hide yes)
+			)
+		)
+		(pin "1"
+		)
+		(pin "2"
+		)
+		(pin "3"
+		)
+		(instances
+			(project "labathome_pcb15"
+				(path "/e4d6926a-1a8b-424d-97c4-66b6ad87e4ac/77dfbe0c-d674-478a-bf0e-cfa040fb2e8f"
+					(reference "SW4")
+					(unit 1)
+				)
+			)
+		)
+	)
+	(symbol
 		(lib_id "power:GND")
 		(at 199.39 25.4 180)
@@
 	(symbol
 		(lib_id "power:+5V")
-		(at 219.71 33.02 270)
+		(at 256.54 29.21 270)
+		(mirror x)
 		(unit 1)
 		(exclude_from_sim no)
@@
 		(on_board yes)
 		(dnp no)
-		(fields_autoplaced yes)
 		(property "Reference" "#PWR035"
-			(at 215.9 33.02 0)
+			(at 252.73 29.21 0)
 			(effects
 				(font
@@
 		)
 		(property "Value" "+5V"
-			(at 223.52 33.0199 90)
+			(at 260.35 29.2101 90)
 			(effects
 				(font
@@
 		)
 		(property "Footprint" ""
-			(at 219.71 33.02 0)
+			(at 256.54 29.21 0)
 			(effects
 				(font
@@
 		)
 		(property "Datasheet" ""
-			(at 219.71 33.02 0)
+			(at 256.54 29.21 0)
 			(effects
 				(font
@@
 		)
 		(property "Description" ""
-			(at 219.71 33.02 0)
+			(at 256.54 29.21 0)
 			(effects
 				(font
