File: labathome_pcb15/labathome_pcb15.kicad_pcb (KiCad board)
At the start: 2 copper layers, 100 x 100 mm, 219 parts, among them J1 Fan1, J10 BME280, J11 QWIIC, J12 CCS811, J13 POWER, J2 OneWire, J3 Audio, J4 Fan2, J5 USB_C_Receptacle_USB2.0, J6 PROG, J7 FAN5V, J8 GN 5V RGB GN, J9 OneWire, K1 G6K-2, M1 W5500_mini, Q1 BC817, Q2 IRLML6344, Q3 BC817, Q4 TIP41, Q5 IRLML6344, SW1 Reset, SW2 Prog, SW3 TERM ON, SW4 OFF TERM ON, SW5 POWER, SW6 YELLOW, SW7 RED, SW8 GREEN, SW9 PROG 5V POWER, U1 SN65HVD230, U10 TAS5805M, U11 AMS1117, U12 LM358, U13 DS18B20, U14 BME680, U15 BME280, U16 CCS811, U17 DS18B20, U18 AHT21, U19 BH1750, U2 IP5306, U20 MPU-6050, U21 MSM261D4030H1CPM, U22 AM612, U23 NRF24L01, U24 SRV05, U25 RY8310, U3 AS4950, U4 ESP32-S3-WROOM-1, U5 LM358, U6 L78L15_SOT89, U7 MAX3485, U8 SRV05-4, U9 FUSB302BMPX, X1 FAN_6024, X2 XGZP6897D, X3 Ebyte E32, X4 SIM7080G

Commit message: PCB_v15 wip
Parts:
- removed C54: 1u, Capacitor_SMD:C_0603_1608Metric
- removed C55, C62: 10u, Capacitor_SMD:C_0603_1608Metric
- removed C56: 10n, Capacitor_SMD:C_0603_1608Metric
- removed C57, C58, C61, C63, C64, C71, C72: u1, Capacitor_SMD:C_0603_1608Metric
- removed C59: 2n2, Capacitor_SMD:C_0603_1608Metric
- removed C65, C66: n33, Capacitor_SMD:C_0603_1608Metric
- removed C67, C68: 1u, Capacitor_SMD:C_1206_3216Metric
- removed C69, C70: 10u, Capacitor_SMD:C_1206_3216Metric
- removed C73: 22u, Capacitor_SMD:C_0603_1608Metric
- removed FB3, FB4: 300R3A, Resistor_SMD:R_1206_3216Metric
- removed JP1: Fan2toFan1, Jumper:SolderJumper-2_P1.3mm_Open_RoundedPad1.0x1.5mm
- removed JP2: USBC_INT, liebler_CONN:Jumper_Trace_025x150x015
- removed L2: 4u7, Inductor_SMD:L_Abracon_ASPI-0630LR
- removed R11, R12, R13, R15, R9: 4k7, Resistor_SMD:R_0402_1005Metric
- removed SW2: Prog, liebler_MECH:Button_2x4x3,5_handsolder
- removed TP1: AO1, TestPoint:TestPoint_Pad_2.0x2.0mm
- removed TP2: AO0, TestPoint:TestPoint_Pad_2.0x2.0mm
- removed TP3: SW, TestPoint:TestPoint_THTPad_1.0x1.0mm_Drill0.5mm
- removed TP4: TP_INT, TestPoint:TestPoint_THTPad_1.0x1.0mm_Drill0.5mm
- removed U12: LM358, Package_SO:SOIC-8_3.9x4.9mm_P1.27mm
- removed U14: BME680, Package_LGA:Bosch_LGA-8_3x3mm_P0.8mm_ClockwisePinNumbering
- removed U15: BME280, Package_LGA:Bosch_LGA-8_2.5x2.5mm_P0.65mm_ClockwisePinNumbering
- removed U16: CCS811, liebler_SEMICONDUCTORS:AMS_LGA-10-1EP_2.7x4mm_P0.6mm
- removed U18: AHT21, liebler_SEMICONDUCTORS:AHT21
- removed U19: BH1750, liebler_MODULES:GY-302
- removed U20: MPU-6050, Sensor_Motion:InvenSense_QFN-24_4x4mm_P0.5mm
- removed U25: RY8310, Package_TO_SOT_SMD:SOT-23-6
- removed U9: FUSB302BMPX, Package_DFN_QFN:WQFN-14-1EP_2.5x2.5mm_P0.5mm_EP1.45x1.45mm
- removed X3: Ebyte E32, liebler_MODULES:Ebyte-E32-900T20D
- added C79: u1, Capacitor_SMD:C_0603_1608Metric, B.Cu at (121.5, 62.6)
- added C80: 10u, Capacitor_SMD:C_1206_3216Metric, B.Cu at (122.3, 64.5)
- added C81: u1, Capacitor_SMD:C_0603_1608Metric, B.Cu at (139.2, 63.7)
- added C82: 56p, Capacitor_SMD:C_0603_1608Metric, B.Cu at (133.5, 67.3)
- added C83: 22u, Capacitor_SMD:C_0603_1608Metric, B.Cu at (122.7, 54.8)
- added C84: 22u, Capacitor_SMD:C_0603_1608Metric, B.Cu at (121.2, 54.8)
- added J14: AUX OUT, liebler_CONN:PJ-327A, B.Cu at (200.0, 103.4)
- added J15: CAN RS 485, liebler_CONN:PhoenixContact_MC_1,5_4-G-3.5_1x04_P3.50mm_Horizontal_smallerCourtyard, F.Cu at (192.0, 126.8)
- added J16: Headphones, liebler_CONN:PJ-327A, B.Cu at (200.0, 113.8)
- added J17: Micro_SD_Card_Det1, liebler_MECH:microSD push, B.Cu at (141.9, 146.0)
- added J19: BH1750, Connector_PinSocket_2.54mm:PinSocket_1x06_P2.54mm_Vertical, F.Cu at (111.2, 123.3)
- added J20: CCS811, Connector_PinSocket_2.54mm:PinSocket_1x08_P2.54mm_Vertical, F.Cu at (115.2, 130.7)
- added J21: GPIO, liebler_CONN:PhoenixContact_MC_1,5_4-G-3.5_1x04_P3.50mm_Horizontal_smallerCourtyard, F.Cu at (192.0, 142.2)
- added J22: Volts, liebler_CONN:PhoenixContact_MC_1,5_4-G-3.5_1x04_P3.50mm_Horizontal_smallerCourtyard, F.Cu at (108.0, 57.7)
- added J23: VL53L5x, Connector_PinSocket_2.54mm:PinSocket_1x06_P2.54mm_Vertical, F.Cu at (123.7, 105.9)
- added J25: MPU6050, Connector_PinSocket_2.54mm:PinSocket_1x08_P2.54mm_Vertical, F.Cu at (133.9, 52.0)
- added J27: ADDA, liebler_CONN:PhoenixContact_MC_1,5_4-G-3.5_1x04_P3.50mm_Horizontal_smallerCourtyard, F.Cu at (108.0, 116.2)
- added J28: ???, liebler_CONN:PhoenixContact_MC_1,5_4-G-3.5_1x04_P3.50mm_Horizontal_smallerCourtyard, F.Cu at (108.0, 85.4)
- added J31: Servo1, Connector_PinHeader_2.54mm:PinHeader_1x03_P2.54mm_Vertical, F.Cu at (146.4, 87.0)
- added J32: Servo2, Connector_PinHeader_2.54mm:PinHeader_1x03_P2.54mm_Vertical, F.Cu at (150.0, 87.0)
- added J33: Servo3, Connector_PinHeader_2.54mm:PinHeader_1x03_P2.54mm_Vertical, F.Cu at (153.6, 87.0)
- added L4: 10u, liebler_PASSIVES:L_0630, B.Cu at (119.2, 69.3)
- added LS1: Speaker, Connector_PinHeader_2.00mm:PinHeader_1x02_P2.00mm_Vertical, B.Cu at (183.0, 96.4)
- added LS2: Speaker, liebler_MECH:SPEAKER_2415, B.Cu at (150.0, 102.8)
- added MK1: Mic, liebler_PASSIVES:Microphone_6mm, F.Cu at (183.4, 113.8)
- added R57: 10k, Resistor_SMD:R_0402_1005Metric, B.Cu at (139.1, 133.0)
- added R58: 10k, Resistor_SMD:R_0402_1005Metric, B.Cu at (145.3, 137.7)
- added R59: M1, Resistor_SMD:R_0402_1005Metric, B.Cu at (133.5, 66.0)
- added R60: 13k3, Resistor_SMD:R_0402_1005Metric, B.Cu at (136.0, 67.3)
- added R61: 10k, Resistor_SMD:R_0402_1005Metric, B.Cu at (135.8, 133.0)
- added R62: 10k, Resistor_SMD:R_0402_1005Metric, B.Cu at (152.5, 113.8)
- added R63: 10k, Resistor_SMD:R_0402_1005Metric, B.Cu at (123.2, 88.3)
- added R64: 10k, Resistor_SMD:R_0402_1005Metric, B.Cu at (111.4, 102.1)
- added R65: 10k, Resistor_SMD:R_0402_1005Metric, B.Cu at (122.5, 81.0)
- added R66: 1k, Resistor_SMD:R_0402_1005Metric, B.Cu at (170.9, 109.8)
- added R67: 10k, Resistor_SMD:R_0402_1005Metric, B.Cu at (170.9, 108.8)
- added U27: TPS54202DDC, Package_TO_SOT_SMD:SOT-23-6_Handsoldering, B.Cu at (122.0, 58.7)
- added Y1: 8MHz, Crystal:Crystal_SMD_3225-4Pin_3.2x2.5mm, B.Cu at (137.9, 84.6)
- C1, C11, C17, C2, C3, C4, C41, C42, C43, C44, C45, C46, C47, C48, C5, C50, C6, C60, C7, D2, D3, D7, J11, J13, J7, K1, L1, Q1, Q2, Q3, Q4, Q5, R1, R18, R19, R2, R22, R28, R29, R3, R33, R34, R35, R4, R45, R46, R48, R5, R53, R54, R6, R7, R8, SW3, SW4, U1, U11, U17, U2, U24, U4, U7, U8, X2: moved to B.Cu
- C10, C8: value u1 -> 10p; moved to B.Cu
- C12: value 470u -> 4u7; footprint Capacitor_THT:CP_Radial_D10.0mm_P3.50mm -> Capacitor_SMD:C_0402_1005Metric; moved to B.Cu
- C13: value 4u7 -> 4u7; moved to B.Cu
- C14: value 22u -> 4u7; footprint Capacitor_SMD:C_1210_3225Metric_Pad1.33x2.70mm_HandSolder -> Capacitor_SMD:C_0402_1005Metric; moved to B.Cu
- C15: value u1 -> 4u7; moved to B.Cu
- C16: value u1 -> 1u; footprint Capacitor_SMD:C_0603_1608Metric -> Capacitor_SMD:C_0402_1005Metric; moved to B.Cu
- C18: value 1u -> 220u; footprint Capacitor_SMD:C_0402_1005Metric -> Capacitor_SMD:CP_Elec_6.3x5.4; moved to B.Cu
- C19: value 470u -> 220u; footprint Capacitor_THT:CP_Radial_D10.0mm_P3.50mm -> Capacitor_SMD:CP_Elec_6.3x5.4; moved to B.Cu
- C20: value 22u -> 1u; footprint Capacitor_SMD:C_1210_3225Metric_Pad1.33x2.70mm_HandSolder -> Capacitor_SMD:C_0402_1005Metric; moved to B.Cu
- C21: value u1 -> 4u7; footprint Capacitor_SMD:C_0603_1608Metric -> Capacitor_SMD:C_0402_1005Metric; moved to B.Cu
- C22: value u22 -> 4u7; footprint Capacitor_SMD:C_0603_1608Metric -> Capacitor_SMD:C_0402_1005Metric; moved to B.Cu
- C23, C24, C25: value u22 -> 1u; footprint Capacitor_SMD:C_0603_1608Metric -> Capacitor_SMD:C_0402_1005Metric; moved to B.Cu
- C26, C27, C32, C33: value 2n2/100V -> u1; footprint Capacitor_SMD:C_0603_1608Metric -> Capacitor_SMD:C_0402_1005Metric; moved to B.Cu
- C28, C29, C30, C31: value 2n2/100V -> 22u; moved to B.Cu
- C34, C35: value 22u -> u1; footprint Capacitor_SMD:C_0603_1608Metric -> Capacitor_SMD:C_0402_1005Metric; moved to B.Cu
- C36: value 22u -> 4u7; footprint Capacitor_SMD:C_0603_1608Metric -> Capacitor_SMD:C_0402_1005Metric; moved to B.Cu
- C37: value 22u -> 1u; footprint Capacitor_SMD:C_0603_1608Metric -> Capacitor_SMD:C_0402_1005Metric; moved to B.Cu
- C38: value 10u -> u1; footprint Capacitor_SMD:C_1206_3216Metric -> Capacitor_SMD:C_0603_1608Metric; moved to B.Cu
- C39: value u1 -> 100u; footprint Capacitor_SMD:C_0603_1608Metric -> Capacitor_THT:CP_Radial_D6.3mm_P2.50mm
- C40, C52, C53: footprint Capacitor_SMD:C_0603_1608Metric -> Capacitor_SMD:C_0402_1005Metric; moved to B.Cu
- C49: value u1 -> 10n; footprint Capacitor_SMD:C_0603_1608Metric -> Capacitor_SMD:C_0402_1005Metric; moved to B.Cu
- C51: value u1 -> u1; moved to B.Cu
- C9: value u47 -> 10p; footprint Capacitor_SMD:C_0805_2012Metric -> Capacitor_SMD:C_0402_1005Metric; moved to B.Cu
- D1: value 100% -> 25%; moved to B.Cu
- D4: value 75% -> 50%; moved to B.Cu
- D5: value 50% -> 75%; moved to B.Cu
- D6: value 25% -> 100%; moved to B.Cu
- FB1: value 300R3A -> Bead; footprint Resistor_SMD:R_1206_3216Metric -> Inductor_SMD:L_0805_2012Metric; moved to B.Cu
- FB2: value 300R3A -> 600R; footprint Resistor_SMD:R_1206_3216Metric -> Inductor_SMD:L_0603_1608Metric; moved to B.Cu
- J1: value Fan1 -> HALL; footprint Connector:FanPinHeader_1x03_P2.54mm_Vertical -> liebler_CONN:PhoenixContact_MC_1,5_4-G-3.5_1x04_P3.50mm_Horizontal_smallerCourtyard
- J10: value BME280 -> BMEx80
- J12: value CCS811 -> I2C_v4
- J3: value Audio -> AUX IN; footprint liebler_CONN:PhoenixContact_MC_1,5_4-G-3.5_1x04_P3.50mm_Horizontal_smallerCourtyard -> liebler_CONN:PJ-327A; moved to B.Cu
- J4: value Fan2 -> SCD4x; footprint Connector:FanPinHeader_1x03_P2.54mm_Vertical -> Connector_PinSocket_2.54mm:PinSocket_1x04_P2.54mm_Vertical
- J5: value USB_C_Receptacle_USB2.0 -> USB_ESP32; footprint liebler_CONN:USB_C_Receptacle_HRO_TYPE-C-31-M-12_smaller -> liebler_CONN:USB_C_Receptacle_HRO_TYPE-C-31-M-12_IMPROVED; moved to B.Cu
- J9: value OneWire -> Barrel_Jack_Switch; footprint liebler_CONN:PhoenixContact_MC_1,5_4-G-3.5_1x04_P3.50mm_Horizontal_smallerCourtyard -> Connector_BarrelJack:BarrelJack_Horizontal
- NT1: value Net-Tie_2 -> NetTie_2; footprint NetTie:NetTie-2_SMD_Pad2.0mm -> NetTie:NetTie-2_SMD_Pad0.5mm
- R10, R16: value 10k -> 2k2; moved to B.Cu
- R14: value 22k -> 2k2; moved to B.Cu
- R17: value 22k -> 10k; moved to B.Cu
- R20, R21, R30, R31, R36, R37, R42, R43, R44, R50: footprint Resistor_SMD:R_0603_1608Metric -> Resistor_SMD:R_0402_1005Metric; moved to B.Cu
- R23: value 4k7 -> 0R; moved to B.Cu
- R24: value 68R -> 2k2; footprint Resistor_SMD:R_0603_1608Metric -> Resistor_SMD:R_0402_1005Metric; moved to B.Cu
- R25: value 68R -> M22; footprint Resistor_SMD:R_0603_1608Metric -> Resistor_SMD:R_0402_1005Metric; moved to B.Cu
- R26, R27: value 68R -> 10k; footprint Resistor_SMD:R_0603_1608Metric -> Resistor_SMD:R_0402_1005Metric; moved to B.Cu
- R38: value 22k -> 1k; footprint Resistor_SMD:R_0603_1608Metric -> Resistor_SMD:R_0402_1005Metric; moved to B.Cu
- R39, R52: value 4k7 -> 10k; footprint Resistor_SMD:R_0603_1608Metric -> Resistor_SMD:R_0402_1005Metric; moved to B.Cu
- R40: value 2k2 -> 1k; footprint Resistor_SMD:R_0603_1608Metric -> Resistor_SMD:R_0402_1005Metric; moved to B.Cu
- R41: value 1k -> 10k; footprint Resistor_SMD:R_0603_1608Metric -> Resistor_SMD:R_0402_1005Metric; moved to B.Cu
- R49: value 10k -> k22; footprint Resistor_SMD:R_0603_1608Metric -> Resistor_SMD:R_0402_1005Metric; moved to B.Cu
- R51: value 22k -> 10k; footprint Resistor_SMD:R_0603_1608Metric -> Resistor_SMD:R_0402_1005Metric; moved to B.Cu
- R55: value 68k -> 10k; footprint Resistor_SMD:R_0603_1608Metric -> Resistor_SMD:R_0402_1005Metric; moved to B.Cu
- R56: value 13k -> 10k; footprint Resistor_SMD:R_0603_1608Metric -> Resistor_SMD:R_0402_1005Metric; moved to B.Cu
- SW1: footprint liebler_MECH:Button_2x4x3,5_handsolder -> liebler_MECH:SW_SPST_TL3342_smaller_handsolder
- SW5: footprint Button_Switch_SMD:SW_SPST_TL3342 -> liebler_MECH:SW_SPST_TL3342_smaller_handsolder
- U10: value TAS5805M -> ~; footprint Package_SO:HTSSOP-28-1EP_4.4x9.7mm_P0.65mm_EP2.85x5.4mm_ThermalVias -> Package_DFN_QFN:QFN-32-1EP_5x5mm_P0.5mm_EP3.6x3.6mm_ThermalVias; moved to B.Cu
- U13: moved to F.Cu
- U21: value MSM261D4030H1CPM -> IPS_240_240; footprint liebler_SEMICONDUCTORS:MSM261D4030H1CPM -> liebler_OPTO:IPS_240_240_1.3
- U3: value AS4950 -> DRV8813; footprint Package_SO:SOIC-8-1EP_3.9x4.9mm_P1.27mm_EP2.29x3mm_ThermalVias -> Package_SO:HTSSOP-28-1EP_4.4x9.7mm_P0.65mm_EP2.85x5.4mm_ThermalVias; moved to B.Cu
- U5: value LM358 -> STM32G431C6Ux; footprint Package_SO:SOIC-8_3.9x4.9mm_P1.27mm -> Package_DFN_QFN:QFN-48-1EP_7x7mm_P0.5mm_EP5.6x5.6mm; moved to B.Cu
- U6: value L78L15_SOT89 -> RFM95W-868S2; footprint Package_TO_SOT_SMD:SOT-89-3_Handsoldering -> RF_Module:HOPERF_RFM9XW_THT
- moved SW9 233.2 mm to (111.6, 54.3), turned to 90 degrees
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Connections:
- C10 pad 1: GND -> BL_HALL3
- C10 pad 2: +15V -> GND
- C12 pad 1: +24V -> +3V3
- C12 pad 2: GNDA -> GND
- C14 pad 1: +24V -> +3.3VA
- C15 pad 1: +3V3 -> +5V
- C15 pad 2: GND -> GNDA
- C16 pad 1: +24V -> Net-(U10-AUXOUT1)
- C16 pad 2: GNDA -> Net-(C16-Pad2)
- C17 pad 1: /audioamplifier/AVDD -> Net-(U10-AUXOUT2)
- C17 pad 2: GND -> Net-(C17-Pad2)
- C18 pad 1: /audioamplifier/VR_DIG -> Net-(U10-LHP)
- C18 pad 2: GND -> /audioamplifier/JACK_DETECT
- C19 pad 1: +24V -> Net-(U10-RHP)
- C19 pad 2: GNDA -> Net-(C19-Pad2)
- C20 pad 1: +24V -> Net-(MK1--)
- C20 pad 2: GNDA -> Net-(U10-LMICN)
- C21 pad 1: +24V -> Net-(U10-VREF)
- C22 pad 1: Net-(U10-OUT_A+) -> Net-(U10-MICBIAS)
- C22 pad 2: Net-(U10-BST_A+) -> GNDA
- C23 pad 1: Net-(U10-OUT_A-) -> Net-(MK1-+)
- C23 pad 2: Net-(U10-BST_A-) -> Net-(U10-LMICP)
- C24 pad 1: Net-(U10-OUT_B+) -> Net-(C24-Pad1)
- C24 pad 2: Net-(U10-BST_B+) -> Net-(U10-RAUXIN)
- C25 pad 1: Net-(U10-OUT_B-) -> Net-(C25-Pad1)
- C25 pad 2: Net-(U10-BST_B-) -> Net-(U10-LAUXIN)
- C26 pad 1: OUT_A+ -> +3V3
- C26 pad 2: GNDA -> GND
- C27 pad 1: OUT_A- -> +3V3
- C27 pad 2: GNDA -> GND
- C28 pad 1: OUT_A- -> GND
- C28 pad 2: Net-(C28-Pad2) -> +5V
- C29 pad 1: OUT_B+ -> +3V8
- C29 pad 2: GNDA -> GND
- C30 pad 1: OUT_A+ -> GND
- C30 pad 2: Net-(C30-Pad2) -> +5V
- C31 pad 1: OUT_B+ -> GND
- C31 pad 2: Net-(C31-Pad2) -> +5V
- C32 pad 1: OUT_B- -> +3V3
- C32 pad 2: GNDA -> GND
- C33 pad 1: OUT_B- -> +3V3
- C33 pad 2: Net-(C33-Pad2) -> GND
- C34 pad 1: GND -> +3V3
- C34 pad 2: +5V -> GND
- C35 pad 1: +3V8 -> +3V3
- C36 pad 1: GND -> +3V3
- C36 pad 2: +5V -> GND
- C37 pad 1: GND -> Net-(U5-VDDA)
- C37 pad 2: +5V -> GND
- C38 pad 1: GND -> Net-(U3-CPL)
- C38 pad 2: +24V -> Net-(U3-CPH)
- C39 pad 1: GND -> +24V
- C39 pad 2: +24V -> GND
- C40 pad 2: SW -> BTN_YEL
- C49 pad 1: GND -> Net-(U5-VDDA)
- C49 pad 2: +3V3 -> GND
- C51 pad 1: GND -> Net-(U3-VCP)
- C51 pad 2: +3V3 -> +24V
- C52 pad 2: +3V3 -> BTN_RED
- C53 pad 2: +3V3 -> BTN_GRN
- C8 pad 1: GND -> BL_HALL1
- C8 pad 2: +15V -> GND
- C9 pad 1: +24V -> BL_HALL2
- D2 pad 1: CANH -> CANL
- D2 pad 2: CANL -> CANH
- D3 pad 1: RS485B -> RS485A
- D3 pad 2: RS485A -> RS485B
- FB1 pad 1: Net-(U10-OUT_A+) -> +3.3VA
- FB1 pad 2: OUT_A+ -> +3V3
- FB2 pad 1: Net-(U10-OUT_A-) -> Net-(U5-VDDA)
- FB2 pad 2: OUT_A- -> +3V3
- J1 pad 3: FAN1_SENSE -> Net-(J1-Pin_3)
- J10 pad 5: unconnected-(J10-Pin_5-Pad5) -> GND
- J10 pad 6: unconnected-(J10-Pin_6-Pad6) -> +3V3
- J12 pad 1: +3V3 -> unconnected-(J12-Pin_1-Pad1)
- J12 pad 2: GND -> I2C_IRQ
- J12 pad 3: SCL -> SDA
- J12 pad 4: SDA -> SCL
- J12 pad 5: GND -> +3V3
- J12 pad 6: unconnected-(J12-Pin_6-Pad6) -> GND
- J13 pad A5: /psu/CC1 -> USBPD_CC1
- J13 pad A6: unconnected-(J13-D+-PadA6) -> USBPD_D+
- J13 pad A7: unconnected-(J13-D--PadA7) -> USBPD_D-
- J13 pad B5: /psu/CC2 -> USBPD_CC2
- J13 pad B6: unconnected-(J13-D+-PadB6) -> USBPD_D+
- J13 pad B7: unconnected-(J13-D--PadB7) -> USBPD_D-
- J4 pad 1: Net-(J4-Pin_1) -> GND
- J4 pad 2: /VFAN -> +3V3
- J4 pad 3: unconnected-(J4-Pin_3-Pad3) -> SCL
- J5 pad A4: +5V -> +5P
- J5 pad A9: +5V -> +5P
- J5 pad B4: +5V -> +5P
- J5 pad B9: +5V -> +5P
- J7 pad 2: Net-(J4-Pin_1) -> Net-(J7-Pin_2)
- J9 pad 1: Net-(J9-Pin_1) -> GND
- J9 pad 2: GND -> +24V
- J9 pad 3: GND -> unconnected-(J9-Pad3)
- M1 pad 3: MOSI -> EXT_MOSI
- M1 pad 4: SCLK -> EXT_CLK
- M1 pad 5: CS -> EXT_CS
- M1 pad 6: INT -> EXT_IO1
- M1 pad 7: MISO -> EXT_MISO
- M1 pad 8: RST -> EXT_IO2
- Q2 pad 3: Net-(J4-Pin_1) -> Net-(J7-Pin_2)
- R10 pad 1: Net-(U5B--) -> Net-(J1-Pin_3)
- R10 pad 2: GND -> BL_HALL3
- R14 pad 1: /AO1 -> Net-(J1-Pin_2)
- R14 pad 2: Net-(U5B--) -> BL_HALL2
- R16 pad 1: Net-(U5A--) -> Net-(J1-Pin_1)
- R16 pad 2: GND -> BL_HALL1
- R17 pad 1: /AO0 -> +3V3
- R17 pad 2: Net-(U5A--) -> BL_HALL1
- R23 pad 1: +3V3 -> GNDA
- R23 pad 2: /audioamplifier/ADR -> Net-(MK1--)
- R24 pad 1: Net-(C30-Pad2) -> Net-(U10-MICBIAS)
- R24 pad 2: GNDA -> Net-(MK1-+)
- R25 pad 1: Net-(C28-Pad2) -> +3V3
- R25 pad 2: GNDA -> /audioamplifier/JACK_DETECT
- R26 pad 1: Net-(C31-Pad2) -> Net-(U10-MODE)
- R26 pad 2: GNDA -> GND
- R27 pad 1: Net-(C33-Pad2) -> /audioamplifier/JACK_DETECT
- R38 pad 1: +3V3 -> BTN_RED
- R38 pad 2: SW -> Net-(R38-Pad2)
- R39 pad 1: Net-(R39-Pad1) -> +3V3
- R39 pad 2: SW -> BTN_RED
- R40 pad 1: Net-(R40-Pad1) -> BTN_GRN
- R40 pad 2: Net-(R39-Pad1) -> Net-(R40-Pad2)
- R41 pad 1: GND -> +3V3
- R41 pad 2: Net-(R40-Pad1) -> BTN_GRN
- R49 pad 1: GND -> Net-(U5-PF1)
- R49 pad 2: Net-(U12A--) -> Net-(R49-Pad2)
- R50 pad 1: GND -> BL_FAULT
- R50 pad 2: AUDIO -> +3V3
- R51 pad 1: Net-(U12B-+) -> +3V3
- R51 pad 2: Net-(U12A--) -> BL_HALL2
- R52 pad 1: Net-(U16-~{RESET}) -> BL_SLEEP
- R54 pad 2: FAN1_SENSE -> EXT_IO2
- R55 pad 1: /psu/5Vx -> Net-(C19-Pad2)
- R55 pad 2: Net-(U25-FB) -> GNDA
- R56 pad 1: GND -> +3V3
- R56 pad 2: Net-(U25-FB) -> uSD_CMD
- SW6 pad S1: Net-(R39-Pad1) -> GND
- SW6 pad S2: Net-(R40-Pad1) -> Net-(R66-Pad2)
- SW7 pad 2: Net-(R40-Pad1) -> Net-(R38-Pad2)
- SW8 pad 1: Net-(R39-Pad1) -> GND
- SW8 pad 2: SW -> Net-(R40-Pad2)
- U10 pad 1: GND -> Net-(U10-LMICP)
- U10 pad 10: SDA1 -> I2S_DAC
- U10 pad 11: SCL1 -> I2S_MCLK
- U10 pad 12: AMP_PDN -> GND
- U10 pad 13: /audioamplifier/AVDD -> +3V3
- U10 pad 14: GNDA -> +3V3
- U10 pad 15: +24V -> unconnected-(U10-CSB/GPIO1-Pad15)
- U10 pad 16: +24V -> SCL
- U10 pad 17: Net-(U10-OUT_B+) -> SDA
- U10 pad 18: Net-(U10-BST_B+) -> Net-(U10-MODE)
- U10 pad 19: GNDA -> Net-(U10-LAUXIN)
- U10 pad 2: +3V3 -> Net-(U10-LMICN)
- U10 pad 20: Net-(U10-OUT_B-) -> Net-(U10-RAUXIN)
- U10 pad 21: Net-(U10-BST_B-) -> Net-(U10-AUXOUT1)
- U10 pad 22: Net-(U10-BST_A-) -> Net-(U10-AUXOUT2)
- U10 pad 23: Net-(U10-OUT_A-) -> Net-(U10-RSPKOUT)
- U10 pad 25: Net-(U10-BST_A+) -> Net-(U10-LSPKOUT)
- U10 pad 26: Net-(U10-OUT_A+) -> +5V
- U10 pad 27: +24V -> Net-(U10-VREF)
- U10 pad 28: +24V -> GNDA
- U10 pad 29: GNDA -> Net-(U10-RHP)
- U10 pad 3: /audioamplifier/ADR -> /audioamplifier/JACK_DETECT
- U10 pad 4: /audioamplifier/VR_DIG -> Net-(U10-LMICP)
- U10 pad 5: GND -> Net-(U10-LMICN)
- U10 pad 6: I2S_LRCLK -> unconnected-(U10-RLIN/GPIO3-Pad6)
- U10 pad 7: I2S_SCLK -> I2S_FS
- U10 pad 8: I2S_SDAT -> I2S_BCLK
- U10 pad 9: unconnected-(U10-SDOUT-Pad9) -> I2S_ADC
- U21 pad 1: +3V3 -> GND
- U21 pad 2: GND -> +3V3
- U21 pad 3: I2S_SCK -> LCD_CLK
- U21 pad 4: I2S_SD -> LCD_DAT
- U21 pad 5: GND -> Net-(U21-RES)
- U21 pad 6: GND -> LCD_DC
- U21 pad 7: GND -> LCD_BACKLIGHT
- U23 pad 3: SPI_IO1 -> EXT_IO1
- U23 pad 4: SPI_IO2 -> EXT_CS
- U23 pad 5: SPI_CLKx -> EXT_CLK
- U23 pad 6: SPI_MOSIx -> EXT_MOSI
- U23 pad 7: SPI_MISO -> EXT_MISO
- U23 pad 8: FAN1_SENSE -> EXT_IO2
- U24 pad 1: /psu/CC1 -> USBPD_D+
- U24 pad 3: unconnected-(U24-IO2-Pad3) -> USBPD_CC2
- U24 pad 4: /psu/CC2 -> USBPD_CC1
- U24 pad 6: /psu/CC1 -> USBPD_D-
- U3 pad 1: GND -> Net-(U3-CPL)
- U3 pad 2: FAN1_DRIVE -> Net-(U3-CPH)
- U3 pad 3: Net-(JP1-B) -> Net-(U3-VCP)
- U3 pad 4: +3V3 -> +24V
- U3 pad 5: +24V -> Net-(J28-Pin_3)
- U3 pad 6: Net-(J1-Pin_1) -> GND
- U3 pad 8: Net-(J1-Pin_2) -> Net-(J28-Pin_2)
- U3 pad 9: GND -> Net-(J28-Pin_1)
- U4 pad 10: 485_DI -> LCD_CLK
- U4 pad 11: MOSI -> LCD_DAT
- U4 pad 12: SCLK -> LCD_DC
- U4 pad 15: 485_DE -> EXT_CS
- U4 pad 16: BUZZER -> EXT_MOSI
- U4 pad 17: RS -> EXT_MISO
- U4 pad 18: ETH_CS -> EXT_CLK
- U4 pad 19: ETH_MOSI -> EXT_IO1
- U4 pad 20: ETH_CLK -> EXT_IO2
- U4 pad 21: ETH_MISO -> I2S_MCLK
- U4 pad 22: ETH_INT -> I2S_DAC
- U4 pad 23: ETH_RST -> I2S_ADC
- U4 pad 24: CSN -> I2S_BCLK
- U4 pad 25: COMMON_RESET -> I2S_FS
- U4 pad 26: BACKLIGHT -> unconnected-(U4-GPIO45-Pad26)
- U4 pad 28: MISO -> unconnected-(U4-SPIIO6/GPIO35/FSPID/SUBSPID-Pad28)
- U4 pad 29: /VOUTB -> unconnected-(U4-SPIIO7/GPIO36/FSPICLK/SUBSPICLK-Pad29)
- U4 pad 30: SDA2 -> unconnected-(U4-SPIDQS/GPIO37/FSPIQ/SUBSPIQ-Pad30)
- U4 pad 31: SCL2 -> unconnected-(U4-GPIO38/FSPIWP/SUBSPIWP-Pad31)
- U4 pad 32: AMP_PDN -> unconnected-(U4-MTCK/GPIO39/CLK_OUT3/SUBSPICS1-Pad32)
- U4 pad 33: /VOUTA -> unconnected-(U4-MTDO/GPIO40/CLK_OUT2-Pad33)
- U4 pad 34: SDA1 -> unconnected-(U4-MTDI/GPIO41/CLK_OUT1-Pad34)
- U4 pad 35: SCL1 -> unconnected-(U4-MTMS/GPIO42-Pad35)
- U4 pad 38: SW1 -> unconnected-(U4-GPIO2/TOUCH2/ADC1_CH1-Pad38)
- U4 pad 39: MON -> unconnected-(U4-GPIO1/TOUCH1/ADC1_CH0-Pad39)
- U4 pad 4: I2S_SDAT -> SDA
- U4 pad 5: I2S_SCLK -> SCL
- U4 pad 6: I2S_LRCLK -> I2C_IRQ
- U4 pad 7: CAN_TX -> uSD_CMD
- U4 pad 8: CAN_RX -> uSD_CLK
- U4 pad 9: 485_RO -> uSD_D0
- U5 pad 1: /AO0 -> +3V3
- U5 pad 2: Net-(U5A--) -> MOVE
- U5 pad 3: /VOUTA -> BTN_RED
- U5 pad 4: GND -> BTN_YEL
- U5 pad 5: /VOUTB -> Net-(U5-PF0)
- U5 pad 6: Net-(U5B--) -> Net-(U5-PF1)
- U5 pad 7: /AO1 -> unconnected-(U5-PG10-Pad7)
- U5 pad 8: +15V -> HEATER
- U6 pad 1: +15V -> GND
- U6 pad 2: GND -> EXT_MISO
- U6 pad 3: +24V -> EXT_MOSI
- U8 pad 5: +5V -> +5P
- X4 pad 2: SPI_MOSIx -> EXT_MOSI
- X4 pad 3: SPI_MISO -> EXT_MISO
- X4 pad 4: SPI_IO1 -> EXT_IO1
- X4 pad 7: SPI_IO2 -> EXT_IO2
Routing:
- net SDA: track 0.00 -> 190.6 mm, vias 0 -> 2
- net SCL: track 0.00 -> 180.3 mm, vias 0 -> 3
- net +5P: track 0.00 -> 120.6 mm, vias 0 -> 4
- net I2C_IRQ: track 0.00 -> 113.0 mm
- net EXT_MISO: track 0.00 -> 103.0 mm
- net EXT_IO2: track 0.00 -> 100.3 mm
- net EXT_MOSI: track 0.00 -> 94.7 mm
- net EXT_CLK: track 0.00 -> 91.0 mm
- net EXT_CS: track 0.00 -> 87.7 mm
- net EXT_IO1: track 0.00 -> 86.4 mm
- net +3V3: track 0.00 -> 77.6 mm
- net HEATER: track 0.00 -> 53.2 mm
- net ADC2_IN4: track 0.00 -> 48.4 mm
- net /USB-: track 0.00 -> 46.7 mm
- net +24V: track 0.00 -> 45.6 mm, vias 0 -> 1
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
Commit message: pcb15 WIP
Parts:
- removed J25: MPU6050, Connector_PinSocket_2.54mm:PinSocket_1x08_P2.54mm_Vertical
- added C54: u1, Capacitor_SMD:C_0402_1005Metric, B.Cu at (121.1, 98.5)
- added C55: u1, Capacitor_SMD:C_0402_1005Metric, B.Cu at (121.1, 97.0)
- added C56: 22u, Capacitor_SMD:C_0603_1608Metric, B.Cu at (121.3, 134.3)
- added C57: u1, Capacitor_SMD:C_0402_1005Metric, B.Cu at (123.3, 134.1)
- added C58: u1, Capacitor_SMD:C_0402_1005Metric, B.Cu at (128.4, 100.7)
- added C59: 1u, Capacitor_SMD:C_0402_1005Metric, B.Cu at (168.4, 58.6)
- added J18: K1, liebler_CONN:PhoenixContact_MC_1,5_4-G-3.5_1x04_P3.50mm_Horizontal_smallerCourtyard, F.Cu at (192.2, 68.5)
- added J24: K1, liebler_CONN:PhoenixContact_MC_1,5_4-G-3.5_1x04_P3.50mm_Horizontal_smallerCourtyard, F.Cu at (192.0, 83.9)
- added R11: 10k, Resistor_SMD:R_0402_1005Metric, B.Cu at (170.2, 85.5)
- added R9: k22, Resistor_SMD:R_0402_1005Metric, B.Cu at (126.7, 135.2)
- added U12: AHT20, liebler_SEMICONDUCTORS:AHT21, B.Cu at (122.1, 136.6)
- added U14: BMP280, Package_LGA:Bosch_LGA-8_2x2.5mm_P0.65mm_ClockwisePinNumbering, B.Cu at (127.9, 102.5)
- added U9: LSM6DS3, Package_LGA:LGA-14_3x2.5mm_P0.5mm_LayoutBorder3x4y, B.Cu at (118.7, 97.4)
- C81, C82: footprint Capacitor_SMD:C_0603_1608Metric -> Capacitor_SMD:C_0402_1005Metric
- D10, D11, D12, D13, D8, D9: footprint liebler_OPTO:LED_PLCC_2835 -> liebler_OPTO:LED_PLCC_2835_Handsoldering
- J12: value I2C_v4 -> TCS34725
- R45, R46: footprint Resistor_SMD:R_0603_1608Metric -> Resistor_SMD:R_0402_1005Metric
- SW7, SW8: footprint liebler_MECH:SW_Push_1P1T_NO_CK_PTS125Sx43PSMTR -> Button_Switch_THT:SW_PUSH-12mm
- moved R29 102.9 mm to (177.6, 87.7), turned to 180 degrees
- moved Q1 99.8 mm to (178.8, 85.2), turned to 0 degrees
- moved D7 97.6 mm to (179.6, 80.9), turned to -90 degrees
- moved K1 60.9 mm to (186.1, 82.0)
- moved U17 54.7 mm to (156.9, 65.4), turned to 90 degrees
- moved C33 27.7 mm to (124.5, 92.2)
- moved C35 27.7 mm to (123.7, 91.0)
- moved C36 27.7 mm to (124.4, 90.0)
- moved U1 22.9 mm to (184.0, 145.6)
- moved D14 22.5 mm to (161.5, 91.7), turned to 0 degrees
- moved D17 21.5 mm to (139.5, 91.7), turned to 0 degrees
- moved R35 20.6 mm to (142.2, 55.6), turned to 90 degrees
- moved C44 18.2 mm to (128.8, 75.9), turned to -90 degrees
- moved C43 17.6 mm to (130.3, 75.9), turned to 90 degrees
- moved Q4 17.3 mm to (144.4, 65.8), turned to 90 degrees
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Connections:
- net Net-(Q5-D) renamed HEATER_SW
- J6 pad 6: PROG_IO0 -> LCD_BACKLIGHT
- K1 pad 2: K3_22 -> K1_12
- K1 pad 3: K3_21 -> K1_11
- K1 pad 4: K3_24 -> K1_14
- K1 pad 5: K3_14 -> K1_24
- K1 pad 6: K3_11 -> K1_21
- K1 pad 7: K3_12 -> K1_22
- R29 pad 2: K3_ON -> Relais
- R32 pad 1: ROT_A -> +3V3
- R32 pad 2: GND -> BRIGHTNESS
- R6 pad 1: PROG_IO0 -> LCD_BACKLIGHT
- U4 pad 21: I2S_MCLK -> LED_RGB
- U4 pad 22: I2S_DAC -> I2S_MCLK
- U4 pad 23: I2S_ADC -> I2S_DAC
- U4 pad 24: I2S_BCLK -> I2S_ADC
- U4 pad 25: I2S_FS -> I2S_BCLK
- U4 pad 26: unconnected-(U4-GPIO45-Pad26) -> I2S_FS
- U4 pad 27: PROG_IO0 -> LCD_BACKLIGHT
- U4 pad 32: unconnected-(U4-MTCK/GPIO39/CLK_OUT3/SUBSPICS1-Pad32) -> 1wire
- U4 pad 33: unconnected-(U4-MTDO/GPIO40/CLK_OUT2-Pad33) -> 485_DI
- U4 pad 34: unconnected-(U4-MTDI/GPIO41/CLK_OUT1-Pad34) -> 485_DE
- U4 pad 35: unconnected-(U4-MTMS/GPIO42-Pad35) -> 485_RO
- U4 pad 38: unconnected-(U4-GPIO2/TOUCH2/ADC1_CH1-Pad38) -> CAN_RX
- U4 pad 39: unconnected-(U4-GPIO1/TOUCH1/ADC1_CH0-Pad39) -> CAN_TX
- U5 pad 10: Servo2 -> HEATER
- U5 pad 11: Servo3 -> Servo1
- U5 pad 25: ADC1_IN11 -> BRIGHTNESS
- U5 pad 26: GPIO_PB13 -> Relais
- U5 pad 27: GPIO_PB14_ADC1_IN5 -> unconnected-(U5-PB14-Pad27)
- U5 pad 8: HEATER -> ROT_A
- U5 pad 9: Servo1 -> ROT_B
Routing:
- net +5V: track 9.66 -> 136.2 mm, vias 0 -> 2
- net 1wire: track 0.00 -> 106.8 mm, vias 0 -> 2
- net SDA: track 190.6 -> 276.2 mm, vias 2 -> 4
- net +24V: track 45.6 -> 130.1 mm, vias 1 -> 0
- net SCL: track 180.3 -> 254.8 mm, vias 3 -> 4
- net Relais: track 0.00 -> 57.7 mm, vias 0 -> 4
- net BRIGHTNESS: track 0.00 -> 50.4 mm, vias 0 -> 3
- net LED_RGB: track 0.00 -> 45.3 mm, vias 0 -> 1
- net MOVE: track 0.00 -> 39.5 mm, vias 0 -> 1
- net ROT_A: track 3.47 -> 42.2 mm
- net GND: track 43.4 -> 81.8 mm, vias 0 -> 1
- net ROT_B: track 1.74 -> 40.0 mm
- net PROG_IO0: track 24.1 -> 0.00 mm
- net /psu/FB: track 1.22 -> 24.1 mm
- net I2C_IRQ: track 113.0 -> 135.1 mm
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Other:
- outline, holes or cut-outs redrawn

Commit message: labathome wip
Parts:
- removed C50: u1, Capacitor_SMD:C_0603_1608Metric
- removed R47: 22R, liebler_PASSIVES:Resistor_100W
- removed R48: 3k3, Resistor_SMD:R_1206_3216Metric
- removed R54, R6: 10k, Resistor_SMD:R_0402_1005Metric
- removed U23: NRF24L01, RF_Module:nRF24L01_Breakout
- removed X2: XGZP6897D, liebler_MODULES:XGZP6897D
- removed X4: SIM7080G, liebler_MODULES:SIM7080G_AND_MODULE
- added J26: Conn_01x06, Connector_PinHeader_2.54mm:PinHeader_1x06_P2.54mm_Vertical, F.Cu at (115.5, 76.3)
- added R12: 1k, Resistor_SMD:R_0603_1608Metric, B.Cu at (145.7, 74.3)
- added R13: 10R, Resistor_SMD:R_1206_3216Metric, B.Cu at (147.2, 62.4)
- added R15: 10R, Resistor_SMD:R_1206_3216Metric, B.Cu at (149.6, 62.5)
- added SW2: OFF TERM ON, liebler_MECH:SW_SPDT_PCM12_handsolder, B.Cu at (196.6, 133.2)
- added U15: NRF24L01, RF_Module:nRF24L01_Breakout, F.Cu at (168.9, 62.5)
- added X3: SIM7080G, liebler_MODULES:SIM7080G_AND_MODULE, F.Cu at (172.5, 68.3)
- C45, C46, C47, C48: footprint Capacitor_SMD:C_0603_1608Metric -> Capacitor_SMD:C_0402_1005Metric
- D1, D4, D5, D6: footprint LED_SMD:LED_0603_1608Metric -> LED_SMD:LED_0805_2012Metric_Pad1.15x1.40mm_HandSolder; moved to F.Cu
- D13: value WHITE -> 1N4007; footprint liebler_OPTO:LED_PLCC_2835_Handsoldering -> Diode_SMD:D_SOD-123; moved to B.Cu
- D14: value WS2812B -> HTR ON; footprint LED_SMD:LED_WS2812B_PLCC4_5.0x5.0mm_P3.2mm -> LED_SMD:LED_0805_2012Metric
- D18: value HTR ON -> WS2812B; footprint LED_SMD:LED_0805_2012Metric -> LED_SMD:LED_WS2812B_PLCC4_5.0x5.0mm_P3.2mm
- D2: value NUP2105 -> PSM712
- D3: value PSM712 -> NUP2105
- D7: value 1N4007 -> WHITE; footprint Diode_SMD:D_SOD-123 -> liebler_OPTO:LED_PLCC_2835_Handsoldering; moved to F.Cu
- FB1: footprint Inductor_SMD:L_0805_2012Metric -> Inductor_SMD:L_0603_1608Metric
- J2: value OneWire -> I2C
- J28: value ??? -> Brushless
- J7: moved to F.Cu
- Q3: value BC817 -> TIP41; footprint Package_TO_SOT_SMD:SOT-23 -> Package_TO_SOT_THT:TO-220-3_Horizontal_TabUp
- Q4: value TIP41 -> BC817; footprint Package_TO_SOT_THT:TO-220-3_Horizontal_TabUp -> Package_TO_SOT_SMD:SOT-23
- R20: value 1k -> K12; footprint Resistor_SMD:R_0402_1005Metric -> Resistor_SMD:R_1206_3216Metric_Pad1.30x1.75mm_HandSolder
- R21: value 1k -> 4k7
- R22: value K12 -> 10k; footprint Resistor_SMD:R_1206_3216Metric_Pad1.30x1.75mm_HandSolder -> Resistor_SMD:R_0402_1005Metric
- R29: footprint Resistor_SMD:R_0603_1608Metric -> Resistor_SMD:R_0402_1005Metric
- R33: value 1k -> 22R; footprint Resistor_SMD:R_0603_1608Metric -> liebler_PASSIVES:Resistor_100W
- R34: value 10R -> 3k3
- R35: value 10R -> 1k; footprint Resistor_SMD:R_1206_3216Metric -> Resistor_SMD:R_0402_1005Metric
- R45: value 1k -> 10k
- R46: value 10k -> K12; footprint Resistor_SMD:R_0402_1005Metric -> Resistor_SMD:R_1206_3216Metric_Pad1.30x1.75mm_HandSolder
- R5: value 4k7 -> 1k
- R8: value K12 -> 1k; footprint Resistor_SMD:R_1206_3216Metric_Pad1.30x1.75mm_HandSolder -> Resistor_SMD:R_0402_1005Metric
- SW4: value OFF TERM ON -> BATT POWER; footprint liebler_MECH:SW_SPDT_PCM12_handsolder -> liebler_MECH:Switch_SS12D00; moved to F.Cu
- U1: value SN65HVD230 -> MAX3485
- U7: value MAX3485 -> SN65HVD230
- moved Q2 128.2 mm to (186.8, 65.6), turned to 0 degrees
- moved R31 124.3 mm to (184.4, 65.9), turned to -90 degrees
- moved R30 121.8 mm to (184.4, 67.8), turned to -90 degrees
- moved J7 97.9 mm to (158.4, 85.8)
- moved R46 75.9 mm to (186.4, 141.6), turned to 180 degrees
- moved R22 73.8 mm to (177.6, 58.2), turned to 180 degrees
- moved SW4 71.4 mm to (131.6, 110.9), turned to 180 degrees
- moved J8 66.0 mm to (134.1, 92.8)
- moved SW5 63.1 mm to (124.2, 119.4), turned to 180 degrees
- moved C29 63.0 mm to (120.3, 120.4), turned to -90 degrees
- moved R28 62.9 mm to (121.1, 116.6), turned to 0 degrees
- moved R7 62.9 mm to (121.1, 118.1), turned to 0 degrees
- moved R42 61.8 mm to (187.3, 120.6), turned to -90 degrees
- moved C7 58.9 mm to (121.9, 120.4), turned to -90 degrees
- moved R20 56.1 mm to (189.5, 133.9)
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Connections:
- net /D10_COOL renamed /actors/D11_COOL
- net /D11_COOL renamed /actors/D13_COOL
- net /D12_COOL renamed /actors/D10_COOL
- net /D14_COOL renamed /actors/D12_COOL
- net BL_IN1 renamed BL_DRV1
- net BL_IN2 renamed BL_DRV2
- net BL_IN3 renamed BL_DRV3
- C11 pad 1: GND -> +3V3
- C11 pad 2: +3V3 -> GND
- C26 pad 1: +3V3 -> GND
- C26 pad 2: GND -> +3V3
- C28 pad 2: +5V -> Net-(SW4-B)
- C3 pad 1: +3V3 -> GND
- C3 pad 2: GND -> +3V3
- C30 pad 2: +5V -> Net-(SW4-B)
- C31 pad 2: +5V -> Net-(SW4-B)
- C4 pad 1: +5VP -> +5P
- D12 pad 1: /D13_COOL -> /actors/D9_COOL
- D13 pad 1: /D9_COOL -> +5V
- D13 pad 2: /D13_COOL -> Net-(D13-A)
- D14 pad 1: +5V -> Net-(D14-K)
- D14 pad 2: Net-(D14-DOUT) -> +24V
- D15 pad 4: Net-(D14-DOUT) -> LED_RGB
- D18 pad 1: Net-(D18-K) -> +5V
- D18 pad 2: +24V -> Net-(D18-DOUT)
- D2 pad 1: CANL -> RS485A
- D2 pad 2: CANH -> RS485B
- D3 pad 1: RS485A -> CANL
- D3 pad 2: RS485B -> CANH
- D7 pad 1: +5V -> /actors/D14_COOL
- D7 pad 2: Net-(D7-A) -> +24V
- D8 pad 2: +24V -> /actors/D14_COOL
- J15 pad 1: unconnected-(J15-Pin_1-Pad1) -> CANH
- J15 pad 2: unconnected-(J15-Pin_2-Pad2) -> CANL
- J15 pad 3: unconnected-(J15-Pin_3-Pad3) -> RS485B
- J15 pad 4: unconnected-(J15-Pin_4-Pad4) -> RS485A
- J18 pad 1: K1_11 -> K1_24
- J18 pad 2: K1_12 -> K1_22
- J18 pad 3: K1_14 -> K1_21
- J18 pad 4: HEATER_SW -> unconnected-(J18-Pin_4-Pad4)
- J2 pad 1: GND -> SCL
- J2 pad 2: OneWire -> SDA
- J2 pad 4: /AO0 -> GND
- J24 pad 1: K1_24 -> K1_11
- J24 pad 2: K1_22 -> K1_12
- J24 pad 3: K1_21 -> K1_14
- J24 pad 4: unconnected-(J24-Pin_4-Pad4) -> HEATER_SW
- J27 pad 3: ADC2_IN3 -> ADC_IN1
- J27 pad 4: ADC2_IN4 -> ADC_IN2
- J6 pad 6: LCD_BACKLIGHT -> BTN_GRN
- J8 pad 1: GND -> +5V
- J8 pad 2: Net-(D17-DOUT) -> Net-(D18-DOUT)
- J8 pad 3: +5V -> GND
- K1 pad 8: Net-(D7-A) -> Net-(D13-A)
- Q1 pad 3: Net-(D7-A) -> Net-(Q1-C)
- Q2 pad 3: Net-(J7-Pin_2) -> HEATER_SW
- Q3 pad 1: Net-(Q3-B) -> Net-(Q1-C)
- Q3 pad 2: GND -> /actors/D9_COOL
- Q3 pad 3: Net-(Q3-C) -> Net-(Q1-B)
- Q4 pad 1: Net-(Q3-C) -> Net-(Q4-B)
- Q4 pad 2: /D9_COOL -> GND
- Q4 pad 3: Net-(Q3-B) -> Net-(D13-A)
- Q5 pad 3: HEATER_SW -> Net-(J7-Pin_2)
- R20 pad 1: RS485B -> RS485A
- R20 pad 2: GND -> Net-(SW2-A)
- R21 pad 1: +3V3 -> Net-(U7-Rs)
- R21 pad 2: RS485A -> GND
- R22 pad 1: RS485A -> +3V3
- R22 pad 2: Net-(SW4-A) -> EXT_IO2
- R29 pad 1: Net-(Q1-B) -> Net-(Q4-B)
- R3 pad 1: +5VP -> +5P
- R30 pad 2: FAN2_DRIVE -> HEATER
- R33 pad 1: Net-(Q3-C) -> +24V
- R33 pad 2: LED_WHITE_P -> HEATER_SW
- R34 pad 1: Net-(Q3-B) -> Net-(D14-K)
- R34 pad 2: GND -> HEATER_SW
- R35 pad 1: Net-(Q3-B) -> Net-(Q5-G)
- R35 pad 2: GND -> FAN2_DRIVE
- R45 pad 1: Net-(Q5-G) -> GND
- R45 pad 2: HEATER -> Net-(Q5-G)
- R46 pad 1: GND -> Net-(SW3-A)
- R46 pad 2: Net-(Q5-G) -> CANH
- R5 pad 1: Net-(U1-Rs) -> RS485B
- R66 pad 1: BTN_YEL -> Net-(R66-Pad1)
- R66 pad 2: Net-(R66-Pad2) -> BTN_YEL
- R8 pad 1: Net-(SW3-A) -> +3V3
- R8 pad 2: CANH -> RS485A
- SW4 pad 1: Net-(SW4-A) -> +5V
- SW4 pad 2: RS485B -> Net-(SW4-B)
- SW4 pad 3: RS485B -> unconnected-(SW4-C-Pad3)
- SW6 pad S1: GND -> Net-(R66-Pad1)
- SW6 pad S2: Net-(R66-Pad2) -> GND
- U1 pad 1: CAN_TX -> 485_RO
- U1 pad 2: GND -> 485_DE
- U1 pad 3: +3V3 -> 485_DE
- U1 pad 4: CAN_RX -> 485_DI
- U1 pad 5: unconnected-(U1-Vref-Pad5) -> GND
- U1 pad 6: CANL -> RS485A
- U1 pad 7: CANH -> RS485B
- U1 pad 8: Net-(U1-Rs) -> +3V3
- U2 pad 1: +5VP -> +5P
- U2 pad 8: +5V -> Net-(SW4-B)
- U24 pad 1: USBPD_D+ -> USBPD_CC1
- U24 pad 3: USBPD_CC2 -> USBPD_D-
- U24 pad 4: USBPD_CC1 -> USBPD_D+
- U24 pad 6: USBPD_D- -> USBPD_CC2
- U4 pad 27: LCD_BACKLIGHT -> BTN_GRN
- U4 pad 31: unconnected-(U4-GPIO38/FSPIWP/SUBSPIWP-Pad31) -> LCD_BACKLIGHT
- U5 pad 10: HEATER -> Servo1
- U5 pad 11: Servo1 -> Servo2
- U5 pad 14: ADC2_IN3 -> Servo3
- U5 pad 15: ADC2_IN4 -> FAN2_DRIVE
- U5 pad 16: BTN_GRN -> HEATER
- U5 pad 19: ADC2_IN12 -> BRIGHTNESS
- U5 pad 2: MOVE -> BTN_YEL
- U5 pad 22: TIM2_CH3 -> unconnected-(U5-PB10-Pad22)
- U5 pad 24: TIM2_CH4 -> Relais
- U5 pad 25: BRIGHTNESS -> BL_RESET
- U5 pad 26: Relais -> BL_FAULT
- U5 pad 27: unconnected-(U5-PB14-Pad27) -> ADC_IN1
- U5 pad 28: GPIO_PB15_ADC2_IN15 -> ADC_IN2
- U5 pad 3: BTN_RED -> MOVE
- U5 pad 36: JTMS -> SWDIO
- U5 pad 37: JTCK -> SWCLK
- U5 pad 4: BTN_YEL -> PC15
- U5 pad 41: GPIO_PB3 -> unconnected-(U5-PB3-Pad41)
- U5 pad 46: BOOT0 -> BTN_RED
- U5 pad 7: unconnected-(U5-PG10-Pad7) -> STM32_RESET
- U7 pad 1: 485_RO -> CAN_TX
- U7 pad 2: 485_DE -> GND
- U7 pad 3: 485_DE -> +3V3
- U7 pad 4: 485_DI -> CAN_RX
- U7 pad 5: GND -> unconnected-(U7-Vref-Pad5)
- U7 pad 6: RS485A -> CANL
- U7 pad 7: RS485B -> CANH
- U7 pad 8: +3V3 -> Net-(U7-Rs)
Routing:
- net +3V3: track 90.0 -> 551.1 mm, vias 0 -> 23
- net GND: track 81.8 -> 177.7 mm, vias 1 -> 112
- net BTN_YEL: track 0.00 -> 87.4 mm, vias 0 -> 2
- net ADC_IN2: track 0.00 -> 56.7 mm
- net BTN_RED: track 0.00 -> 54.3 mm, vias 0 -> 2
- net ADC_IN1: track 0.00 -> 51.0 mm
- net ADC2_IN4: track 48.4 -> 0.00 mm
- net ROT_A: track 42.2 -> 87.7 mm, vias 0 -> 1
- net ADC2_IN3: track 44.8 -> 0.00 mm
- net +5V: track 136.2 -> 178.8 mm, vias 2 -> 7
- net ROT_B: track 40.0 -> 81.5 mm, vias 0 -> 1
- net FAN2_DRIVE: track 0.00 -> 31.3 mm
- net I2C_IRQ: track 135.1 -> 166.3 mm, vias 0 -> 6
- net /audioamplifier/JACK_DETECT: track 14.3 -> 41.2 mm, vias 1 -> 2
- net EXT_IO1: track 86.4 -> 112.8 mm
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- added copper zone on B.Cu, net GND
- added copper zone on F.Cu, net GND
- added copper zone on B.Cu, net GNDA
- added copper zone on F.Cu, net GNDA

Commit message: labathome15 v0.0.1
Parts:
- added DRAWING1: Polarity, liebler_DRAWINGS:barrel_jack_positive_polarity, F.Cu at (118.5, 67.8)
- added DRAWING2: Glasses, liebler_DRAWINGS:googles, F.Cu at (140.8, 72.2)
- added DRAWING3: Hot, liebler_DRAWINGS:hot, F.Cu at (138.3, 63.2)
- added DRAWING4: qwiic, liebler_DRAWINGS:qwiic, B.Cu at (103.5, 135.8)
- added DRAWING5: Speaker, liebler_DRAWINGS:speaker, F.Cu at (160.4, 107.8)
- D15: value WS2812B -> RGB3
- D16: value WS2812B -> RGB2
- D17: value WS2812B -> RGB1
- D18: value WS2812B -> RGB0
- J26: value Conn_01x06 -> G D C T R 3
- J7: moved to B.Cu
- L1: footprint Inductor_SMD:L_Abracon_ASPI-0630LR -> liebler_PASSIVES:L_0630
- moved C57 15.5 mm to (117.6, 148.5), turned to 90 degrees
- moved U12 11.6 mm to (119.7, 148.0), turned to 0 degrees
- moved R9 11.1 mm to (118.2, 142.4), turned to 0 degrees
- moved C56 10.5 mm to (117.8, 144.2)
- moved R45 6.39 mm to (161.9, 81.5), turned to -90 degrees
- moved R12 4.50 mm to (148.0, 70.5)
- moved Q1 4.47 mm to (148.2, 67.2), turned to 180 degrees
- moved SW1 4.41 mm to (182.5, 145.2), turned to 90 degrees
- moved R35 4.27 mm to (161.0, 81.5), turned to 90 degrees
- moved U13 3.32 mm to (181.8, 124.0)
- moved R42 3.30 mm to (184.5, 122.3)
- moved D13 2.60 mm to (179.1, 83.4)
- moved R1 1.90 mm to (184.1, 148.9), turned to 180 degrees
- moved R25 1.80 mm to (188.2, 118.8), turned to 0 degrees
- moved Q5 1.62 mm to (162.2, 84.3)
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Connections:
- J18 pad 4: unconnected-(J18-Pin_4-Pad4) -> GND
- J21 pad 1: unconnected-(J21-Pin_1-Pad1) -> GND
- J21 pad 2: unconnected-(J21-Pin_2-Pad2) -> GND
- J21 pad 3: unconnected-(J21-Pin_3-Pad3) -> +3V3
- J21 pad 4: unconnected-(J21-Pin_4-Pad4) -> 1wire
Routing:
- net +3V3: track 551.1 -> 565.8 mm, vias 23 -> 43
- net GND: track 177.7 -> 186.2 mm, vias 112 -> 125
- net GNDA: track 8.80 -> 15.6 mm, vias 42 -> 50
- net LED_WHITE_P: track 21.1 -> 27.0 mm
- net FAN2_DRIVE: track 31.3 -> 37.2 mm
- net 1wire: track 110.1 -> 114.2 mm
- net BL_RESET: track 16.1 -> 12.3 mm
- net Net-(U12-VDD): track 6.33 -> 9.45 mm
- net USBPD_CC2: track 31.7 -> 28.9 mm
- net SDA: track 294.6 -> 291.9 mm
- net Net-(J7-Pin_2): track 3.03 -> 5.41 mm
- net Net-(Q5-G): track 4.76 -> 2.48 mm
- net Net-(Q1-B): track 15.4 -> 13.1 mm
- net Net-(Q1-C): track 8.02 -> 5.91 mm
- net Net-(J1-Pin_1): track 0.00 -> 1.96 mm
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- added copper zone on B.Cu, net +3V3
- added copper zone on F.Cu, net +3V3
Other:
- outline, holes or cut-outs redrawn
- board text added: "100%"
- board text added: "1wire"
- board text added: "24V"
- board text added: "25%"
- board text added: "3V3"
- board text added: "485A"
- board text added: "485B"
- board text added: "5"
- board text added: "50%"
- board text added: "5V"
- board text added: "5V from USB PD"
- board text added: "5V from USB Prog"
- board text added: "5V0"
- board text added: "75%"
- board text added: "8-24V"
- board text added: "ADC1"
- board text added: "ADC2"
- board text added: "AUX IN"
- board text added: "AUX OUT"
- board text added: "BAT ON"
- board text added: "BH1750"
- board text added: "BMEx80"
- board text added: "Brightness"
- board text added: "CANH"
- board text added: "CANL"
- board text added: "CCS811"
- board text added: "DAC1"
- board text added: "DAC2"
- board text added: "ESP Prog"
- board text added: "ESP Reset"
- board text added: "G"
- board text added: "GND"
- board text added: "Green Btn"
- board text added: "HA1"
- board text added: "HA2"
- board text added: "HA3"
- board text added: "Headphones"
- board text added: "Heater"
- board text added: "Heater On"
- board text added: "K1.11"
- board text added: "K1.12"
- board text added: "K1.14"
- board text added: "K1.21"
- board text added: "K1.22"
- board text added: "K1.24"
- board text added: "Mic"
- board text added: "MicroSD"
- board text added: "NRF24L01"
- board text added: "PH1"
- board text added: "PH2"
- board text added: "PH3"
- board text added: "PIR Sensor"
- board text added: "RFM95"
- board text added: "RXD"
- board text added: "Red Button"
- board text added: "S"
- board text added: "SCD4x"
- board text added: "SCL"
- board text added: "SDA"
- board text added: "SIM7080"
- board text added: "STM Prog"
- board text added: "SWCLK"
- board text added: "SWDIO"
- board text added: "Speaker"
- board text added: "TCS34725"
- board text added: "TXD"
- board text added: "USB ESP32"
- board text added: "USB PD (STM)"
- board text added: "VL53L5x"
- board text added: "W5500"
- board text added: "WS2812"
- board text added: "Yellow Encoder"
- board text added: "lab@home v15 2024-01-07 Klaus Liebler"
