File: labathome_pcb15/labathome_pcb15.kicad_pcb (KiCad board)
At the start: 2 copper layers, 100 x 100 mm, 229 parts, among them J1 HALL, J10 BMEx80, J11 QWIIC, J12 TCS34725, J13 POWER, J14 AUX OUT, J15 CAN RS 485, J16 Headphones, J17 Micro_SD_Card_Det1, J18 K1, J19 BH1750, J2 I2C, J20 CCS811, J21 GPIO, J22 Volts, J23 VL53L5x, J24 K1, J26 G D C T R 3, J27 ADDA, J28 Brushless, J3 AUX IN, J31 Servo1, J32 Servo2, J33 Servo3, J4 SCD4x, J5 USB_ESP32, J6 PROG, J7 FAN5V, J8 GN 5V RGB GN, J9 Barrel_Jack_Switch, K1 G6K-2, M1 W5500_mini, Q1 BC817, Q2 IRLML6344, Q3 TIP41, Q4 BC817, Q5 IRLML6344, SW1 Reset, SW2 OFF TERM ON, SW3 TERM ON, SW4 BATT POWER, SW5 POWER, SW6 YELLOW, SW7 RED, SW8 GREEN, SW9 PROG 5V POWER, U1 MAX3485, U11 AMS1117, U12 AHT20, U13 DS18B20, U14 BMP280, U15 NRF24L01, U17 DS18B20, U2 IP5306, U21 IPS_240_240, U22 AM612, U24 SRV05, U27 TPS54202DDC, U3 DRV8813, U4 ESP32-S3-WROOM-1, U5 STM32G431C6Ux, U6 RFM95W-868S2, U7 SN65HVD230, U8 SRV05-4, U9 LSM6DS3, X1 FAN_6024, X3 SIM7080G, Y1 8MHz

Commit message: labathome_pcb15 v0.0.2
Parts:
- removed J26: G D C T R 3, Connector_PinHeader_2.54mm:PinHeader_1x06_P2.54mm_Vertical
- added C50: 22p, Capacitor_SMD:C_0402_1005Metric, B.Cu at (140.4, 84.5)
- added C61: u1, Capacitor_SMD:C_0402_1005Metric, B.Cu at (137.8, 82.4)
- added J25: STM Debug, liebler_CONN:JST_SH_BM06B-SRSS-TB_1x06-1MP_P1.00mm_Vertical_handsolder, F.Cu at (126.0, 79.0)
- moved R64 10.4 mm to (130.8, 94.7), turned to 180 degrees
- moved R51 9.30 mm to (130.8, 96.0), turned to 180 degrees
- moved R17 6.01 mm to (130.8, 97.0), turned to 180 degrees
- moved J8 1.93 mm to (134.2, 94.7)
- moved C32 0.72 mm to (125.5, 90.0)
- moved C36 0.72 mm to (125.5, 90.9)
- moved R22 0.70 mm to (177.6, 57.5)
- moved NT1 0.70 mm to (170.2, 97.3)
- moved C24 0.38 mm to (173.9, 91.4)
- moved Y1 0.32 mm to (137.8, 84.6)
- moved C25 0.30 mm to (172.1, 91.4)
- moved FB2 0.27 mm to (126.5, 92.1)
- moved C37 0.21 mm to (127.8, 90.9), turned to 180 degrees
- moved C49 0.21 mm to (127.8, 90.0), turned to 180 degrees
- moved C59 0.10 mm to (168.6, 58.4)
Connections:
- U5 pad 4: PC15 -> unconnected-(U5-PC15-Pad4)
Routing:
- net GND: track 186.2 -> 230.8 mm, vias 125 -> 442
- net +24V: track 152.5 -> 165.3 mm, vias 3 -> 6
- net SWDIO: track 12.5 -> 1.56 mm, vias 0 -> 1
- net +3V3: track 565.8 -> 556.0 mm, vias 43 -> 48
- net SWCLK: track 9.70 -> 0.79 mm, vias 0 -> 1
- net SDA: track 291.9 -> 285.8 mm
- net SCL: track 274.0 -> 268.0 mm
- net UART4_TX: track 8.28 -> 3.09 mm, vias 0 -> 1
- net BL_HALL1: track 26.2 -> 30.2 mm, vias 0 -> 2
- net UART4_RX: track 6.25 -> 2.92 mm, vias 0 -> 1
- net Net-(D18-DOUT): track 3.54 -> 6.19 mm
- net EXT_IO2: track 100.9 -> 98.4 mm
- net K1_14: track 14.8 -> 16.8 mm
- net EXT_MOSI: track 93.9 -> 95.8 mm
- net Net-(C50-Pad2): track 5.11 -> 6.98 mm
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Other:
- board text added: "5V from USB ESP32"
- board text added: "5V from USB STM32 (PD)"
- board text added: "USB STM32 (PD)"
- board text removed: "5V from USB PD"
- board text removed: "5V from USB Prog"
- board text removed: "Heater"
- board text removed: "USB PD (STM)"

Commit message: labathome_pcb15 ready for first review
Parts:
- added D19: INFO, LED_SMD:LED_0805_2012Metric, F.Cu at (118.5, 77.7)
- added R6: k22, Resistor_SMD:R_0402_1005Metric, B.Cu at (183.5, 76.2)
- C61: value u1 -> 22p
- R34: value 3k3 -> k22; footprint Resistor_SMD:R_1206_3216Metric -> Resistor_SMD:R_0402_1005Metric
- moved R34 67.4 mm to (118.8, 74.6), turned to 180 degrees
- moved U17 2.83 mm to (158.1, 62.8), turned to -90 degrees
- moved D12 2.50 mm to (147.5, 57.5)
- moved D7 2.00 mm to (152.5, 58.0)
- moved D10 1.80 mm to (147.5, 73.0)
- moved D9 1.80 mm to (152.5, 73.0)
- moved D14 1.30 mm to (182.1, 77.7)
- moved C61 0.50 mm to (137.3, 82.4)
- moved C50 0.36 mm to (140.1, 84.6)
- moved Y1 0.35 mm to (137.4, 84.6)
- moved R49 0.27 mm to (134.4, 85.2)
Connections:
- D14 pad 2: +24V -> HEATER
- R34 pad 1: Net-(D14-K) -> GND
- R34 pad 2: HEATER_SW -> Net-(D19-K)
- U5 pad 41: unconnected-(U5-PB3-Pad41) -> LED_INFO
Routing:
- net +24V: track 165.3 -> 123.2 mm, vias 6 -> 4
- net LED_INFO: track 0.00 -> 12.6 mm, vias 0 -> 1
- net +3V3: track 556.0 -> 546.2 mm, vias 48 -> 46
- net Net-(D14-K): track 7.73 -> 1.62 mm
- net /actors/D9_COOL: track 5.43 -> 9.85 mm, vias 0 -> 1
- net Net-(D19-K): track 0.00 -> 3.61 mm, vias 0 -> 1
- net HEATER_SW: track 5.94 -> 2.71 mm
- net /actors/D13_COOL: track 3.33 -> 5.25 mm
- net 1wire: track 113.1 -> 114.8 mm
- net HEATER: track 69.4 -> 71.0 mm, vias 2 -> 3
- net /actors/D10_COOL: track 4.53 -> 5.62 mm
- net SDA: track 285.8 -> 286.8 mm
- net GND: track 230.8 -> 231.9 mm, vias 442 -> 438
- net /actors/D11_COOL: track 3.32 -> 4.35 mm
- net /actors/D12_COOL: track 3.33 -> 4.35 mm
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- added copper zone on F.Cu, net /actors/D10_COOL
- added copper zone on F.Cu, net /actors/D11_COOL
- added copper zone on F.Cu, net /actors/D12_COOL
- added copper zone on F.Cu, net /actors/D13_COOL
- added copper zone on F.Cu, net /actors/D14_COOL
- added copper zone on F.Cu, net /actors/D9_COOL
Other:
- board text added: "5V from USB PD"
- board text added: "Green Button"
- board text added: "Heater"
- board text added: "STM32 Prog"
- board text added: "USB STM32+PD"
- board text added: "lab@home v15 2024-07-05 Klaus Liebler For Science /Education / DIY"
- board text removed: "5V from USB STM32 (PD)"
- board text removed: "Green Btn"
- board text removed: "Heater On"
- board text removed: "STM Prog"
- board text removed: "USB STM32 (PD)"
- board text removed: "lab@home v15 2024-01-07 Klaus Liebler"
