File: labathome_pcb15/labathome_pcb15.kicad_pcb (KiCad board)
At the start: 2 copper layers, 100 x 100 mm, 239 parts, among them J1 HALL, J10 BMEx80, J11 QWIIC, J12 TCS34725, J13 POWER, J14 AUX OUT, J15 CAN RS 485, J16 Headphones, J17 Micro_SD_Card_Det1, J18 K1, J19 BH1750, J2 I2C, J20 CCS811, J21 GPIO, J22 Volts, J23 VL53L5x, J24 K1, J26 STDC14, J27 ADDA, J28 Brushless, J3 AUX IN, J31 Servo1, J32 Servo2, J33 Servo3, J4 SCD4x, J5 USB_ESP32, J6 PROG, J7 FAN5V, J8 GN 5V RGB GN, J9 Barrel_Jack_Switch, K1 G6K-2, M1 W5500_mini, Q1 BC817, Q2 IRLML6344, Q3 TIP41, Q4 BC817, Q5 IRLML6344, SW1 Reset, SW10 USBPD ADC2 EXT, SW2 ON RS TERM, SW3 ON CAN TERM, SW4 BATT POWER, SW5 POWER, SW6 YELLOW, SW7 RED, SW8 GREEN, SW9 PROG 5V POWER, U1 MAX3485, U10 NAU8822, U11 AMS1117, U12 AHT20, U13 DS18B20, U14 BMP280, U15 NRF24L01, U17 DS18B20, U2 IP5306, U21 IPS_240_240, U22 AM612, U24 SRV05, U27 TPS54202DDC, U3 DRV8313, U4 ESP32-S3-WROOM-1, U5 STM32G431C6Ux, U6 RFM95W-868S2, U7 SN65HVD230, U8 SRV05-4, U9 LSM6DS3, X1 FAN_6024, X3 SIM7080G, Y1 8MHz/12pF

Commit message: Further improventents in PCB layout
Parts:
- removed JP1: JFS, Jumper:SolderJumper-2_P1.3mm_Bridged2Bar_RoundedPad1.0x1.5mm
- added C25: u1/16V, Capacitor_SMD:C_0402_1005Metric, B.Cu at (134.4, 85.7)
- moved R12 19.4 mm to (133.0, 56.6), turned to 180 degrees
- moved Q1 14.1 mm to (135.9, 56.8), turned to 180 degrees
- moved Q3 13.6 mm to (140.8, 53.0), turned to -90 degrees
- moved R13 13.4 mm to (138.3, 52.8)
- moved R15 13.4 mm to (136.0, 52.8)
- moved U11 13.2 mm to (132.0, 66.9)
- moved C41 13.2 mm to (126.6, 64.1), turned to 0 degrees
- moved C43 12.3 mm to (126.6, 66.4)
- moved C44 12.3 mm to (126.6, 67.4)
- moved C42 11.8 mm to (126.6, 65.1), turned to 180 degrees
- moved R35 4.57 mm to (161.8, 86.5), turned to -90 degrees
- moved R45 3.13 mm to (161.5, 85.1), turned to 0 degrees
- moved Q5 2.20 mm to (162.3, 82.7), turned to 90 degrees
- moved C34 1.00 mm to (133.8, 81.9)
- moved C61 0.68 mm to (137.9, 82.2)
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Connections:
- SW6 pad MP: (no net) -> GND
- U10 pad 7: Net-(JP1-B) -> I2S_FS
- U4 pad 23: I2S_DAC -> I2S_FS
- U4 pad 26: I2S_FS -> I2S_DAC
Routing:
- net GND: track 240.1 -> 461.0 mm, vias 442 -> 429
- net I2S_FS: track 1.88 -> 36.9 mm, vias 0 -> 2
- net Net-(JP1-B): track 30.9 -> 0.00 mm
- net /actors/D9_COOL: track 9.85 -> 0.00 mm, vias 1 -> 0
- net /audioamplifier/JACK_DETECT: track 37.7 -> 45.6 mm
- net GNDA: track 15.2 -> 22.1 mm, vias 99 -> 97
- net +5V: track 180.5 -> 187.1 mm
- net Net-(Q1-C): track 5.37 -> 11.2 mm
- net FAN2_DRIVE: track 37.3 -> 33.0 mm
- net +3V3: track 567.7 -> 571.8 mm, vias 45 -> 61
- net Net-(Q1-B): track 7.75 -> 11.1 mm
- net I2S_DAC: track 36.0 -> 39.3 mm, vias 0 -> 2
- net ROT_B: track 78.2 -> 79.8 mm
- net STM32_RESET: track 0.00 -> 1.39 mm
- net +24V: track 122.5 -> 123.9 mm
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
Commit message: Final PCB as ordered @ JLCPCB
Parts:
- added JP1: Jumper_2_Bridged, Jumper:SolderJumper-2_P1.3mm_Bridged2Bar_Pad1.0x1.5mm, B.Cu at (181.9, 117.8)
- R23: footprint Resistor_SMD:R_0402_1005Metric -> Diode_SMD:D_0805_2012Metric_Pad1.15x1.40mm_HandSolder
- moved C25 12.4 mm to (138.5, 74.0), turned to -90 degrees
- moved R23 0.93 mm to (184.1, 117.8)
- moved R49 0.88 mm to (135.0, 85.4)
- moved C8 0.45 mm to (110.5, 95.7)
- moved R16 0.45 mm to (110.0, 94.3)
- moved Y1 0.40 mm to (138.1, 84.5)
- moved C50 0.40 mm to (140.7, 84.5)
- moved C61 0.15 mm to (138.1, 82.2)
Connections:
- J26 pad 12: unconnected-(J26-Pin_12-Pad12) -> STM32_RESET
Routing:
- net STM32_RESET: track 1.39 -> 25.3 mm, vias 0 -> 2
- net +3V3: track 571.8 -> 574.4 mm
- net Net-(JP1-B): track 3.50 -> 5.86 mm
- net /audioamplifier/JACK_DETECT: track 45.6 -> 46.9 mm
- net Net-(U5-PF0): track 5.62 -> 6.44 mm
- net Net-(C50-Pad2): track 7.02 -> 6.30 mm
- net Net-(U5-PF1): track 1.34 -> 2.04 mm
- net Net-(U10-LMICN): track 30.2 -> 30.7 mm
- net GNDA: vias 97 -> 98

Commit message: lbathome 15.1
Parts:
- removed R65: 10k, Resistor_SMD:R_0402_1005Metric
- removed SW10: USBPD ADC2 EXT, liebler_MECH:SW_SPDT_PCM12_handsolder
- removed Y1: 8MHz/12pF, Crystal:Crystal_SMD_3225-4Pin_3.2x2.5mm
- added C52: u1/50V, Capacitor_SMD:C_0603_1608Metric, B.Cu at (112.0, 90.0)
- added C63: u1/50V, Capacitor_SMD:C_0603_1608Metric, B.Cu at (111.6, 81.6)
- added C64: u1, Capacitor_SMD:C_0603_1608Metric, B.Cu at (103.5, 114.5)
- added J30: Srv4, liebler_CONN:PinHeader_1x03_P2.54mm_Vertical_smallerCourtyard, F.Cu at (153.8, 86.8)
- added J34: STM32 EXT, Connector_PinHeader_2.54mm:PinHeader_2x03_P2.54mm_Vertical, F.Cu at (120.7, 95.3)
- added R38: r1, Resistor_THT:R_Axial_DIN0309_L9.0mm_D3.2mm_P12.70mm_Horizontal, F.Cu at (111.2, 87.1)
- added U16: LM358, Package_SO:SOIC-8_3.9x4.9mm_P1.27mm, B.Cu at (104.5, 110.1)
- C12, C13, C14, C15, C21, C22: value 4u7 -> 4u7
- C50: value 15p -> u1
- C61: value 15p -> 4u7/6V3
- FB2: value 600R -> 600R
- J31: value Servo1 -> Srv1; footprint Connector_PinHeader_2.54mm:PinHeader_1x03_P2.54mm_Vertical -> liebler_CONN:PinHeader_1x03_P2.54mm_Vertical_smallerCourtyard
- J32: value Servo2 -> Srv2; footprint Connector_PinHeader_2.54mm:PinHeader_1x03_P2.54mm_Vertical -> liebler_CONN:PinHeader_1x03_P2.54mm_Vertical_smallerCourtyard
- J33: value Servo3 -> Srv3; footprint Connector_PinHeader_2.54mm:PinHeader_1x03_P2.54mm_Vertical -> liebler_CONN:PinHeader_1x03_P2.54mm_Vertical_smallerCourtyard
- J8: value GN 5V RGB GN -> 3V GN RGB 5V
- R49: value k22 -> 10k; footprint Resistor_SMD:R_0402_1005Metric -> Resistor_SMD:R_0805_2012Metric_Pad1.20x1.40mm_HandSolder
- R52: value 10k -> 22k; footprint Resistor_SMD:R_0402_1005Metric -> Resistor_SMD:R_0805_2012Metric_Pad1.20x1.40mm_HandSolder
- U5: value STM32G431C6Ux -> STM32G431R8Tx; footprint Package_DFN_QFN:QFN-48-1EP_7x7mm_P0.5mm_EP5.6x5.6mm -> Package_QFP:LQFP-64_10x10mm_P0.5mm
- moved R67 46.6 mm to (172.2, 109.5), turned to 180 degrees
- moved R43 36.9 mm to (109.9, 142.2)
- moved U9 35.9 mm to (118.4, 135.3), turned to 0 degrees
- moved C54 34.7 mm to (117.9, 133.3)
- moved R49 34.7 mm to (104.8, 102.6), turned to -90 degrees
- moved C55 32.7 mm to (119.8, 133.3), turned to 0 degrees
- moved R2 32.5 mm to (178.8, 145.6), turned to 90 degrees
- moved G*** 30.0 mm to (182.1, 83.0)
- moved R52 29.6 mm to (103.9, 105.4)
- moved R50 28.7 mm to (108.5, 108.7), turned to -90 degrees
- moved R44 26.8 mm to (120.7, 136.6)
- moved R64 21.4 mm to (111.4, 103.8)
- moved R17 20.1 mm to (110.8, 95.4), turned to 90 degrees
- moved R51 19.8 mm to (111.4, 100.3)
- moved C36 16.8 mm to (137.7, 79.4), turned to 0 degrees
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Connections:
- C50 pad 1: GND -> +3V3
- C50 pad 2: Net-(C50-Pad2) -> GND
- C61 pad 1: GND -> Net-(U3-V3P3)
- C61 pad 2: Net-(U5-PF0) -> GND
- J11 pad MP: (no net) -> GND
- J27 pad 2: DAC1_OUT2 -> DAC1_OUT2x
- J27 pad 4: ADC_IN2_EXT -> ADC_IN2
- J8 pad 2: Net-(D18-DOUT) -> GND
- J8 pad 3: +5V -> Net-(D18-DOUT)
- J8 pad 4: GND -> +5V
- R49 pad 1: Net-(U5-PF1) -> GND
- R49 pad 2: Net-(C50-Pad2) -> Net-(U16A--)
- R50 pad 1: BL_FAULT -> GND
- R50 pad 2: +3V3 -> DAC1_OUT2
- R52 pad 1: BL_SLEEP -> Net-(U16B-+)
- R52 pad 2: +3V3 -> Net-(U16A--)
- R68 pad 2: Net-(SW10-C) -> 24V_SENSE
- R69 pad 1: Net-(SW10-C) -> 24V_SENSE
- U24 pad 1: USBPD_CC1 -> USBPD_D-
- U24 pad 3: USBPD_D- -> USBPD_CC1
- U3 pad 10: GND -> BL_ISENSE
- U3 pad 15: +3V3 -> Net-(U3-V3P3)
- U3 pad 6: GND -> BL_ISENSE
- U3 pad 7: GND -> BL_ISENSE
- U4 pad 4: SDA -> I2C_IRQ
- U4 pad 5: SCL -> SDA
- U4 pad 6: I2C_IRQ -> SCL
- U5 pad 10: Servo1 -> Servo3
- U5 pad 11: Servo2 -> Servo4
- U5 pad 12: DAC1_OUT1 -> ROT_A
- U5 pad 13: DAC1_OUT2 -> ROT_B
- U5 pad 14: Servo3 -> FAN2_DRIVE
- U5 pad 15: FAN2_DRIVE -> GND
- U5 pad 16: HEATER -> +3V3
- U5 pad 17: BL_HALL2 -> LED_WHITE_P
- U5 pad 18: BL_HALL1 -> DAC1_OUT1
- U5 pad 19: BRIGHTNESS -> DAC1_OUT2
- U5 pad 2: BTN_YEL -> MOVE
- U5 pad 20: Net-(U5-VDDA) -> BL_HALL3
- U5 pad 21: Net-(U5-VDDA) -> BL_HALL2
- U5 pad 22: unconnected-(U5-PB10-Pad22) -> ADC_IN1
- U5 pad 23: +3V3 -> ADC_IN2
- U5 pad 24: Relais -> BL_HALL1
- U5 pad 25: BL_RESET -> OPAMP3Q
- U5 pad 26: BL_FAULT -> OPAMP3-
- U5 pad 27: ADC_IN1 -> GND
- U5 pad 28: ADC_IN2 -> Net-(U5-VDDA)
- U5 pad 29: BL_ENABLEx -> Net-(U5-VDDA)
- U5 pad 3: MOVE -> HEATER
- U5 pad 30: BL_DRV1 -> UART3_TX
- U5 pad 31: BL_DRV2 -> GND
- U5 pad 32: BL_DRV3 -> +3V3
- U5 pad 33: USBPD_D- -> UART3_RX
- U5 pad 34: USBPD_D+ -> PB12
- U5 pad 35: +3V3 -> OPAMP3+
- U5 pad 36: SWDIO -> BL_ISENSE
- U5 pad 37: SWCLK -> 24V_SENSE
- U5 pad 38: SCL -> BL_DRV1
- U5 pad 39: UART4_TX -> BL_DRV2
- U5 pad 4: unconnected-(U5-PC15-Pad4) -> Relais
- U5 pad 40: UART4_RX -> BL_DRV3
- U5 pad 41: LED_INFO -> BL_FAULT
- U5 pad 42: USBPD_CC2 -> BL_SLEEP
- U5 pad 43: BL_HALL3 -> USBPD_CC1
- U5 pad 44: USBPD_CC1 -> USBPD_CC2
- U5 pad 45: SDA -> USBPD_D-
- U5 pad 46: BTN_RED -> USBPD_D+
- U5 pad 47: LED_WHITE_P -> GND
- U5 pad 49: GND -> SWDIO
- U5 pad 5: Net-(U5-PF0) -> BRIGHTNESS
- U5 pad 6: Net-(U5-PF1) -> BTN_YEL
- U5 pad 8: ROT_A -> Servo1
- U5 pad 9: ROT_B -> Servo2
Routing:
- net GND: track 461.0 -> 408.6 mm, vias 429 -> 362
- net +24V: track 123.9 -> 167.1 mm, vias 4 -> 5
- net I2C_IRQ: track 167.6 -> 124.8 mm, vias 5 -> 4
- net ADC_IN2: track 26.6 -> 65.4 mm
- net BL_ISENSE: track 0.00 -> 35.6 mm, vias 0 -> 2
- net ADC_IN2_EXT: track 33.0 -> 0.00 mm
- net ROT_A: track 86.3 -> 59.0 mm
- net ROT_B: track 79.8 -> 52.7 mm
- net 24V_SENSE: track 0.00 -> 20.2 mm
- net BTN_YEL: track 84.0 -> 66.1 mm
- net Servo4: track 0.00 -> 16.8 mm
- net +5V: track 187.1 -> 173.2 mm
- net OPAMP3-: track 0.00 -> 13.3 mm
- net ADC_IN1: track 50.2 -> 63.5 mm
- net HEATER: track 70.6 -> 58.2 mm
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Other:
- outline, holes or cut-outs redrawn
- board text added: "B15"
- board text added: "Movement"
- board text added: "OP 3+"
- board text added: "OP3-"
- board text added: "OP3Q"
- board text added: "RX3"
- board text added: "Sig"
- board text added: "TX3"
- board text added: "lab@home v15.1 2024-08-01 Klaus Liebler For Science /Education / DIY"
- board text removed: "5"
- board text removed: "G"
- board text removed: "PIR Sensor"
- board text removed: "S"
- board text removed: "lab@home v15 2024-07-08 Klaus Liebler For Science /Education / DIY"
