File: labathome_pcb15/audioamplifier.kicad_sch (KiCad schematic)
At the start: 33 parts, among them U1 TAS5805M

Commit message: PCB_v15 wip
Parts:
- removed C1, C8: 470u, Capacitor_THT:CP_Radial_D10.0mm_P3.50mm, symbol Device:CP
- removed C10, C5: u1, Capacitor_SMD:C_0603_1608Metric, symbol Device:C
- removed C11: u22, Capacitor_SMD:C_0603_1608Metric, symbol Device:C
- removed C2: 4u7, Capacitor_SMD:C_0402_1005Metric, symbol Device:C
- removed C26, C27, C28, C29, C30, C31, C32, C33: 2n2/100V, Capacitor_SMD:C_0603_1608Metric, symbol Device:C
- removed C3, C9: 22u, Capacitor_SMD:C_1210_3225Metric_Pad1.33x2.70mm_HandSolder, symbol Device:C
- removed C4: u1, Capacitor_SMD:C_0402_1005Metric, symbol Device:C
- removed C6, C7: 1u, Capacitor_SMD:C_0402_1005Metric, symbol Device:C
- removed FB2, FB3, FB4: 300R3A, Resistor_SMD:R_1206_3216Metric, symbol Device:FerriteBead_Small
- removed NT1: Net-Tie_2, NetTie:NetTie-2_SMD_Pad2.0mm, symbol Device:Net-Tie_2
- removed R4: 4k7, Resistor_SMD:R_0402_1005Metric, symbol Device:R
- removed U1: TAS5805M, Package_SO:HTSSOP-28-1EP_4.4x9.7mm_P0.65mm_EP2.85x5.4mm_ThermalVias, symbol liebler_SEMICONDUCTORS:TAS5805M
- added C15, C21, C22: 4u7, Capacitor_SMD:C_0402_1005Metric, symbol Device:C
- added C16, C17, C20, C23, C24, C25: 1u, Capacitor_SMD:C_0402_1005Metric, symbol Device:C
- added C18, C19: 220u, Capacitor_SMD:CP_Elec_6.3x5.4, symbol Device:C_Polarized
- added J14: AUX OUT, liebler_CONN:PJ-327A, symbol Connector_Audio:AudioJack3_SwitchT
- added J16: Headphones, liebler_CONN:PJ-327A, symbol Connector_Audio:AudioJack3_SwitchT
- added J3: AUX IN, liebler_CONN:PJ-327A, symbol Connector_Audio:AudioJack3_SwitchT
- added LS1: Speaker, Connector_PinHeader_2.00mm:PinHeader_1x02_P2.00mm_Vertical, symbol Device:Speaker
- added LS2: Speaker, liebler_MECH:SPEAKER_2415, symbol Mechanical:MountingHole
- added MK1: Mic, liebler_PASSIVES:Microphone_6mm, symbol Device:Microphone_Condenser
- added NT1: NetTie_2, NetTie:NetTie-2_SMD_Pad0.5mm, symbol Device:NetTie_2
- added R23: 0R, Resistor_SMD:R_0402_1005Metric, symbol Device:R
- added R55: 10k, Resistor_SMD:R_0402_1005Metric, symbol Device:R
- added U10: ~, Package_DFN_QFN:QFN-32-1EP_5x5mm_P0.5mm_EP3.6x3.6mm_ThermalVias, symbol liebler_SEMICONDUCTORS:NAU88C22
- C12, C13, C14: value u22 -> 4u7; footprint Capacitor_SMD:C_0603_1608Metric -> Capacitor_SMD:C_0402_1005Metric
- FB1: value 300R3A -> Bead; footprint Resistor_SMD:R_1206_3216Metric -> Inductor_SMD:L_0603_1608Metric
- R24: value 68R -> 2k2; footprint Resistor_SMD:R_0603_1608Metric -> Resistor_SMD:R_0402_1005Metric
- R25: value 68R -> M22; footprint Resistor_SMD:R_0603_1608Metric -> Resistor_SMD:R_0402_1005Metric
- R26, R27: value 68R -> 10k; footprint Resistor_SMD:R_0603_1608Metric -> Resistor_SMD:R_0402_1005Metric
Connections:
- net OUT_A+ is gone; now on net +3V3: FB1.2
- net +3V3: now also C12.1, C13.1, R25.1, U10.13 (VDDC), U10.14 (VDDB)
- net GND: now also C12.2, C13.2, R26.2, NT1.1, U10.12 (VSSD)
- net GNDA: now also C14.2, C15.2, C21.2, C22.2, J14.S, J16.S, J16.TN, J3.S, NT1.2, R23.1, R55.2, U10.24 (VSSSPK), U10.28 (VSSA), U10.33 (EXPOSED_PAD); no longer R24.2, R25.2, R26.2
- net JACK_DETECT: now reaches R27.1
- net JACK_DETECT: now also R25.2, C18.2, J16.T, U10.3 (LLIN/GPIO2)
- net +3.3VA: now reaches C14.1
- net +3.3VA: now also FB1.1, U10.31 (VDDA)
- net at R24.1: now also C22.1, U10.32 (MICBIAS)
- net at R26.1: now also U10.18 (MODE)
- new net: C17.2, J14.R
- new net: C16.2, J14.T
- new net: C19.1, U10.29 (RHP)
- new net: C19.2, J16.R, R55.1
- new net: C24.1, J3.R
- new net: C24.2, U10.20 (RAUXIN)
- new net: LS1.1, U10.25 (LSPKOUT)
- new net: LS1.2, U10.23 (RSPKOUT)
- new net: C23.1, MK1.2 (+), R24.2
- new net: C25.1, J3.T
- new net: C25.2, U10.19 (LAUXIN)
- new net: C17.1, U10.22 (AUXOUT2)
- new net: C20.1, MK1.1 (-), R23.2
- new net: C18.1, U10.30 (LHP)
- new net: C20.2, U10.2 (LMICN), U10.5 (RMICN)
- new net: C23.2, U10.1 (LMICP), U10.4 (RMICP)
- new net: C21.1, U10.27 (VREF)
- new net: C16.1, U10.21 (AUXOUT1)
- new net +5V: C15.1, U10.26 (VDDSPK)
- new net I2S_ADC: U10.9 (ADCOUT)
- new net I2S_BCLK: U10.8 (BCLK)
- new net I2S_DAC: U10.10 (DACIN)
- new net I2S_FS: U10.7 (FS)
- new net I2S_MCLK: U10.11 (MCLK)
- new net SCL: U10.16 (SCLK)
- new net SDA: U10.17 (SDIO)
- no-connect marks 1 -> 2

Commit message: labathome wip
Parts:
- FB1: footprint Inductor_SMD:L_0603_1608Metric -> Inductor_SMD:L_0603_1608Metric
Changed lines of the file:
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@@
 			)
 		)
-		(property "Footprint" "Inductor_SMD:L_0603_1608Metric "
+		(property "Footprint" "Inductor_SMD:L_0603_1608Metric"
 			(at 125.73 38.608 90)
 			(effects

Commit message: labathome_pcb15 v0.0.2
Parts:
- added DRAWING5: Speaker, liebler_DRAWINGS:speaker, symbol Mechanical:Fiducial
Changed lines of the file:
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@@
+	)
+	(symbol
+		(lib_id "Mechanical:Fiducial")
+		(at 143.51 100.33 0)
+		(unit 1)
+		(exclude_from_sim yes)
+		(in_bom no)
+		(on_board yes)
+		(dnp no)
+		(fields_autoplaced yes)
+		(property "Reference" "DRAWING5"
+			(at 146.05 99.0599 0)
+			(effects
+				(font
+					(size 1.27 1.27)
+				)
+				(justify left)
+			)
+		)
+		(property "Value" "Speaker"
+			(at 146.05 101.5999 0)
+			(effects
+				(font
+					(size 1.27 1.27)
+				)
+				(justify left)
+			)
+		)
+		(property "Footprint" "liebler_DRAWINGS:speaker"
+			(at 143.51 100.33 0)
+			(effects
+				(font
+					(size 1.27 1.27)
+				)
+				(hide yes)
+			)
+		)
+		(property "Datasheet" "~"
+			(at 143.51 100.33 0)
+			(effects
+				(font
+					(size 1.27 1.27)
+				)
+				(hide yes)
+			)
+		)
+		(property "Description" "Fiducial Marker"
+			(at 143.51 100.33 0)
+			(effects
+				(font
+					(size 1.27 1.27)
+				)
+				(hide yes)
+			)
+		)
+		(instances
+			(project "labathome_pcb15"
+				(path "/e4d6926a-1a8b-424d-97c4-66b6ad87e4ac/2f2efef3-f887-4727-9b58-1fbd8d1c6d1d"
+					(reference "DRAWING5")
+					(unit 1)
+				)
+			)
+		)
 	)
 	(symbol

Commit message: labathome_pcb15
Parts:
- added JP1: JFS, Jumper:SolderJumper-2_P1.3mm_Bridged2Bar_RoundedPad1.0x1.5mm, symbol Jumper:Jumper_2_Small_Bridged
- added R54: M1, Resistor_SMD:R_0402_1005Metric, symbol Device:R
- R25: value M22 -> M1
- U10: value ~ -> NAU8822
Connections:
- net +3V3: now also R54.1; no longer R25.1
- net I2S_FS: now also JP1.1 (A); no longer U10.7 (FS)
- new net: R25.1, R54.2
- new net: JP1.2 (B), U10.7 (FS)
Changed lines of the file:
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@@
 	(wire
 		(pts
+			(xy 142.24 59.69) (xy 144.78 59.69)
+		)
+		(stroke
+			(width 0)
+			(type default)
+		)
+	)
+	(wire
+		(pts
 			(xy 100.33 87.63) (xy 102.87 87.63)
 		)
@@
 	(wire
 		(pts
+			(xy 147.32 68.58) (xy 142.24 68.58)
+		)
+		(stroke
+			(width 0)
+			(type default)
+		)
+	)
+	(wire
+		(pts
 			(xy 44.45 102.87) (xy 44.45 101.6)
 		)
@@
 	(wire
 		(pts
+			(xy 142.24 68.58) (xy 142.24 67.31)
+		)
+		(stroke
+			(width 0)
+			(type default)
+		)
+	)
+	(wire
+		(pts
 			(xy 59.69 82.55) (xy 50.8 82.55)
 		)
@@
 	(wire
 		(pts
+			(xy 144.78 60.96) (xy 147.32 60.96)
+		)
+		(stroke
+			(width 0)
+			(type default)
+		)
+	)
+	(wire
+		(pts
 			(xy 53.34 102.87) (xy 44.45 102.87)
 		)
@@
 	(wire
 		(pts
+			(xy 144.78 59.69) (xy 144.78 60.96)
+		)
+		(stroke
+			(width 0)
+			(type default)
+		)
+	)
+	(wire
+		(pts
 			(xy 60.96 102.87) (xy 74.93 102.87)
 		)
@@
 	(global_label "I2S_FS"
 		(shape bidirectional)
-		(at 74.93 58.42 180)
+		(at 69.85 58.42 180)
 		(fields_autoplaced yes)
 		(effects
@@
 		)
 		(property "Intersheetrefs" "${INTERSHEET_REFS}"
-			(at 64.544 58.42 0)
+			(at 59.464 58.42 0)
 			(effects
 				(font
@@
 	)
 	(symbol
+		(lib_id "Device:R")
+		(at 142.24 63.5 0)
+		(unit 1)
+		(exclude_from_sim no)
+		(in_bom yes)
+		(on_board yes)
+		(dnp no)
+		(property "Reference" "R54"
+			(at 140.208 63.5 90)
+			(effects
+				(font
+					(size 1.27 1.27)
+				)
+			)
+		)
+		(property "Value" "M1"
+			(at 142.24 63.5 90)
+			(effects
+				(font
+					(size 1.27 1.27)
+				)
+			)
+		)
+		(property "Footprint" "Resistor_SMD:R_0402_1005Metric"
+			(at 140.462 63.5 90)
+			(effects
+				(font
+					(size 1.27 1.27)
+				)
+				(hide yes)
+			)
+		)
+		(property "Datasheet" "~"
+			(at 142.24 63.5 0)
+			(effects
+				(font
+					(size 1.27 1.27)
+				)
+				(hide yes)
+			)
+		)
+		(property "Description" "Resistor"
+			(at 142.24 63.5 0)
+			(effects
+				(font
+					(size 1.27 1.27)
+				)
+				(hide yes)
+			)
+		)
+		(pin "1"
+		)
+		(pin "2"
+		)
+		(instances
+			(project "labathome_pcb15"
+				(path "/e4d6926a-1a8b-424d-97c4-66b6ad87e4ac/2f2efef3-f887-4727-9b58-1fbd8d1c6d1d"
+					(reference "R54")
+					(unit 1)
+				)
+			)
+		)
+	)
+	(symbol
 		(lib_id "Device:Speaker")
 		(at 107.95 90.17 0)
@@
 			)
 		)
-		(property "Value" "M22"
+		(property "Value" "M1"
 			(at 147.32 72.39 90)
 			(effects
@@
 	)
 	(symbol
+		(lib_id "Jumper:Jumper_2_Small_Bridged")
+		(at 72.39 58.42 0)
+		(unit 1)
+		(exclude_from_sim yes)
+		(in_bom yes)
+		(on_board yes)
+		(dnp no)
+		(property "Reference" "JP1"
+			(at 72.39 53.34 0)
+			(effects
+				(font
+					(size 1.27 1.27)
+				)
+			)
+		)
+		(property "Value" "JFS"
+			(at 57.15 58.42 0)
+			(effects
+				(font
+					(size 1.27 1.27)
+				)
+			)
+		)
+		(property "Footprint" "Jumper:SolderJumper-2_P1.3mm_Bridged2Bar_RoundedPad1.0x1.5mm"
+			(at 72.39 58.42 0)
+			(effects
+				(font
+					(size 1.27 1.27)
+				)
+				(hide yes)
+			)
+		)
+		(property "Datasheet" "~"
+			(at 72.39 58.42 0)
+			(effects
+				(font
+					(size 1.27 1.27)
+				)
+				(hide yes)
+			)
+		)
+		(property "Description" "Jumper, 2-pole, small symbol, bridged"
+			(at 72.39 58.42 0)
+			(effects
+				(font
+					(size 1.27 1.27)
+				)
+				(hide yes)
+			)
+		)
+		(pin "2"
+		)
+		(pin "1"
+		)
+		(instances
+			(project ""
+				(path "/e4d6926a-1a8b-424d-97c4-66b6ad87e4ac/2f2efef3-f887-4727-9b58-1fbd8d1c6d1d"
+					(reference "JP1")
+					(unit 1)
+				)
+			)
+		)
+	)
+	(symbol
 		(lib_id "power:GNDA")
 		(at 134.62 52.07 0)
@@
 			)
 		)
-		(property "Value" "~"
+		(property "Value" "NAU8822"
 			(at 87.63 49.53 0)
 			(effects
@@
 	(symbol
 		(lib_id "power:+3V3")
-		(at 147.32 68.58 0)
+		(at 147.32 60.96 0)
 		(unit 1)
 		(exclude_from_sim no)
@@
 		(dnp no)
 		(property "Reference" "#PWR0177"
-			(at 147.32 72.39 0)
+			(at 147.32 64.77 0)
 			(effects
 				(font
@@
 		)
 		(property "Value" "+3V3"
-			(at 147.32 64.516 0)
+			(at 147.32 56.896 0)
 			(effects
 				(font
@@
 		)
 		(property "Footprint" ""
-			(at 147.32 68.58 0)
+			(at 147.32 60.96 0)
 			(effects
 				(font
@@
 		)
 		(property "Datasheet" ""
-			(at 147.32 68.58 0)
+			(at 147.32 60.96 0)
 			(effects
 				(font
@@
 		)
 		(property "Description" "Power symbol creates a global label with name \"+3V3\""
-			(at 147.32 68.58 0)
+			(at 147.32 60.96 0)
 			(effects
 				(font

Commit message: labathome_pcb5 ready for review, 2nd
Parts:
- removed DRAWING5: Speaker, liebler_DRAWINGS:speaker, symbol Mechanical:Fiducial
Changed lines of the file:
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@@
-	)
-	(symbol
-		(lib_id "Mechanical:Fiducial")
-		(at 143.51 100.33 0)
-		(unit 1)
-		(exclude_from_sim yes)
-		(in_bom no)
-		(on_board yes)
-		(dnp no)
-		(fields_autoplaced yes)
-		(property "Reference" "DRAWING5"
-			(at 146.05 99.0599 0)
-			(effects
-				(font
-					(size 1.27 1.27)
-				)
-				(justify left)
-			)
-		)
-		(property "Value" "Speaker"
-			(at 146.05 101.5999 0)
-			(effects
-				(font
-					(size 1.27 1.27)
-				)
-				(justify left)
-			)
-		)
-		(property "Footprint" "liebler_DRAWINGS:speaker"
-			(at 143.51 100.33 0)
-			(effects
-				(font
-					(size 1.27 1.27)
-				)
-				(hide yes)
-			)
-		)
-		(property "Datasheet" "~"
-			(at 143.51 100.33 0)
-			(effects
-				(font
-					(size 1.27 1.27)
-				)
-				(hide yes)
-			)
-		)
-		(property "Description" "Fiducial Marker"
-			(at 143.51 100.33 0)
-			(effects
-				(font
-					(size 1.27 1.27)
-				)
-				(hide yes)
-			)
-		)
-		(instances
-			(project "labathome_pcb15"
-				(path "/e4d6926a-1a8b-424d-97c4-66b6ad87e4ac/2f2efef3-f887-4727-9b58-1fbd8d1c6d1d"
-					(reference "DRAWING5")
-					(unit 1)
-				)
-			)
-		)
 	)
 	(symbol

Commit message: Various PCB and Code updates after review from Jana Marie Hemsing. Big Thankyou
Parts:
- removed C16, C17, C20, C23, C24, C25: 1u, Capacitor_SMD:C_0402_1005Metric, symbol Device:C
- added C16, C17, C20, C23, C24, C62: 1u, Capacitor_Tantalum_SMD:CP_EIA-3216-10_Kemet-I, symbol Device:C_Polarized_Small
Connections:
- net at J14.R: now also C17.2
- net at J14.T: now also C16.2
- net at J3.R: now also C24.1
- net at U10.20 (RAUXIN): now also C24.2
- net at MK1.2 (+), R24.2: now also C23.1
- net at J3.T: now also C62.1
- net at U10.19 (LAUXIN): now also C62.2
- net at U10.22 (AUXOUT2): now also C17.1
- net at MK1.1 (-), R23.2: now also C20.1
- net at U10.2 (LMICN), U10.5 (RMICN): now also C20.2
- net at U10.1 (LMICP), U10.4 (RMICP): now also C23.2
- net at U10.21 (AUXOUT1): now also C16.1

Commit message: Further improventents in PCB layout
Parts:
- removed JP1: JFS, Jumper:SolderJumper-2_P1.3mm_Bridged2Bar_RoundedPad1.0x1.5mm, symbol Jumper:Jumper_2_Small_Bridged
Connections:
- net I2S_FS: now also U10.7 (FS)
- no-connect marks 2 -> 4
Changed lines of the file:
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@@
 	)
 	(junction
+		(at 119.38 36.83)
+		(diameter 0)
+		(color 0 0 0 0)
+	)
+	(junction
+		(at 104.14 36.83)
+		(diameter 0)
+		(color 0 0 0 0)
+	)
+	(junction
 		(at 44.45 91.44)
 		(diameter 0)
@@
 	)
 	(no_connect
+		(at 118.11 66.04)
+	)
+	(no_connect
 		(at 74.93 81.28)
 	)
@@
 		(at 74.93 72.39)
 	)
+	(no_connect
+		(at 50.8 74.93)
+	)
 	(wire
 		(pts
@@
 	(wire
 		(pts
+			(xy 119.38 36.83) (xy 123.19 36.83)
+		)
+		(stroke
+			(width 0)
+			(type default)
+		)
+	)
+	(wire
+		(pts
 			(xy 69.85 99.06) (xy 69.85 96.52)
 		)
@@
 	(wire
 		(pts
+			(xy 116.84 36.83) (xy 119.38 36.83)
+		)
+		(stroke
+			(width 0)
+			(type default)
+		)
+	)
+	(wire
+		(pts
+			(xy 104.14 36.83) (xy 97.79 36.83)
+		)
+		(stroke
+			(width 0)
+			(type default)
+		)
+	)
+	(wire
+		(pts
 			(xy 53.34 96.52) (xy 53.34 102.87)
 		)
@@
 	(global_label "I2S_FS"
 		(shape bidirectional)
-		(at 69.85 58.42 180)
+		(at 74.93 58.42 180)
 		(fields_autoplaced yes)
 		(effects
@@
 		)
 		(property "Intersheetrefs" "${INTERSHEET_REFS}"
-			(at 59.464 58.42 0)
+			(at 64.544 58.42 0)
 			(effects
 				(font
@@
 	)
 	(symbol
+		(lib_id "power:PWR_FLAG")
+		(at 119.38 36.83 0)
+		(unit 1)
+		(exclude_from_sim no)
+		(in_bom yes)
+		(on_board yes)
+		(dnp no)
+		(fields_autoplaced yes)
+		(property "Reference" "#FLG06"
+			(at 119.38 34.925 0)
+			(effects
+				(font
+					(size 1.27 1.27)
+				)
+				(hide yes)
+			)
+		)
+		(property "Value" "PWR_FLAG"
+			(at 119.38 31.75 0)
+			(effects
+				(font
+					(size 1.27 1.27)
+				)
+			)
+		)
+		(property "Footprint" ""
+			(at 119.38 36.83 0)
+			(effects
+				(font
+					(size 1.27 1.27)
+				)
+				(hide yes)
+			)
+		)
+		(property "Datasheet" "~"
+			(at 119.38 36.83 0)
+			(effects
+				(font
+					(size 1.27 1.27)
+				)
+				(hide yes)
+			)
+		)
+		(property "Description" "Special symbol for telling ERC where power comes from"
+			(at 119.38 36.83 0)
+			(effects
+				(font
+					(size 1.27 1.27)
+				)
+				(hide yes)
+			)
+		)
+		(pin "1"
+		)
+		(instances
+			(project ""
+				(path "/e4d6926a-1a8b-424d-97c4-66b6ad87e4ac/2f2efef3-f887-4727-9b58-1fbd8d1c6d1d"
+					(reference "#FLG06")
+					(unit 1)
+				)
+			)
+		)
+	)
+	(symbol
 		(lib_id "Device:R")
 		(at 38.1 91.44 90)
@@
 	(symbol
 		(lib_id "power:+3.3VA")
-		(at 123.19 36.83 90)
+		(at 116.84 36.83 90)
 		(unit 1)
 		(exclude_from_sim no)
@@
 		(dnp no)
 		(property "Reference" "#PWR0180"
-			(at 127 36.83 0)
+			(at 120.65 36.83 0)
 			(effects
 				(font
@@
 		)
 		(property "Value" "+3.3VA"
-			(at 120.142 34.29 90)
+			(at 113.792 34.29 90)
 			(effects
 				(font
@@
 		)
 		(property "Footprint" ""
-			(at 123.19 36.83 0)
+			(at 116.84 36.83 0)
 			(effects
 				(font
@@
 		)
 		(property "Datasheet" ""
-			(at 123.19 36.83 0)
+			(at 116.84 36.83 0)
 			(effects
 				(font
@@
 		)
 		(property "Description" "Power symbol creates a global label with name \"+3.3VA\""
-			(at 123.19 36.83 0)
+			(at 116.84 36.83 0)
 			(effects
 				(font
@@
 	(symbol
 		(lib_id "power:GNDA")
-		(at 97.79 36.83 90)
+		(at 104.14 36.83 90)
 		(unit 1)
 		(exclude_from_sim no)
@@
 		(dnp no)
 		(property "Reference" "#PWR0183"
-			(at 104.14 36.83 0)
+			(at 110.49 36.83 0)
 			(effects
 				(font
@@
 		)
 		(property "Value" "GNDA"
-			(at 98.044 39.116 90)
+			(at 104.394 39.116 90)
 			(effects
 				(font
@@
 		)
 		(property "Footprint" ""
-			(at 97.79 36.83 0)
+			(at 104.14 36.83 0)
 			(effects
 				(font
@@
 		)
 		(property "Datasheet" ""
-			(at 97.79 36.83 0)
+			(at 104.14 36.83 0)
 			(effects
 				(font
@@
 		)
 		(property "Description" "Power symbol creates a global label with name \"GNDA\" , analog ground"
-			(at 97.79 36.83 0)
+			(at 104.14 36.83 0)
 			(effects
 				(font
@@
 	)
 	(symbol
-		(lib_id "Jumper:Jumper_2_Small_Bridged")
-		(at 72.39 58.42 0)
-		(unit 1)
-		(exclude_from_sim yes)
-		(in_bom yes)
-		(on_board yes)
-		(dnp no)
-		(property "Reference" "JP1"
-			(at 72.39 53.34 0)
-			(effects
-				(font
-					(size 1.27 1.27)
-				)
-			)
-		)
-		(property "Value" "JFS"
-			(at 57.15 58.42 0)
-			(effects
-				(font
-					(size 1.27 1.27)
-				)
-			)
-		)
-		(property "Footprint" "Jumper:SolderJumper-2_P1.3mm_Bridged2Bar_RoundedPad1.0x1.5mm"
-			(at 72.39 58.42 0)
-			(effects
-				(font
-					(size 1.27 1.27)
-				)
-				(hide yes)
-			)
-		)
-		(property "Datasheet" "~"
-			(at 72.39 58.42 0)
-			(effects
-				(font
-					(size 1.27 1.27)
-				)
-				(hide yes)
-			)
-		)
-		(property "Description" "Jumper, 2-pole, small symbol, bridged"
-			(at 72.39 58.42 0)
-			(effects
-				(font
-					(size 1.27 1.27)
-				)
-				(hide yes)
-			)
-		)
-		(pin "2"
-		)
-		(pin "1"
-		)
-		(instances
-			(project ""
-				(path "/e4d6926a-1a8b-424d-97c4-66b6ad87e4ac/2f2efef3-f887-4727-9b58-1fbd8d1c6d1d"
-					(reference "JP1")
-					(unit 1)
-				)
-			)
-		)
-	)
-	(symbol
 		(lib_id "power:GNDA")
 		(at 134.62 52.07 0)
@@
 					(unit 1)
 				)
+			)
+		)
+	)
+	(symbol
+		(lib_id "power:PWR_FLAG")
+		(at 104.14 36.83 0)
+		(unit 1)
+		(exclude_from_sim no)
+		(in_bom yes)
+		(on_board yes)
+		(dnp no)
+		(fields_autoplaced yes)
+		(property "Reference" "#FLG07"
+			(at 104.14 34.925 0)
+			(effects
+				(font
+					(size 1.27 1.27)
+				)
+				(hide yes)
+			)
+		)
+		(property "Value" "PWR_FLAG"
+			(at 104.14 31.75 0)
+			(effects
+				(font
+					(size 1.27 1.27)
+				)
+			)
+		)
+		(property "Footprint" ""
+			(at 104.14 36.83 0)
+			(effects
+				(font
+					(size 1.27 1.27)
+				)
+				(hide yes)
+			)
+		)
+		(property "Datasheet" "~"
+			(at 104.14 36.83 0)
+			(effects
+				(font
+					(size 1.27 1.27)
+				)
+				(hide yes)
+			)
+		)
+		(property "Description" "Special symbol for telling ERC where power comes from"
+			(at 104.14 36.83 0)
+			(effects
+				(font
+					(size 1.27 1.27)
+				)
+				(hide yes)
+			)
+		)
+		(pin "1"
+		)
+		(instances
+			(project ""
+				(path "/e4d6926a-1a8b-424d-97c4-66b6ad87e4ac/2f2efef3-f887-4727-9b58-1fbd8d1c6d1d"
+					(reference "#FLG07")
+					(unit 1)
+				)
