File: labathome_pcb15/audioamplifier.kicad_sch (KiCad schematic)
At the start: 30 parts, among them J14 AUX OUT, J16 Headphones, J3 AUX IN, U10 NAU8822

Commit message: Final PCB as ordered @ JLCPCB
Parts:
- added JP1: Jumper_2_Bridged, Jumper:SolderJumper-2_P1.3mm_Bridged2Bar_Pad1.0x1.5mm, symbol Jumper:Jumper_2_Bridged
- R23: footprint Resistor_SMD:R_0402_1005Metric -> Diode_SMD:D_0805_2012Metric_Pad1.15x1.40mm_HandSolder; now not fitted
Connections:
- net GNDA: now also JP1.1 (A)
- net at C20.1, MK1.1 (-), R23.2: now also JP1.2 (B)
Changed lines of the file:
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@@
+	)
+	(junction
+		(at 34.29 91.44)
+		(diameter 0)
+		(color 0 0 0 0)
 	)
 	(junction
@@
 	(wire
 		(pts
+			(xy 44.45 88.9) (xy 44.45 91.44)
+		)
+		(stroke
+			(width 0)
+			(type default)
+		)
+	)
+	(wire
+		(pts
 			(xy 72.39 91.44) (xy 74.93 91.44)
 		)
@@
 		(pts
 			(xy 50.8 77.47) (xy 50.8 80.01)
+		)
+		(stroke
+			(width 0)
+			(type default)
+		)
+	)
+	(wire
+		(pts
+			(xy 34.29 88.9) (xy 34.29 91.44)
 		)
 		(stroke
@@
 				(justify right)
 				(hide yes)
+			)
+		)
+	)
+	(symbol
+		(lib_id "Jumper:Jumper_2_Bridged")
+		(at 39.37 88.9 0)
+		(unit 1)
+		(exclude_from_sim yes)
+		(in_bom yes)
+		(on_board yes)
+		(dnp no)
+		(fields_autoplaced yes)
+		(property "Reference" "JP1"
+			(at 39.37 83.82 0)
+			(effects
+				(font
+					(size 1.27 1.27)
+				)
+			)
+		)
+		(property "Value" "Jumper_2_Bridged"
+			(at 39.37 86.36 0)
+			(effects
+				(font
+					(size 1.27 1.27)
+				)
+			)
+		)
+		(property "Footprint" "Jumper:SolderJumper-2_P1.3mm_Bridged2Bar_Pad1.0x1.5mm"
+			(at 39.37 88.9 0)
+			(effects
+				(font
+					(size 1.27 1.27)
+				)
+				(hide yes)
+			)
+		)
+		(property "Datasheet" "~"
+			(at 39.37 88.9 0)
+			(effects
+				(font
+					(size 1.27 1.27)
+				)
+				(hide yes)
+			)
+		)
+		(property "Description" "Jumper, 2-pole, closed/bridged"
+			(at 39.37 88.9 0)
+			(effects
+				(font
+					(size 1.27 1.27)
+				)
+				(hide yes)
+			)
+		)
+		(pin "2"
+		)
+		(pin "1"
+		)
+		(instances
+			(project ""
+				(path "/e4d6926a-1a8b-424d-97c4-66b6ad87e4ac/2f2efef3-f887-4727-9b58-1fbd8d1c6d1d"
+					(reference "JP1")
+					(unit 1)
+				)
 			)
 		)
@@
 		(in_bom yes)
 		(on_board yes)
-		(dnp no)
+		(dnp yes)
 		(property "Reference" "R23"
 			(at 38.1 89.408 90)
@@
 			)
 		)
-		(property "Footprint" "Resistor_SMD:R_0402_1005Metric"
+		(property "Footprint" "Diode_SMD:D_0805_2012Metric_Pad1.15x1.40mm_HandSolder"
 			(at 38.1 93.218 90)
 			(effects

Commit message: lbathome 15.1
Parts:
- C12, C13, C14, C15, C21, C22: value 4u7 -> 4u7
Changed lines of the file:
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@@
 			)
 		)
-		(property "Value" "4u7	"
+		(property "Value" "4u7"
 			(at 78.74 107.9499 0)
 			(effects
@@
 			)
 		)
-		(property "Value" "4u7	"
+		(property "Value" "4u7"
 			(at 138.43 49.5299 0)
 			(effects
@@
 			)
 		)
-		(property "Value" "4u7	"
+		(property "Value" "4u7"
 			(at 104.14 107.9499 0)
 			(effects
@@
 			)
 		)
-		(property "Value" "4u7	"
+		(property "Value" "4u7"
 			(at 115.57 49.5299 0)
 			(effects
@@
 			)
 		)
-		(property "Value" "4u7	"
+		(property "Value" "4u7"
 			(at 127 49.5299 0)
 			(effects
@@
 			)
 		)
-		(property "Value" "4u7	"
+		(property "Value" "4u7"
 			(at 149.86 49.5299 0)
 			(effects

Commit message: Updates in PCB, arduino test firmware
Other:
- company: (none) -> Klaus Liebler
- title: (none) -> lab@home
Changed lines of the file:
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@@
 	(generator_version "8.0")
 	(paper "A4")
+	(title_block
+		(title "lab@home")
+		(date "2024-08-19")
+		(rev "15.1")
+		(company "Klaus Liebler")
+	)
 	(junction
 		(at 142.24 82.55)

Commit message: Reverse mount LEDs, switch
Parts:
- FB1: value Bead -> 600R
Changed lines of the file:
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@@
 			)
 		)
-		(property "Value" "Bead"
+		(property "Value" "600R"
 			(at 125.6919 33.02 90)
 			(effects

Commit message: Various last minute
Parts:
- added C65, C66: u1, Capacitor_SMD:C_0201_0603Metric, symbol Device:C
- added TP6: G3, TestPoint:TestPoint_THTPad_D1.0mm_Drill0.5mm, symbol Connector:TestPoint_Small
- R26: footprint Resistor_SMD:R_0402_1005Metric -> Resistor_SMD:R_0201_0603Metric
Connections:
- net +3V3: now also C65.1, C66.1
- net GND: now also C65.2, C66.2
- net at U10.6 (RLIN/GPIO3): now also TP6.1
- no-connect marks 4 -> 3
Other:
- moved on the sheet: C12, C13, C14, C15

Commit message: 4 Layers
Parts:
- R25, R27, R54, R55: footprint Resistor_SMD:R_0402_1005Metric -> Resistor_SMD:R_0201_0603Metric
Connections:
- net at C22.1, U10.32 (MICBIAS): now also R24.2; no longer R24.1
- net at C23.1, MK1.2 (+): now also R24.1; no longer R24.2
Other:
- moved on the sheet: R54
Changed lines of the file:
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@@
 	)
 	(junction
-		(at 147.32 77.47)
+		(at 74.93 102.87)
 		(diameter 0)
 		(color 0 0 0 0)
 	)
 	(junction
-		(at 144.78 91.44)
+		(at 147.32 77.47)
 		(diameter 0)
 		(color 0 0 0 0)
 	)
 	(junction
-		(at 152.4 49.53)
+		(at 144.78 91.44)
 		(diameter 0)
 		(color 0 0 0 0)
 	)
 	(junction
-		(at 74.93 102.87)
+		(at 152.4 49.53)
 		(diameter 0)
 		(color 0 0 0 0)
@@
 	(wire
 		(pts
-			(xy 142.24 59.69) (xy 144.78 59.69)
+			(xy 60.96 102.87) (xy 74.93 102.87)
 		)
 		(stroke
@@
 	(wire
 		(pts
-			(xy 147.32 68.58) (xy 142.24 68.58)
-		)
-		(stroke
-			(width 0)
-			(type default)
-		)
-	)
-	(wire
-		(pts
 			(xy 62.23 85.09) (xy 64.77 85.09)
 		)
@@
 	(wire
 		(pts
-			(xy 142.24 68.58) (xy 142.24 67.31)
+			(xy 147.32 68.58) (xy 147.32 67.31)
 		)
 		(stroke
@@
 	(wire
 		(pts
-			(xy 144.78 60.96) (xy 147.32 60.96)
-		)
-		(stroke
-			(width 0)
-			(type default)
-		)
-	)
-	(wire
-		(pts
 			(xy 53.34 102.87) (xy 44.45 102.87)
 		)
@@
 	(wire
 		(pts
-			(xy 144.78 59.69) (xy 144.78 60.96)
-		)
-		(stroke
-			(width 0)
-			(type default)
-		)
-	)
-	(wire
-		(pts
-			(xy 60.96 102.87) (xy 74.93 102.87)
-		)
-		(stroke
-			(width 0)
-			(type default)
-		)
-	)
-	(wire
-		(pts
 			(xy 153.67 71.12) (xy 153.67 74.93)
 		)
@@
 	(symbol
 		(lib_id "Device:R")
-		(at 142.24 63.5 0)
+		(at 147.32 63.5 0)
 		(unit 1)
 		(exclude_from_sim no)
@@
 		(dnp no)
 		(property "Reference" "R54"
-			(at 140.208 63.5 90)
+			(at 145.288 63.5 90)
 			(effects
 				(font
@@
 		)
 		(property "Value" "M1"
-			(at 142.24 63.5 90)
+			(at 147.32 63.5 90)
 			(effects
 				(font
@@
 			)
 		)
-		(property "Footprint" "Resistor_SMD:R_0402_1005Metric"
-			(at 140.462 63.5 90)
+		(property "Footprint" "Resistor_SMD:R_0201_0603Metric"
+			(at 145.542 63.5 90)
 			(effects
 				(font
@@
 		)
 		(property "Datasheet" "~"
-			(at 142.24 63.5 0)
+			(at 147.32 63.5 0)
 			(effects
 				(font
@@
 		)
 		(property "Description" "Resistor"
-			(at 142.24 63.5 0)
+			(at 147.32 63.5 0)
 			(effects
 				(font
@@
 	)
 	(symbol
-		(lib_id "Device:R")
-		(at 57.15 102.87 270)
-		(unit 1)
-		(exclude_from_sim no)
-		(in_bom yes)
-		(on_board yes)
-		(dnp no)
-		(property "Reference" "R24"
-			(at 57.15 100.838 90)
-			(effects
-				(font
-					(size 1.27 1.27)
-				)
-			)
-		)
-		(property "Value" "2k2"
-			(at 57.15 102.87 90)
-			(effects
-				(font
-					(size 1.27 1.27)
-				)
-			)
-		)
-		(property "Footprint" "Resistor_SMD:R_0402_1005Metric"
-			(at 57.15 101.092 90)
-			(effects
-				(font
-					(size 1.27 1.27)
-				)
-				(hide yes)
-			)
-		)
-		(property "Datasheet" "~"
-			(at 57.15 102.87 0)
-			(effects
-				(font
-					(size 1.27 1.27)
-				)
-				(hide yes)
-			)
-		)
-		(property "Description" "Resistor"
-			(at 57.15 102.87 0)
-			(effects
-				(font
-					(size 1.27 1.27)
-				)
-				(hide yes)
-			)
-		)
-		(pin "1"
-		)
-		(pin "2"
-		)
-		(instances
-			(project "labathome_pcb15"
-				(path "/e4d6926a-1a8b-424d-97c4-66b6ad87e4ac/2f2efef3-f887-4727-9b58-1fbd8d1c6d1d"
-					(reference "R24")
-					(unit 1)
-				)
-			)
-		)
-	)
-	(symbol
 		(lib_id "Device:C_Polarized_Small")
 		(at 72.39 87.63 90)
@@
 			)
 		)
-		(property "Footprint" "Resistor_SMD:R_0402_1005Metric"
+		(property "Footprint" "Resistor_SMD:R_0201_0603Metric"
 			(at 145.542 72.39 90)
 			(effects
@@
 			)
 		)
-		(property "Footprint" "Resistor_SMD:R_0402_1005Metric"
+		(property "Footprint" "Resistor_SMD:R_0201_0603Metric"
 			(at 140.462 87.63 90)
 			(effects
@@
 			)
 		)
-		(property "Footprint" "Resistor_SMD:R_0402_1005Metric"
+		(property "Footprint" "Resistor_SMD:R_0201_0603Metric"
 			(at 145.542 87.63 90)
 			(effects
@@
 	)
 	(symbol
+		(lib_id "Device:R")
+		(at 57.15 102.87 90)
+		(unit 1)
+		(exclude_from_sim no)
+		(in_bom yes)
+		(on_board yes)
+		(dnp no)
+		(property "Reference" "R24"
+			(at 55.8799 100.33 0)
+			(effects
+				(font
+					(size 1.27 1.27)
+				)
+				(justify left)
+			)
+		)
+		(property "Value" "2k2"
+			(at 58.674 102.87 90)
+			(effects
+				(font
+					(size 1.27 1.27)
+				)
+				(justify left)
+			)
+		)
+		(property "Footprint" "Resistor_SMD:R_0402_1005Metric"
+			(at 57.15 104.648 90)
+			(effects
+				(font
+					(size 1.27 1.27)
+				)
+				(hide yes)
+			)
+		)
+		(property "Datasheet" "~"
+			(at 57.15 102.87 0)
+			(effects
+				(font
+					(size 1.27 1.27)
+				)
+				(hide yes)
+			)
+		)
+		(property "Description" "Resistor"
+			(at 57.15 102.87 0)
+			(effects
+				(font
+					(size 1.27 1.27)
+				)
+				(hide yes)
+			)
+		)
+		(pin "1"
+		)
+		(pin "2"
+		)
+		(instances
+			(project "labathome_pcb15"
+				(path "/e4d6926a-1a8b-424d-97c4-66b6ad87e4ac/2f2efef3-f887-4727-9b58-1fbd8d1c6d1d"
+					(reference "R24")
+					(unit 1)
+				)
+			)
+		)
+	)
+	(symbol
 		(lib_id "Device:C")
 		(at 152.4 45.72 0)
@@
 	(symbol
 		(lib_id "power:+3V3")
-		(at 147.32 60.96 0)
+		(at 147.32 59.69 0)
 		(unit 1)
 		(exclude_from_sim no)
@@
 		(dnp no)
 		(property "Reference" "#PWR0177"
-			(at 147.32 64.77 0)
+			(at 147.32 63.5 0)
 			(effects
 				(font
@@
 		)
 		(property "Value" "+3V3"
-			(at 147.32 56.896 0)
+			(at 147.32 55.626 0)
 			(effects
 				(font
@@
 		)
 		(property "Footprint" ""
-			(at 147.32 60.96 0)
+			(at 147.32 59.69 0)
 			(effects
 				(font
@@
 		)
 		(property "Datasheet" ""
-			(at 147.32 60.96 0)
+			(at 147.32 59.69 0)
 			(effects
 				(font
@@
 		)
 		(property "Description" "Power symbol creates a global label with name \"+3V3\""
-			(at 147.32 60.96 0)
+			(at 147.32 59.69 0)
 			(effects
 				(font

Commit message: Minimal changes
Parts:
- added TP1: G2, TestPoint:TestPoint_THTPad_D1.0mm_Drill0.5mm, symbol Connector:TestPoint_Small
Connections:
- net JACK_DETECT: now also TP1.1
Changed lines of the file:
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@@
 	(wire
 		(pts
+			(xy 57.15 78.74) (xy 74.93 78.74)
+		)
+		(stroke
+			(width 0)
+			(type default)
+		)
+	)
+	(wire
+		(pts
 			(xy 147.32 68.58) (xy 147.32 67.31)
 		)
@@
 					(unit 1)
 				)
+			)
+		)
+	)
+	(symbol
+		(lib_id "Connector:TestPoint_Small")
+		(at 57.15 78.74 180)
+		(unit 1)
+		(exclude_from_sim no)
+		(in_bom yes)
+		(on_board yes)
+		(dnp no)
+		(fields_autoplaced yes)
+		(property "Reference" "TP1"
+			(at 58.42 77.4699 0)
+			(effects
+				(font
+					(size 1.27 1.27)
+				)
+				(justify right)
+			)
+		)
+		(property "Value" "G2"
+			(at 58.42 80.0099 0)
+			(effects
+				(font
+					(size 1.27 1.27)
+				)
+				(justify right)
+			)
+		)
+		(property "Footprint" "TestPoint:TestPoint_THTPad_D1.0mm_Drill0.5mm"
+			(at 52.07 78.74 0)
+			(effects
+				(font
+					(size 1.27 1.27)
+				)
+				(hide yes)
+			)
+		)
+		(property "Datasheet" "~"
+			(at 52.07 78.74 0)
+			(effects
+				(font
+					(size 1.27 1.27)
+				)
+				(hide yes)
+			)
+		)
+		(property "Description" "test point"
+			(at 57.15 78.74 0)
+			(effects
+				(font
+					(size 1.27 1.27)
+				)
+				(hide yes)
+			)
+		)
+		(pin "1"
+		)
+		(instances
+			(project "labathome_pcb15"
+				(path "/e4d6926a-1a8b-424d-97c4-66b6ad87e4ac/2f2efef3-f887-4727-9b58-1fbd8d1c6d1d"
+					(reference "TP1")
+					(unit 1)
+				)

Commit message: TPS2116
Parts:
- LS1: footprint Connector_PinHeader_2.00mm:PinHeader_1x02_P2.00mm_Vertical -> Inductor_SMD:L_Abracon_ASPI-0425
Changed lines of the file:
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@@
 			)
 		)
-		(property "Footprint" "Connector_PinHeader_2.00mm:PinHeader_1x02_P2.00mm_Vertical"
+		(property "Footprint" "Inductor_SMD:L_Abracon_ASPI-0425"
 			(at 107.95 85.09 0)
 			(effects
